File: Hardware/ETH1LCR3/MCU.kicad_sch (KiCad schematic)
At the start: 1 part, among them U301 STM32H743ZITx

Commit message: Hardware
Parts:
- removed U301: STM32H743ZITx, Package_QFP:LQFP-144_20x20mm_P0.5mm, symbol MCU_ST_STM32H7:STM32H743ZITx
- added C401, C403, C404, C405, C408, C410, C412, C415, C421, C422: 0.1u, Capacitor_SMD:C_0603_1608Metric_Pad1.08x0.95mm_HandSolder, symbol Device:C
- added C402, C406, C414: 1u, Capacitor_SMD:C_0603_1608Metric_Pad1.08x0.95mm_HandSolder, symbol Device:C
- added C416, C417: 8p, Capacitor_SMD:C_0603_1608Metric_Pad1.08x0.95mm_HandSolder, symbol Device:C
- added C418: 10u, Capacitor_SMD:C_0603_1608Metric_Pad1.08x0.95mm_HandSolder, symbol Device:C
- added C419, C420: 2u2, Capacitor_SMD:C_0603_1608Metric_Pad1.08x0.95mm_HandSolder, symbol Device:C
- added D401: ASMB-MTB1-0B3A2, LED_SMD:LED_Avago_PLCC4_3.2x2.8mm_CW, symbol LED:ASMB-MTB1-0A3A2
- added FB401: 742792031, Inductor_SMD:L_0805_2012Metric_Pad1.05x1.20mm_HandSolder, symbol Device:FerriteBead
- added J401: 20021111-00010T4LF, Connector_PinHeader_1.27mm:PinHeader_2x05_P1.27mm_Vertical, symbol Connector_Generic:Conn_02x05_Odd_Even
- added JP401: Open, Jumper:SolderJumper-2_P1.3mm_Open_Pad1.0x1.5mm, symbol Jumper:SolderJumper_2_Open
- added R402, R405: 10k, Resistor_SMD:R_0603_1608Metric_Pad0.98x0.95mm_HandSolder, symbol Device:R
- added R406: 0, Resistor_SMD:R_0603_1608Metric_Pad0.98x0.95mm_HandSolder, symbol Device:R
- added R407, R408: 4k7, Resistor_SMD:R_0603_1608Metric_Pad0.98x0.95mm_HandSolder, symbol Device:R
- added RN401: EXB-V8V102JV, Resistor_SMD:R_Array_Concave_4x0603, symbol Device:R_Pack04
- added U402: REF2033AIDDCT, Package_TO_SOT_SMD:SOT-23-5, symbol ETH1ISO224:REF19xxAIDDCT
- added U403: STM32H743VITx, Package_QFP:LQFP-100_14x14mm_P0.5mm, symbol MCU_ST_STM32H7:STM32H743VITx
- added U404: 24LC08B-E/MS, Package_SO:MSOP-8_3x3mm_P0.65mm, symbol Memory_EEPROM:24LC08
- added Y401: NX5032GA-16, ETH1ISO224:NX5032GA, symbol Device:Crystal
Connections:
- new net: D401.1 (RK), RN401.8 (R1.2)
- new net: D401.2 (GK), RN401.7 (R2.2)
- new net: D401.3 (BK), RN401.6 (R3.2)
- new net: C416.1, U403.12 (PH0), Y401.1
- new net: C417.1, U403.13 (PH1), Y401.2
- new net: C420.1, U403.73 (VCAP)
- new net: R406.1, U403.94 (BOOT0)
- new net: C419.1, U403.48 (VCAP)
- new net +3.3V: C401.1, C404.1, C408.1, C410.1, C412.1, C414.1, C422.2, D401.4 (A), FB401.2, J401.1 (Pin_1), R402.2, R405.1, R407.1, R408.1, U403.100 (VDD), U403.11 (VDD), U403.27 (VDD), U403.50 (VDD), U403.6 (VBAT), U403.75 (VDD), U404.8 (VCC)
- new net +3.3VADC: C403.1, C406.1, U402.5 (Vref), U403.20 (VREF+)
- new net +5V: C402.1, C405.1, U402.3 (EN), U402.4 (Vin)
- new net EEPROM_nWP: U403.91 (PB5), U404.7 (WP)
- new net GND: C401.2, C402.2, C403.2, C404.2, C405.2, C406.2, C408.2, C410.2, C412.2, C414.2, C415.2, C416.2, C417.2, C418.2, C419.2, C420.2, C421.2, C422.1, J401.3 (Pin_3), J401.5 (Pin_5), JP401.2 (B), R406.2, U402.2 (GND), U403.10 (VSS), U403.19 (VSSA), U403.26 (VSS), U403.49 (VSS), U403.74 (VSS), U403.99 (VSS), U404.1 (A0), U404.2 (A1), U404.3 (A2), U404.4 (GND)
- new net I2C1_SCL: R408.2, U403.92 (PB6), U404.6 (SCL)
- new net I2C1_SDA: R407.2, U403.93 (PB7), U404.5 (SDA)
- new net LED_BLUE: RN401.3 (R3.1), U403.63 (PC6)
- new net LED_GREEN: RN401.2 (R2.1), U403.65 (PC8)
- new net LED_RED: RN401.1 (R1.1), U403.66 (PC9)
- new net MCU_DEF: JP401.1 (A), R402.1, U403.1 (PE2)
- new net NRST: C415.1, J401.10 (Pin_10), R405.2, U403.14 (NRST)
- new net REF_CLK: U403.23 (PA1)
- new net RMII_CRS_DV: U403.31 (PA7)
- new net RMII_MDC: U403.16 (PC1)
- new net RMII_MDIO: U403.24 (PA2)
- new net RMII_RXD0: U403.32 (PC4)
- new net RMII_RXD1: U403.33 (PC5)
- new net RMII_TXD0: U403.51 (PB12)
- new net RMII_TXD1: U403.52 (PB13)
- new net RMII_TXEN: U403.47 (PB11)
- new net TCK_SWCLK: J401.4 (Pin_4), U403.76 (PA14)
- new net TMS_SWDIO: J401.2 (Pin_2), U403.72 (PA13)
- new net VCOM: U402.1 (Vbias)
- new net VDDA: C418.1, C421.1, FB401.1, U403.21 (VDDA)
- no-connect marks 0 -> 68
Other:
- note added: "Connect to VBAT"

Commit message: Hardware
Parts:
- removed U402: REF2033AIDDCT, Package_TO_SOT_SMD:SOT-23-5, symbol ETH1ISO224:REF19xxAIDDCT
- added U301: REF2033, Package_TO_SOT_SMD:SOT-23-5, symbol Reference_Voltage:REF2033
- Y401: footprint ETH1ISO224:NX5032GA -> (none)
Connections:
- net +3.3VADC: now also U301.5 (Vref)
- net +5V: now also U301.3 (EN), U301.4 (IN)
- net GND: now also U301.2 (GND)
Other:
- moved on the sheet: C402, C405

Commit message: Hardware
Parts:
- added C310, C311: 0.1u, Capacitor_SMD:C_0603_1608Metric_Pad1.08x0.95mm_HandSolder, symbol Device:C
- added R301: 51, Resistor_SMD:R_0603_1608Metric_Pad0.98x0.95mm_HandSolder, symbol Device:R
- added R303: 1k, Resistor_SMD:R_0603_1608Metric_Pad0.98x0.95mm_HandSolder, symbol Device:R
- added R304: 1k5, Resistor_SMD:R_0603_1608Metric_Pad0.98x0.95mm_HandSolder, symbol Device:R
- added U301: SN74LV1T34DBV, Package_TO_SOT_SMD:SOT-23-5, symbol Logic_LevelTranslator:SN74LV1T34DBV
- added U303: 74LVC1G74DP, Package_SO:TSSOP-8_3x3mm_P0.65mm, symbol ETH1LCR3:74LVC1G74DP
- renumbered U301 to U302
Connections:
- net +5V: now also C310.1, C311.1, U301.5 (VCC), U303.6 (~{CLR}), U303.7 (~{PRE}), U303.8 (VCC)
- net GND: now also C310.2, C311.2, R304.1, U301.3 (GND), U303.4 (GND)
- new net: R301.2, U301.2 (A)
- new net: U301.4 (Y), U303.2 (D)
- new net: R303.1, U303.5 (Q)
- new net: R303.2, R304.2
- new net PHI_OUT: U303.1 (CLK)
- no-connect marks 68 -> 69
Other:
- moved on the sheet: C414, C418, C421, FB401

Commit message: Hardware
Parts:
- removed C402, C406: 1u, Capacitor_SMD:C_0603_1608Metric_Pad1.08x0.95mm_HandSolder, symbol Device:C
- removed C403, C405: 0.1u, Capacitor_SMD:C_0603_1608Metric_Pad1.08x0.95mm_HandSolder, symbol Device:C
- added C302: 100n, symbol Device:C
- added C303, C306: 0.1u, Capacitor_SMD:C_0603_1608Metric_Pad1.08x0.95mm_HandSolder, symbol Device:C
- added C305: 1u, Capacitor_SMD:C_0603_1608Metric_Pad1.08x0.95mm_HandSolder, symbol Device:C
- added R309, R311: 100k, symbol Device:R
- added R310, R312: 110k, symbol Device:R
- added R313: 56k, symbol Device:R
- added R314: 160k, symbol Device:R
- added R315, R316: 0, symbol Device:R
- added R317: 3k, symbol Device:R
- added R318, R320: 2k, symbol Device:R
- added R319: 1k, symbol Device:R
- added R321: 3k6, symbol Device:R
- added R322: 1k6, symbol Device:R
- U302: now not fitted; now left out of the parts list
Connections:
- net +3.3VADC: now also R315.2; no longer U403.20 (VREF+)
- net +5V: now also C305.1, C306.1, R309.1, R311.1, R317.1
- net GND: now also C303.1, C305.2, C306.2, R318.2, R320.2, R322.2
- new net: C302.2, R311.2, R312.1
- new net +2V5: R313.1, R316.2
- new net +3V3: R319.1
- new net +3V3_ADC: R319.2, R320.1
- new net +5V_ADC: R317.2, R318.1
- new net -5V: R312.2, R314.2
- new net -5V_ADC: C303.2, R313.2, R314.1
- new net IV_ADC: C302.1, R309.2, R310.2
- new net I_VOLTAGE: R310.1
- new net VBOOST_ADC: R321.2, R322.1
- new net VREF+: R315.1, R316.1, U403.20 (VREF+)
- new net V_BOOST: R321.1
- no-connect marks 69 -> 70
Other:
- moved on the sheet: R301, R303, R304, U301, U303

Commit message: Hardware
Parts:
- C302: footprint (none) -> Capacitor_SMD:C_0603_1608Metric_Pad1.08x0.95mm_HandSolder
- R309, R310, R311, R312, R313, R314, R315, R316, R317, R318, R319, R320, R321, R322: footprint (none) -> Resistor_SMD:R_0603_1608Metric_Pad0.98x0.95mm_HandSolder
- renumbered C401 to C301, C404 to C304, C408 to C307, C410 to C308, C412 to C309, C414 to C312, C415 to C313, C416 to C314, C417 to C315, C419 to C316, C420 to C317, C418 to C318, C421 to C319, C422 to C320, D401 to D301, FB401 to FB301, J401 to J301, JP401 to JP301, R402 to R302, R405 to R305, R406 to R306, R407 to R307, R408 to R308, RN401 to RN301, U403 to U304, U404 to U305, Y401 to Y301
Other:
- moved on the sheet: R315, R316

Commit message: Software and hardware
Parts:
- removed R301: 51, Resistor_SMD:R_0603_1608Metric_Pad0.98x0.95mm_HandSolder, symbol Device:R
- removed R319: 1k, Resistor_SMD:R_0603_1608Metric_Pad0.98x0.95mm_HandSolder, symbol Device:R
- removed R320: 2k, Resistor_SMD:R_0603_1608Metric_Pad0.98x0.95mm_HandSolder, symbol Device:R
- added R303: 51, symbol Device:R
- added R311: 47, Resistor_SMD:R_0603_1608Metric_Pad0.98x0.95mm_HandSolder, symbol Device:R
- added R317, R318: 4k7, Resistor_SMD:R_0603_1608Metric_Pad0.98x0.95mm_HandSolder, symbol Device:R
- renumbered C304 to C302, C307 to C303, C308 to C304, C302 to C305, C309 to C306, C310 to C307, C303 to C308, C311 to C309, C314 to C310, C312 to C311, C313 to C312, C315 to C313, C316 to C314, C317 to C315, C318 to C316, C319 to C317, C305 to C318, C320 to C319, C306 to C320, R317 to R301, R318 to R302, R310 to R304, R309 to R305, R321 to R306, R322 to R307, R311 to R308, R312 to R309, R302 to R310, R313 to R312, R314 to R313, R303 to R314, R304 to R315, R305 to R316, R306 to R319, R315 to R320, R316 to R321, R307 to R322, R308 to R323, U303 to U302, U304 to U303, U305 to U304, U302 to U305
Connections:
- net +5V_ADC is gone; now on net ADC_+5V: R301.2, R302.1
- net -5V_ADC is gone; now on net ADC_-5V: C308.2, R312.2, R313.1
- net IV_ADC is gone; now on net ADC_IV_1: C305.1, R304.2, R305.2
- net VBOOST_ADC is gone; now on net ADC_VBOOST: R306.2, R307.1
- net +2V5: now also R311.1; no longer R312.1
- net ADS_DIN: now also U303.80 (PC12)
- net ADS_DOUT: now also U303.79 (PC11)
- net ADS_SCLK: now also U303.78 (PC10)
- net ADS_START: now also U303.82 (PD1)
- net ADS_~{CS}: now also U303.77 (PA15)
- net ADS_~{DRDY}: now also U303.81 (PD0)
- net CALIB_100: now also U303.83 (PD2)
- net CALIB_100K: now also U303.86 (PD5)
- net CALIB_10K: now also U303.85 (PD4)
- net CALIB_1K: now also U303.84 (PD3)
- net DAC0_OUT: now also U303.28 (PA4)
- net DAC1_OUT: now also U303.29 (PA5)
- net DC_BIAS_U-I: now also U303.3 (PE4)
- net DDS_RESET: now also U303.45 (PE15)
- net DDS_SCLK: now also U303.42 (PE12)
- net DDS_SDATA: now also U303.44 (PE14)
- net DDS_~{FSYNC1}: now also U303.40 (PE10)
- net DDS_~{FSYNC2}: now also U303.41 (PE11)
- net EN_BOOST: now also U303.54 (PB15)
- net FE_SW1: now also U303.57 (PD10)
- net FE_SW2: now also U303.58 (PD11)
- net FE_SW3: now also U303.59 (PD12)
- net FE_SW4: now also U303.60 (PD13)
- net FE_SW5: now also U303.61 (PD14)
- net FE_SW6: now also U303.62 (PD15)
- net FE_V_SHORT: now also U303.2 (PE3)
- net GND: now also R318.1
- net MAX_BOOST: now also U303.53 (PB14)
- net PGA_A0: now also U303.70 (PA11)
- net PGA_A1: now also U303.71 (PA12)
- net PGA_G1: now also U303.67 (PA8)
- net PGA_G10: now also U303.69 (PA10)
- net PGA_G3: now also U303.68 (PA9)
- net PSD_RC_A: now also U303.7 (PC13)
- net PSD_RC_B: now also U303.8 (PC14)
- net PSD_RC_C: now also U303.9 (PC15)
- net SELECT_RELAY: now also U303.4 (PE5)
- net TRIG_EN: now also U303.15 (PC0)
- net TRIG_IN: now also U303.18 (PC3_C)
- net TRIG_OUT: now also U303.17 (PC2_C)
- net VREF+: now also R317.2
- net ADC_IV_2: now reaches C305.2, R308.2, R309.1
- net ADC_IV_2: now also U303.35 (PB1)
- net at U301.2 (A): now also R303.2
- net SYNCH_OUT: now reaches R314.2, R315.2
- net SYNCH_OUT: now also U303.98 (PE1)
- net ADC_VBOOST: now reaches U303.22 (PA0)
- net ADC_+5V: now reaches U303.25 (PA3)
- net ADC_-5V: now reaches U303.30 (PA6)
- net ADC_IV_1: now reaches U303.34 (PB0)
- net at U303.37 (PE7): now also R317.1, R318.2
- net INPUT_COMP: now reaches U303.39 (PE9)
- net SYNCH_CDE: now reaches U303.97 (PE0)
- net SYNCH_CDE: now also R303.1
- new net: R311.2, R312.1
- no-connect marks 70 -> 22
Other:
- moved on the sheet: C305, C308, C310, C313, C314, C315, R301, R302, R304, R305, R306, R307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

Commit message: Hardware
Parts:
- added R324: 0, Resistor_SMD:R_0603_1608Metric_Pad0.98x0.95mm_HandSolder, symbol Device:R
Connections:
- net GND: now also R324.1
- net at R317.1, R318.2, U303.37 (PE7): now also R324.2
- net CXN_REL1: now reaches U303.87 (PD6)
- net CXN_REL2: now reaches U303.88 (PD7)
- net CXN_REL3: now reaches U303.89 (PB3)
- net CXN_REL4: now reaches U303.90 (PB4)
- net CXN_REL5: now reaches U303.95 (PB8)
- net CXN_REL6: now reaches U303.96 (PB9)
- no-connect marks 22 -> 16
Other:
- moved on the sheet: C305, C314, C315, R303, R304, R305, R308, R309, R314, R315, R317, R318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

Commit message: Hardware
Parts:
- R303: footprint (none) -> Resistor_SMD:R_0603_1608Metric_Pad0.98x0.95mm_HandSolder
- Y301: footprint (none) -> ETH1LCR3:NX5032GA
Changed lines of the file:
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@@
 			)
 		)
-		(property "Footprint" ""
+		(property "Footprint" "ETH1LCR3:NX5032GA"
 			(at 101.6 49.53 0)
 			(effects
@@
 			)
 		)
-		(property "Footprint" ""
+		(property "Footprint" "Resistor_SMD:R_0603_1608Metric_Pad0.98x0.95mm_HandSolder"
 			(at 30.48 90.678 90)
 			(effects
