File: Hardware/ETH1LCR3/MCU.kicad_sch (KiCad schematic)
At the start: 55 parts, among them J301 20021111-00010T4LF, U301 SN74LV1T34DBV, U302 74LVC1G74DP, U303 STM32H743VITx, U304 24LC08B-E/MS, U305 REF2033, Y301 NX5032GA-16

Commit message: PCB layout
Parts:
- JP301: now left out of the parts list
- U301: footprint Package_TO_SOT_SMD:SOT-23-5 -> Package_TO_SOT_SMD:SOT-23-5_HandSoldering
Changed lines of the file:
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@@
 			)
 		)
-		(property "Footprint" "Package_TO_SOT_SMD:SOT-23-5"
+		(property "Footprint" "Package_TO_SOT_SMD:SOT-23-5_HandSoldering"
 			(at 59.69 95.25 0)
 			(effects
@@
 		(unit 1)
 		(exclude_from_sim no)
-		(in_bom yes)
+		(in_bom no)
 		(on_board yes)
 		(dnp no)

Commit message: PCB layout
Parts:
- added C313: 0.1u, Capacitor_SMD:C_0603_1608Metric_Pad1.08x0.95mm_HandSolder, symbol Device:C
- renumbered C312 to C311, C313 to C312, C311 to C314, C314 to C315, C315 to C316, C316 to C317, C317 to C318, C318 to C319, C319 to C320, C320 to C321, R314 to R311, R311 to R312, R312 to R313, R313 to R314, R324 to R319, R319 to R320, R320 to R321, R321 to R322, R322 to R323, R323 to R324
Connections:
- net GND: now also C313.2
- net at R317.1, R318.2, R319.2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: now also C313.1
Other:
- moved on the sheet: C305, C314, C317, C318, FB301, R303, R304, R305, R308, R309, R311, R315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

Commit message: PCB layout
Parts:
- removed JP301: Open, Jumper:SolderJumper-2_P1.3mm_Open_Pad1.0x1.5mm, symbol Jumper:SolderJumper_2_Open
- added J302: Conn_01x02, Connector_PinHeader_2.54mm:PinHeader_1x02_P2.54mm_Vertical, symbol Connector_Generic:Conn_01x02
Connections:
- net DAC0_OUT: now also U303.29 (PA5); no longer U303.28 (PA4)
- net DAC1_OUT: now also U303.28 (PA4); no longer U303.29 (PA5)
- net GND: now also J302.2 (Pin_2)
- net MCU_DEF: now also J302.1 (Pin_1)
Other:
- moved on the sheet: R310
Changed lines of the file:
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@@
 	)
 	(junction
-		(at 68.58 29.21)
+		(at 71.12 29.21)
 		(diameter 0)
 		(color 0 0 0 0)
@@
 	(wire
 		(pts
-			(xy 68.58 30.48) (xy 68.58 29.21)
+			(xy 71.12 29.21) (xy 71.12 33.02)
 		)
 		(stroke
@@
 	(wire
 		(pts
-			(xy 80.01 29.21) (xy 68.58 29.21)
+			(xy 82.55 29.21) (xy 71.12 29.21)
 		)
 		(stroke
@@
 	(wire
 		(pts
-			(xy 68.58 38.1) (xy 68.58 39.37)
+			(xy 71.12 35.56) (xy 71.12 39.37)
 		)
 		(stroke
@@
 	(wire
 		(pts
-			(xy 68.58 29.21) (xy 68.58 27.94)
+			(xy 71.12 29.21) (xy 71.12 27.94)
 		)
 		(stroke
@@
 	)
 	(label "MCU_DEF"
-		(at 80.01 29.21 180)
+		(at 82.55 29.21 180)
 		(fields_autoplaced yes)
 		(effects
@@
 	(hierarchical_label "DAC1_OUT"
 		(shape output)
-		(at 189.23 41.91 0)
+		(at 189.23 39.37 0)
 		(fields_autoplaced yes)
 		(effects
@@
 	(hierarchical_label "DAC0_OUT"
 		(shape output)
-		(at 189.23 39.37 0)
+		(at 189.23 41.91 0)
 		(fields_autoplaced yes)
 		(effects
@@
 	)
 	(symbol
+		(lib_id "Connector_Generic:Conn_01x02")
+		(at 66.04 33.02 0)
+		(mirror y)
+		(unit 1)
+		(exclude_from_sim no)
+		(in_bom yes)
+		(on_board yes)
+		(dnp no)
+		(property "Reference" "J302"
+			(at 63.5 33.0199 0)
+			(effects
+				(font
+					(size 1.27 1.27)
+				)
+				(justify left)
+			)
+		)
+		(property "Value" "Conn_01x02"
+			(at 63.5 35.5599 0)
+			(effects
+				(font
+					(size 1.27 1.27)
+				)
+				(justify left)
+			)
+		)
+		(property "Footprint" "Connector_PinHeader_2.54mm:PinHeader_1x02_P2.54mm_Vertical"
+			(at 66.04 33.02 0)
+			(effects
+				(font
+					(size 1.27 1.27)
+				)
+				(hide yes)
+			)
+		)
+		(property "Datasheet" "~"
+			(at 66.04 33.02 0)
+			(effects
+				(font
+					(size 1.27 1.27)
+				)
+				(hide yes)
+			)
+		)
+		(property "Description" "Generic connector, single row, 01x02, script generated (kicad-library-utils/schlib/autogen/connector/)"
+			(at 66.04 33.02 0)
+			(effects
+				(font
+					(size 1.27 1.27)
+				)
+				(hide yes)
+			)
+		)
+		(pin "2"
+		)
+		(pin "1"
+		)
+		(instances
+			(project "ETH1LCR3"
+				(path "/6623bacb-57aa-43ce-9e51-b38a560dd9fc/6f6e1f41-595d-4dda-881d-b12a543de398"
+					(reference "J302")
+					(unit 1)
+				)
+			)
+		)
+	)
+	(symbol
 		(lib_id "Device:R")
 		(at 265.43 111.76 0)
@@
 	(symbol
 		(lib_id "power:+3.3V")
-		(at 68.58 20.32 0)
+		(at 71.12 20.32 0)
 		(unit 1)
 		(exclude_from_sim no)
@@
 		(fields_autoplaced yes)
 		(property "Reference" "#PWR0313"
-			(at 68.58 24.13 0)
+			(at 71.12 24.13 0)
 			(effects
 				(font
@@
 		)
 		(property "Value" "+3.3V"
-			(at 68.58 16.764 0)
+			(at 71.12 16.764 0)
 			(effects
 				(font
@@
 		)
 		(property "Footprint" ""
-			(at 68.58 20.32 0)
+			(at 71.12 20.32 0)
 			(effects
 				(font
@@
 		)
 		(property "Datasheet" ""
-			(at 68.58 20.32 0)
+			(at 71.12 20.32 0)
 			(effects
 				(font
@@
 		)
 		(property "Description" "Power symbol creates a global label with name \"+3.3V\""
-			(at 68.58 20.32 0)
+			(at 71.12 20.32 0)
 			(effects
 				(font
@@
 	(symbol
 		(lib_id "Device:R")
-		(at 68.58 24.13 0)
+		(at 71.12 24.13 0)
 		(mirror x)
 		(unit 1)
@@
 		(fields_autoplaced yes)
 		(property "Reference" "R310"
-			(at 66.802 22.9616 0)
+			(at 69.342 22.9616 0)
 			(effects
 				(font
@@
 		)
 		(property "Value" "10k"
-			(at 66.802 25.273 0)
+			(at 69.342 25.273 0)
 			(effects
 				(font
@@
 		)
 		(property "Footprint" "Resistor_SMD:R_0603_1608Metric_Pad0.98x0.95mm_HandSolder"
-			(at 66.802 24.13 90)
+			(at 69.342 24.13 90)
 			(effects
 				(font
@@
 		)
 		(property "Datasheet" "~"
-			(at 68.58 24.13 0)
+			(at 71.12 24.13 0)
 			(effects
 				(font
@@
 		)
 		(property "Description" ""
-			(at 68.58 24.13 0)
+			(at 71.12 24.13 0)
 			(effects
 				(font
@@
 	(symbol
 		(lib_id "power:GND")
-		(at 68.58 39.37 0)
+		(at 71.12 39.37 0)
 		(unit 1)
 		(exclude_from_sim no)
@@
 		(fields_autoplaced yes)
 		(property "Reference" "#PWR0314"
-			(at 68.58 45.72 0)
+			(at 71.12 45.72 0)
 			(effects
 				(font
@@
 		)
 		(property "Value" "GND"
-			(at 68.58 43.815 0)
+			(at 71.12 43.815 0)
 			(effects
 				(font
@@
 		)
 		(property "Footprint" ""
-			(at 68.58 39.37 0)
+			(at 71.12 39.37 0)
 			(effects
 				(font
@@
 		)
 		(property "Datasheet" ""
-			(at 68.58 39.37 0)
+			(at 71.12 39.37 0)
 			(effects
 				(font
@@
 		)
 		(property "Description" "Power symbol creates a global label with name \"GND\" , ground"
-			(at 68.58 39.37 0)
+			(at 71.12 39.37 0)
 			(effects
 				(font
@@
 					(unit 1)
 				)
-			)
-		)
-	)
-	(symbol
-		(lib_id "Jumper:SolderJumper_2_Open")
-		(at 68.58 34.29 90)
-		(mirror x)
-		(unit 1)
-		(exclude_from_sim no)
-		(in_bom no)
-		(on_board yes)
-		(dnp no)
-		(fields_autoplaced yes)
-		(property "Reference" "JP301"
-			(at 65.405 33.02 90)
-			(effects
-				(font
-					(size 1.27 1.27)
-				)
-				(justify left)
-			)
-		)
-		(property "Value" "Open"
-			(at 65.405 35.56 90)
-			(effects
-				(font
-					(size 1.27 1.27)
-				)
-				(justify left)
-			)
-		)
-		(property "Footprint" "Jumper:SolderJumper-2_P1.3mm_Open_Pad1.0x1.5mm"
-			(at 68.58 34.29 0)
-			(effects
-				(font
-					(size 1.27 1.27)
-				)
-				(hide yes)
-			)
-		)
-		(property "Datasheet" "~"
-			(at 68.58 34.29 0)
-			(effects
-				(font
-					(size 1.27 1.27)
-				)
-				(hide yes)
-			)
-		)
-		(property "Description" ""
-			(at 68.58 34.29 0)
-			(effects
-				(font
-					(size 1.27 1.27)
-				)
-				(hide yes)
-			)
-		)
-		(pin "1"
-		)
-		(pin "2"
-		)
-		(instances
-			(project ""
-				(path "/6623bacb-57aa-43ce-9e51-b38a560dd9fc/6f6e1f41-595d-4dda-881d-b12a543de398"
-					(reference "JP301")
-					(unit 1)
-				)

Commit message: PCB layout
Connections:
- net CXN_REL1: now also U303.96 (PB9); no longer U303.87 (PD6)
- net CXN_REL2: now also U303.95 (PB8); no longer U303.88 (PD7)
- net CXN_REL3: now also U303.90 (PB4); no longer U303.89 (PB3)
- net CXN_REL4: now also U303.87 (PD6); no longer U303.90 (PB4)
- net CXN_REL5: now also U303.88 (PD7); no longer U303.95 (PB8)
- net CXN_REL6: now also U303.89 (PB3); no longer U303.96 (PB9)
- net DC_BIAS_U-I: now also U303.55 (PD8); no longer U303.3 (PE4)
- net DDS_RESET: now also U303.98 (PE1); no longer U303.45 (PE15)
- net FE_SW5: now also U303.56 (PD9); no longer U303.61 (PD14)
- net FE_SW6: now also U303.2 (PE3); no longer U303.62 (PD15)
- net FE_V_SHORT: now also U303.3 (PE4); no longer U303.2 (PE3)
- net PGA_G10: now also U303.46 (PB10); no longer U303.69 (PA10)
- net SYNCH_CDE: now also U303.5 (PE6); no longer U303.97 (PE0)
- net SYNCH_OUT: now also U303.97 (PE0); no longer U303.98 (PE1)
- net TRIG_EN: now also U303.17 (PC2_C); no longer U303.15 (PC0)
- net TRIG_OUT: now also U303.15 (PC0); no longer U303.17 (PC2_C)
Changed lines of the file:
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@@
 	)
 	(no_connect
-		(at 144.78 115.57)
-	)
-	(no_connect
 		(at 80.01 118.11)
 	)
@@
 	)
 	(no_connect
-		(at 187.96 97.79)
-	)
-	(no_connect
-		(at 144.78 118.11)
+		(at 187.96 54.61)
 	)
 	(no_connect
@@
 	)
 	(no_connect
-		(at 144.78 67.31)
-	)
-	(no_connect
 		(at 30.48 41.91)
 	)
@@
 	)
 	(no_connect
+		(at 144.78 130.81)
+	)
+	(no_connect
 		(at 30.48 31.75)
 	)
 	(no_connect
+		(at 144.78 90.17)
+	)
+	(no_connect
 		(at 260.35 38.1)
 	)
 	(no_connect
+		(at 144.78 133.35)
+	)
+	(no_connect
 		(at 144.78 72.39)
 	)
@@
 	(wire
 		(pts
+			(xy 143.51 118.11) (xy 144.78 118.11)
+		)
+		(stroke
+			(width 0)
+			(type default)
+		)
+	)
+	(wire
+		(pts
 			(xy 187.96 49.53) (xy 189.23 49.53)
 		)
@@
 	(wire
 		(pts
+			(xy 143.51 62.23) (xy 144.78 62.23)
+		)
+		(stroke
+			(width 0)
+			(type default)
+		)
+	)
+	(wire
+		(pts
 			(xy 101.6 54.61) (xy 101.6 55.88)
 		)
@@
 	(wire
 		(pts
+			(xy 187.96 97.79) (xy 189.23 97.79)
+		)
+		(stroke
+			(width 0)
+			(type default)
+		)
+	)
+	(wire
+		(pts
 			(xy 236.22 109.22) (xy 240.03 109.22)
 		)
@@
 	(wire
 		(pts
-			(xy 133.35 54.61) (xy 144.78 54.61)
+			(xy 133.35 52.07) (xy 144.78 52.07)
 		)
 		(stroke
@@
 	(wire
 		(pts
-			(xy 187.96 54.61) (xy 189.23 54.61)
-		)
-		(stroke
-			(width 0)
-			(type default)
-		)
-	)
-	(wire
-		(pts
 			(xy 187.96 72.39) (xy 209.55 72.39)
 		)
@@
 	(wire
 		(pts
-			(xy 87.63 157.48) (xy 102.87 157.48)
+			(xy 143.51 115.57) (xy 144.78 115.57)
 		)
 		(stroke
@@
 	(wire
 		(pts
-			(xy 143.51 62.23) (xy 144.78 62.23)
+			(xy 87.63 157.48) (xy 102.87 157.48)
 		)
 		(stroke
@@
 	(wire
 		(pts
-			(xy 143.51 133.35) (xy 144.78 133.35)
+			(xy 187.96 90.17) (xy 214.63 90.17)
 		)
 		(stroke
@@
 	(wire
 		(pts
-			(xy 143.51 130.81) (xy 144.78 130.81)
-		)
-		(stroke
-			(width 0)
-			(type default)
-		)
-	)
-	(wire
-		(pts
 			(xy 143.51 77.47) (xy 144.78 77.47)
 		)
@@
 	(wire
 		(pts
-			(xy 187.96 87.63) (xy 209.55 87.63)
-		)
-		(stroke
-			(width 0)
-			(type default)
-		)
-	)
-	(wire
-		(pts
 			(xy 175.26 20.32) (xy 175.26 21.59)
 		)
@@
 	(wire
 		(pts
-			(xy 187.96 90.17) (xy 209.55 90.17)
-		)
-		(stroke
-			(width 0)
-			(type default)
-		)
-	)
-	(wire
-		(pts
 			(xy 143.51 74.93) (xy 144.78 74.93)
 		)
@@
 	(wire
 		(pts
-			(xy 143.51 90.17) (xy 144.78 90.17)
-		)
-		(stroke
-			(width 0)
-			(type default)
-		)
-	)
-	(wire
-		(pts
 			(xy 66.04 104.14) (xy 66.04 102.87)
 		)
@@
 	(wire
 		(pts
-			(xy 133.35 52.07) (xy 144.78 52.07)
+			(xy 132.08 67.31) (xy 144.78 67.31)
 		)
 		(stroke
@@
 	(wire
 		(pts
+			(xy 187.96 85.09) (xy 214.63 85.09)
+		)
+		(stroke
+			(width 0)
+			(type default)
+		)
+	)
+	(wire
+		(pts
 			(xy 101.6 45.72) (xy 101.6 44.45)
 		)
@@
 	(wire
 		(pts
+			(xy 187.96 87.63) (xy 214.63 87.63)
+		)
+		(stroke
+			(width 0)
+			(type default)
+		)
+	)
+	(wire
+		(pts
 			(xy 62.23 191.77) (xy 62.23 190.5)
 		)
@@
 	(wire
 		(pts
-			(xy 187.96 85.09) (xy 209.55 85.09)
+			(xy 34.29 113.03) (xy 35.56 113.03)
 		)
 		(stroke
@@
 	(wire
 		(pts
-			(xy 34.29 113.03) (xy 35.56 113.03)
+			(xy 59.69 74.93) (xy 59.69 73.66)
 		)
 		(stroke
@@
 	(wire
 		(pts
-			(xy 59.69 74.93) (xy 59.69 73.66)
+			(xy 254 60.96) (xy 256.54 60.96)
 		)
 		(stroke
@@
 	(wire
 		(pts
-			(xy 254 60.96) (xy 256.54 60.96)
+			(xy 143.51 54.61) (xy 144.78 54.61)
 		)
 		(stroke
@@
 	)
 	(label "I2C1_SDA"
-		(at 209.55 90.17 180)
+		(at 214.63 90.17 180)
 		(fields_autoplaced yes)
 		(effects
@@
 	)
 	(label "SYNCH_OUT"
-		(at 133.35 54.61 0)
+		(at 133.35 52.07 0)
 		(fields_autoplaced yes)
 		(effects
@@
 	)
 	(label "I2C1_SCL"
-		(at 209.55 87.63 180)
+		(at 214.63 87.63 180)
 		(fields_autoplaced yes)
 		(effects
@@
 	)
 	(label "EEPROM_nWP"
-		(at 209.55 85.09 180)
+		(at 214.63 85.09 180)
 		(fields_autoplaced yes)
 		(effects
@@
 	)
 	(label "SYNCH_CDE"
-		(at 133.35 52.07 0)
+		(at 132.08 67.31 0)
 		(fields_autoplaced yes)
 		(effects
@@
 	(hierarchical_label "CXN_REL5"
 		(shape output)
-		(at 189.23 92.71 0)
+		(at 143.51 113.03 180)
 		(fields_autoplaced yes)
 		(effects
@@
 				(size 1.27 1.27)
 			)
-			(justify left)
+			(justify right)
 		)
 	)
@@
 	(hierarchical_label "TRIG_OUT"
 		(shape output)
-		(at 189.23 120.65 0)
+		(at 189.23 115.57 0)
 		(fields_autoplaced yes)
 		(effects
@@
 	(hierarchical_label "TRIG_EN"
 		(shape output)
-		(at 189.23 115.57 0)
+		(at 189.23 120.65 0)
 		(fields_autoplaced yes)
 		(effects
@@
 	(hierarchical_label "FE_SW6"
 		(shape output)
-		(at 143.51 133.35 180)
+		(at 143.51 59.69 180)
 		(fields_autoplaced yes)
 		(effects
@@
 	(hierarchical_label "CXN_REL2"
 		(shape output)
-		(at 143.51 113.03 180)
+		(at 189.23 92.71 0)
 		(fields_autoplaced yes)
 		(effects
@@
 				(size 1.27 1.27)
 			)
-			(justify right)
+			(justify left)
 		)
 	)
@@
 	(hierarchical_label "PGA_G10"
 		(shape output)
-		(at 189.23 54.61 0)
+		(at 189.23 97.79 0)
 		(fields_autoplaced yes)
 		(effects
@@
 	(hierarchical_label "DC_BIAS_U-I"
 		(shape output)
-		(at 143.51 62.23 180)
+		(at 143.51 115.57 180)
 		(fields_autoplaced yes)
 		(effects
@@
 	(hierarchical_label "DDS_RESET"
 		(shape output)
-		(at 143.51 90.17 180)
+		(at 143.51 54.61 180)
 		(fields_autoplaced yes)
 		(effects
@@
 	(hierarchical_label "CXN_REL6"
 		(shape output)
-		(at 189.23 95.25 0)
+		(at 189.23 80.01 0)
 		(fields_autoplaced yes)
 		(effects
@@
 	(hierarchical_label "CXN_REL1"
 		(shape output)
-		(at 143.51 110.49 180)
+		(at 189.23 95.25 0)
 		(fields_autoplaced yes)
 		(effects
@@
 				(size 1.27 1.27)
 			)
-			(justify right)
+			(justify left)
 		)
 	)
@@
 	(hierarchical_label "CXN_REL3"
 		(shape output)
-		(at 189.23 80.01 0)
+		(at 189.23 82.55 0)
 		(fields_autoplaced yes)
 		(effects
@@
 	(hierarchical_label "CXN_REL4"
 		(shape output)
-		(at 189.23 82.55 0)
+		(at 143.51 110.49 180)
 		(fields_autoplaced yes)
 		(effects
@@
 				(size 1.27 1.27)
 			)
-			(justify left)
+			(justify right)
 		)
 	)
@@
 	(hierarchical_label "FE_SW5"
 		(shape output)
-		(at 143.51 130.81 180)
+		(at 143.51 118.11 180)
 		(fields_autoplaced yes)
 		(effects
@@
 	(hierarchical_label "FE_V_SHORT"
 		(shape output)
-		(at 143.51 59.69 180)
+		(at 143.51 62.23 180)
 		(fields_autoplaced yes)
 		(effects

Commit message: PCB layout
Connections:
- net ADS_DIN: now also U303.44 (PE14); no longer U303.80 (PC12)
- net ADS_DOUT: now also U303.43 (PE13); no longer U303.79 (PC11)
- net ADS_SCLK: now also U303.42 (PE12); no longer U303.78 (PC10)
- net ADS_START: now also U303.45 (PE15); no longer U303.82 (PD1)
- net ADS_~{CS}: now also U303.41 (PE11); no longer U303.77 (PA15)
- net ADS_~{DRDY}: now also U303.40 (PE10); no longer U303.81 (PD0)
- net DDS_SCLK: now also U303.78 (PC10); no longer U303.42 (PE12)
- net DDS_SDATA: now also U303.80 (PC12); no longer U303.44 (PE14)
- net DDS_~{FSYNC1}: now also U303.82 (PD1); no longer U303.40 (PE10)
- net DDS_~{FSYNC2}: now also U303.81 (PD0); no longer U303.41 (PE11)
Changed lines of the file:
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@@
 	)
 	(no_connect
-		(at 144.78 85.09)
-	)
-	(no_connect
 		(at 80.01 118.11)
 	)
@@
 	)
 	(no_connect
+		(at 187.96 67.31)
+	)
+	(no_connect
 		(at 30.48 41.91)
 	)
@@
 	)
 	(no_connect
-		(at 144.78 90.17)
+		(at 187.96 143.51)
 	)
 	(no_connect
@@
 	(wire
 		(pts
+			(xy 143.51 90.17) (xy 144.78 90.17)
+		)
+		(stroke
+			(width 0)
+			(type default)
+		)
+	)
+	(wire
+		(pts
 			(xy 250.19 25.4) (xy 250.19 26.67)
 		)
@@
 	(wire
 		(pts
-			(xy 187.96 67.31) (xy 189.23 67.31)
+			(xy 143.51 85.09) (xy 144.78 85.09)
 		)
 		(stroke
@@
 	(wire
 		(pts
-			(xy 187.96 143.51) (xy 189.23 143.51)
-		)
-		(stroke
-			(width 0)
-			(type default)
-		)
-	)
-	(wire
-		(pts
 			(xy 73.66 102.87) (xy 73.66 104.14)
 		)
@@
 	(hierarchical_label "ADS_~{DRDY}"
 		(shape input)
-		(at 143.51 95.25 180)
+		(at 143.51 77.47 180)
 		(fields_autoplaced yes)
 		(effects
@@
 	(hierarchical_label "DDS_SDATA"
 		(shape output)
-		(at 143.51 87.63 180)
+		(at 189.23 146.05 0)
 		(fields_autoplaced yes)
 		(effects
@@
 				(size 1.27 1.27)
 			)
-			(justify right)
+			(justify left)
 		)
 	)
@@
 	(hierarchical_label "ADS_START"
 		(shape output)
-		(at 143.51 97.79 180)
+		(at 143.51 90.17 180)
 		(fields_autoplaced yes)
 		(effects
@@
 	(hierarchical_label "DDS_~{FSYNC1}"
 		(shape output)
-		(at 143.51 77.47 180)
+		(at 143.51 97.79 180)
 		(fields_autoplaced yes)
 		(effects
@@
 	(hierarchical_label "ADS_~{CS}"
 		(shape output)
-		(at 189.23 67.31 0)
+		(at 143.51 80.01 180)
 		(fields_autoplaced yes)
 		(effects
@@
 				(size 1.27 1.27)
 			)
-			(justify left)
+			(justify right)
 		)
 	)
@@
 	(hierarchical_label "ADS_DIN"
 		(shape output)
-		(at 189.23 146.05 0)
+		(at 143.51 87.63 180)
 		(fields_autoplaced yes)
 		(effects
@@
 				(size 1.27 1.27)
 			)
-			(justify left)
+			(justify right)
 		)
 	)
@@
 	(hierarchical_label "ADS_DOUT"
 		(shape input)
-		(at 189.23 143.51 0)
+		(at 143.51 85.09 180)
 		(fields_autoplaced yes)
 		(effects
@@
 				(size 1.27 1.27)
 			)
-			(justify left)
+			(justify right)
 		)
 	)
@@
 	(hierarchical_label "DDS_~{FSYNC2}"
 		(shape output)
-		(at 143.51 80.01 180)
+		(at 143.51 95.25 180)
 		(fields_autoplaced yes)
 		(effects
@@
 	(hierarchical_label "DDS_SCLK"
 		(shape output)
-		(at 143.51 82.55 180)
+		(at 189.23 140.97 0)
 		(fields_autoplaced yes)
 		(effects
@@
 				(size 1.27 1.27)
 			)
-			(justify right)
+			(justify left)
 		)
 	)
@@
 	(hierarchical_label "ADS_SCLK"
 		(shape output)
-		(at 189.23 140.97 0)
+		(at 143.51 82.55 180)
 		(fields_autoplaced yes)
 		(effects
@@
 				(size 1.27 1.27)
 			)
-			(justify left)
+			(justify right)
 		)
 	)
