File: Hardware/ETH1LCR3/DDS.kicad_sch (KiCad schematic)
At the start: 60 parts, among them U501 AD9834, U502 AD9834, U503 LMH6644MT, U504 74LVC1G04, U505 SN74LV1T34DBV, U506 TLV3501AIDBV

Commit message: Schematic
Parts:
- removed R515, R519: 2k, symbol Device:R
- added RN501: MPMT2001AT, Package_TO_SOT_SMD:SOT-23, symbol Device:VoltageDivider_CenterPin3
- added U507: 74LVC1G74DP, symbol ETH1LCR3:74LVC1G74DP
- C501, C502, C503, C504, C505, C506, C507, C508, C509, C510, C511, C512, C513, C514, C515, C516, C517, C518, C519, C520: footprint (none) -> Capacitor_SMD:C_0603_1608Metric_Pad1.08x0.95mm_HandSolder
- R501, R502, R503, R504, R505, R506, R507, R508, R509, R510, R511, R512, R513, R514, R516, R517, R518, R520, R521, R522, R523, R524, R525, R526: footprint (none) -> Resistor_SMD:R_0603_1608Metric_Pad0.98x0.95mm_HandSolder
- U504: value 74LVC1G04 -> SN74LVC1G04DBV; footprint (none) -> Package_TO_SOT_SMD:SOT-23-5_HandSoldering
Connections:
- net +5VA is gone; now on net +5V: U505.5 (VCC)
- net DC_BIAS_VOLTAGE: now also RN501.1
- net GND: now also RN501.2, U507.4 (GND)
- net +5V: now reaches U506.4 (V+)
- net +5V: now also RV501.1, U507.7 (~{PRE}), U507.8 (VCC)
- net at U503.9 (-): now also RN501.3
- net at R525.2: now also U507.1 (CLK)
- net at U505.4 (Y): now also U507.6 (~{CLR})
- new net: U507.2 (D), U507.3 (~{Q})
- new net PHI_OUT: U507.5 (Q)
Other:
- moved on the sheet: C519, C520, R518, R523, R524, R525, R526, RV501, U503C, U503E, U505, U506

Commit message: Hardware
Parts:
- added C521, C522: 4u7, symbol Device:C
- added C523, C524, C525, C526, C527, C528: 100n, symbol Device:C
- added L507, L508: MLZ2012M100WT, symbol Device:L
- added X501: SG-5032CAN, Oscillator:Oscillator_SMD_SeikoEpson_SG8002LB-4Pin_5.0x3.2mm, symbol Oscillator:SG-5032CAN
Connections:
- net +5V: now also C525.1, C526.1, C527.1
- net 27MHz: now also X501.3 (OUT)
- net GND: now also C521.2, C522.2, C523.1, C524.1, C525.2, C526.2, C527.2, C528.2, X501.2 (GND)
- net -5V: now reaches U503.11 (V-)
- net -5V: now also C523.2
- net V_BOOST: now reaches U503.4 (V+)
- net V_BOOST: now also C524.2
- net AVDD_DDS: now reaches C511.1, C513.1, U502.4 (AVDD)
- net AVDD_DDS: now also C501.1, C502.1, U501.4 (AVDD), C521.1, L507.1
- net DVDD_DDS: now reaches C512.1, U502.5 (DVDD)
- net DVDD_DDS: now also C509.1, U501.5 (DVDD), U504.5 (VCC), C522.1, C528.1, L508.1, X501.4 (VCC)
- new net +3.3V: L507.2, L508.2
- no-connect marks 4 -> 5
Other:
- moved on the sheet: U503E, U507

Commit message: Hardware
Parts:
- C501: renamed from C528; value 100n -> 0.1u; footprint (none) -> Capacitor_SMD:C_0603_1608Metric_Pad1.08x0.95mm_HandSolder
- C520: renamed from C524; value 100n -> 0.1u; footprint (none) -> Capacitor_SMD:C_0603_1608Metric_Pad1.08x0.95mm_HandSolder
- C521: renamed from C523; value 100n -> 0.1u; footprint (none) -> Capacitor_SMD:C_0603_1608Metric_Pad1.08x0.95mm_HandSolder
- C526: renamed from C527; value 100n -> 0.1u; footprint (none) -> Capacitor_SMD:C_0603_1608Metric_Pad1.08x0.95mm_HandSolder
- C527: renamed from C525; value 100n -> 0.1u; footprint (none) -> Capacitor_SMD:C_0603_1608Metric_Pad1.08x0.95mm_HandSolder
- C528: renamed from C526; value 100n -> 0.1u; footprint (none) -> Capacitor_SMD:C_0603_1608Metric_Pad1.08x0.95mm_HandSolder
- L501, L502, L503, L504, L505, L506, L507, L508: footprint (none) -> Inductor_SMD:L_0805_2012Metric_Pad1.05x1.20mm_HandSolder
- U507: footprint (none) -> Package_SO:TSSOP-8_3x3mm_P0.65mm
- renumbered C508 to C502, C510 to C503, C501 to C504, C511 to C505, C515 to C506, C509 to C507, C502 to C508, C503 to C509, C512 to C510, C513 to C511, C514 to C512, C504 to C513, C505 to C514, C516 to C515, C517 to C516, C506 to C517, C507 to C518, C518 to C519, C519 to C522, C521 to C523, C520 to C524, C522 to C525, R516 to R504, R504 to R505, R505 to R506, R522 to R507, R520 to R508, R521 to R509, R506 to R510, R507 to R511, R510 to R512, R523 to R513, R524 to R514, R526 to R515, R508 to R516, R509 to R517, R511 to R518, R512 to R519, R513 to R520, R514 to R521, R525 to R522, R518 to R523, R517 to R524, U504 to U501, U501 to U502, U502 to U503, U505 to U504, U503 to U505

Commit message: Hardware
Connections:
- net RESET_DDS renamed DDS_RESET
Other:
- moved on the sheet: R503, U501, U504
Changed lines of the file:
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@@
 	)
 	(junction
+		(at 87.63 66.04)
+		(diameter 0)
+		(color 0 0 0 0)
+	)
+	(junction
 		(at 168.91 140.97)
 		(diameter 0)
@@
 	)
 	(junction
-		(at 72.39 177.8)
-		(diameter 0)
-		(color 0 0 0 0)
-	)
-	(junction
-		(at 87.63 69.85)
+		(at 73.66 177.8)
 		(diameter 0)
 		(color 0 0 0 0)
@@
 	(wire
 		(pts
-			(xy 96.52 69.85) (xy 97.79 69.85)
-		)
-		(stroke
-			(width 0)
-			(type default)
-		)
-	)
-	(wire
-		(pts
 			(xy 30.48 125.73) (xy 53.34 125.73)
 		)
@@
 	(wire
 		(pts
-			(xy 40.64 160.02) (xy 41.91 160.02)
-		)
-		(stroke
-			(width 0)
-			(type default)
-		)
-	)
-	(wire
-		(pts
 			(xy 114.3 130.81) (xy 125.73 130.81)
 		)
@@
 	(wire
 		(pts
-			(xy 68.58 177.8) (xy 72.39 177.8)
+			(xy 69.85 177.8) (xy 73.66 177.8)
 		)
 		(stroke
@@
 	(wire
 		(pts
-			(xy 72.39 177.8) (xy 83.82 177.8)
+			(xy 73.66 177.8) (xy 85.09 177.8)
 		)
 		(stroke
@@
 	(wire
 		(pts
-			(xy 87.63 69.85) (xy 88.9 69.85)
+			(xy 87.63 66.04) (xy 97.79 66.04)
 		)
 		(stroke
@@
 	(wire
 		(pts
-			(xy 40.64 160.02) (xy 40.64 177.8)
+			(xy 41.91 160.02) (xy 41.91 177.8)
 		)
 		(stroke
@@
 	(wire
 		(pts
-			(xy 72.39 177.8) (xy 72.39 194.31)
+			(xy 73.66 177.8) (xy 73.66 194.31)
 		)
 		(stroke
@@
 	(wire
 		(pts
-			(xy 97.79 90.17) (xy 147.32 90.17)
+			(xy 97.79 90.17) (xy 106.68 90.17)
 		)
 		(stroke
@@
 	(wire
 		(pts
-			(xy 40.64 194.31) (xy 72.39 194.31)
+			(xy 40.64 194.31) (xy 73.66 194.31)
 		)
 		(stroke
@@
 	(wire
 		(pts
-			(xy 87.63 59.69) (xy 87.63 69.85)
+			(xy 87.63 59.69) (xy 87.63 66.04)
 		)
 		(stroke
@@
 	(wire
 		(pts
+			(xy 114.3 90.17) (xy 147.32 90.17)
+		)
+		(stroke
+			(width 0)
+			(type default)
+		)
+	)
+	(wire
+		(pts
 			(xy 181.61 80.01) (xy 182.88 80.01)
 		)
@@
 	(wire
 		(pts
-			(xy 99.06 177.8) (xy 173.99 177.8)
+			(xy 100.33 177.8) (xy 173.99 177.8)
 		)
 		(stroke
@@
 	(wire
 		(pts
-			(xy 87.63 69.85) (xy 87.63 72.39)
+			(xy 87.63 66.04) (xy 87.63 72.39)
 		)
 		(stroke
@@
 	(wire
 		(pts
-			(xy 97.79 69.85) (xy 97.79 90.17)
+			(xy 97.79 66.04) (xy 97.79 90.17)
 		)
 		(stroke
@@
 		)
 	)
-	(hierarchical_label "RESET_DDS"
+	(hierarchical_label "DDS_RESET"
 		(shape input)
 		(at 40.64 194.31 180)
@@
 	(symbol
 		(lib_id "Logic_LevelTranslator:SN74LV1T34DBV")
-		(at 91.44 177.8 0)
+		(at 92.71 177.8 0)
 		(unit 1)
 		(exclude_from_sim no)
@@
 		(dnp no)
 		(property "Reference" "U504"
-			(at 105.41 172.466 0)
+			(at 106.68 172.466 0)
 			(effects
 				(font
@@
 		)
 		(property "Value" "SN74LV1T34DBV"
-			(at 105.41 175.006 0)
+			(at 106.68 175.006 0)
 			(effects
 				(font
@@
 		)
 		(property "Footprint" "Package_TO_SOT_SMD:SOT-23-5"
-			(at 107.95 184.15 0)
+			(at 109.22 184.15 0)
 			(effects
 				(font
@@
 		)
 		(property "Datasheet" "https://www.ti.com/lit/ds/symlink/sn74lv1t34.pdf"
-			(at 81.28 182.88 0)
+			(at 82.55 182.88 0)
 			(effects
 				(font
@@
 		)
 		(property "Description" "Single Power Supply, Single Buffer GATE, CMOS Logic, Level Shifter, SOT-23-5"
-			(at 91.44 177.8 0)
+			(at 92.71 177.8 0)
 			(effects
 				(font
@@
 	(symbol
 		(lib_id "power:GND")
-		(at 58.42 187.96 0)
+		(at 59.69 187.96 0)
 		(unit 1)
 		(exclude_from_sim no)
@@
 		(dnp no)
 		(property "Reference" "#PWR0510"
-			(at 58.42 194.31 0)
+			(at 59.69 194.31 0)
 			(effects
 				(font
@@
 		)
 		(property "Value" "GND"
-			(at 58.42 191.77 0)
+			(at 59.69 191.77 0)
 			(effects
 				(font
@@
 		)
 		(property "Footprint" ""
-			(at 58.42 187.96 0)
+			(at 59.69 187.96 0)
 			(effects
 				(font
@@
 		)
 		(property "Datasheet" ""
-			(at 58.42 187.96 0)
+			(at 59.69 187.96 0)
 			(effects
 				(font
@@
 		)
 		(property "Description" "Power symbol creates a global label with name \"GND\" , ground"
-			(at 58.42 187.96 0)
+			(at 59.69 187.96 0)
 			(effects
 				(font
@@
 	(symbol
 		(lib_id "power:+5V")
-		(at 91.44 170.18 0)
+		(at 92.71 170.18 0)
 		(unit 1)
 		(exclude_from_sim no)
@@
 		(fields_autoplaced yes)
 		(property "Reference" "#PWR0518"
-			(at 91.44 173.99 0)
+			(at 92.71 173.99 0)
 			(effects
 				(font
@@
 		)
 		(property "Value" "+5V"
-			(at 91.44 165.1 0)
+			(at 92.71 165.1 0)
 			(effects
 				(font
@@
 		)
 		(property "Footprint" ""
-			(at 91.44 170.18 0)
+			(at 92.71 170.18 0)
 			(effects
 				(font
@@
 		)
 		(property "Datasheet" ""
-			(at 91.44 170.18 0)
+			(at 92.71 170.18 0)
 			(effects
 				(font
@@
 		)
 		(property "Description" "Power symbol creates a global label with name \"+5V\""
-			(at 91.44 170.18 0)
+			(at 92.71 170.18 0)
 			(effects
 				(font
@@
 	(symbol
 		(lib_id "power:GND")
-		(at 91.44 185.42 0)
+		(at 92.71 185.42 0)
 		(unit 1)
 		(exclude_from_sim no)
@@
 		(dnp no)
 		(property "Reference" "#PWR0519"
-			(at 91.44 191.77 0)
+			(at 92.71 191.77 0)
 			(effects
 				(font
@@
 		)
 		(property "Value" "GND"
-			(at 91.44 189.23 0)
+			(at 92.71 189.23 0)
 			(effects
 				(font
@@
 		)
 		(property "Footprint" ""
-			(at 91.44 185.42 0)
+			(at 92.71 185.42 0)
 			(effects
 				(font
@@
 		)
 		(property "Datasheet" ""
-			(at 91.44 185.42 0)
+			(at 92.71 185.42 0)
 			(effects
 				(font
@@
 		)
 		(property "Description" "Power symbol creates a global label with name \"GND\" , ground"
-			(at 91.44 185.42 0)
+			(at 92.71 185.42 0)
 			(effects
 				(font
@@
 	(symbol
 		(lib_id "Device:R")
-		(at 92.71 69.85 270)
+		(at 110.49 90.17 270)
 		(unit 1)
 		(exclude_from_sim no)
@@
 		(dnp no)
 		(property "Reference" "R503"
-			(at 92.71 65.024 90)
+			(at 110.49 85.344 90)
 			(effects
 				(font
@@
 		)
 		(property "Value" "4k7"
-			(at 92.71 67.564 90)
+			(at 110.49 87.884 90)
 			(effects
 				(font
@@
 		)
 		(property "Footprint" "Resistor_SMD:R_0603_1608Metric_Pad0.98x0.95mm_HandSolder"
-			(at 92.71 68.072 90)
+			(at 110.49 88.392 90)
 			(effects
 				(font
@@
 		)
 		(property "Datasheet" "~"
-			(at 92.71 69.85 0)
+			(at 110.49 90.17 0)
 			(effects
 				(font
@@
 		)
 		(property "Description" "Resistor"
-			(at 92.71 69.85 0)
+			(at 110.49 90.17 0)
 			(effects
 				(font
@@
 	(symbol
 		(lib_id "74xGxx:74LVC1G04")
-		(at 53.34 177.8 0)
+		(at 54.61 177.8 0)
 		(mirror y)
 		(unit 1)
@@
 		(fields_autoplaced yes)
 		(property "Reference" "U501"
-			(at 71.12 171.4814 0)
+			(at 72.39 171.4814 0)
 			(effects
 				(font
@@
 		)
 		(property "Value" "SN74LVC1G04DBV"
-			(at 71.12 174.0214 0)
+			(at 72.39 174.0214 0)
 			(effects
 				(font
@@
 		)
 		(property "Footprint" "Package_TO_SOT_SMD:SOT-23-5_HandSoldering"
-			(at 53.34 177.8 0)
+			(at 54.61 177.8 0)
 			(effects
 				(font
@@
 		)
 		(property "Datasheet" "https://www.ti.com/lit/ds/symlink/sn74lvc1g04.pdf"
-			(at 53.34 177.8 0)
+			(at 54.61 177.8 0)
 			(effects
 				(font
@@
 		)
 		(property "Description" "Single NOT Gate, Low-Voltage CMOS"
-			(at 53.34 177.8 0)
+			(at 54.61 177.8 0)
 			(effects
 				(font
@@
 	(symbol
 		(lib_id "ETH1LCR3:DVDD_DDS")
-		(at 58.42 167.64 0)
+		(at 59.69 167.64 0)
 		(unit 1)
 		(exclude_from_sim no)
@@
 		(fields_autoplaced yes)
 		(property "Reference" "#PWR0509"
-			(at 58.42 171.45 0)
+			(at 59.69 171.45 0)
 			(effects
 				(font
@@
 		)
 		(property "Value" "DVDD_DDS"
-			(at 58.42 162.56 0)
+			(at 59.69 162.56 0)
 			(effects
 				(font
@@
 		)
 		(property "Footprint" ""
-			(at 58.42 167.64 0)
+			(at 59.69 167.64 0)
 			(effects
 				(font
@@
 		)
 		(property "Datasheet" ""
-			(at 58.42 167.64 0)
+			(at 59.69 167.64 0)
 			(effects
 				(font
@@
 		)
 		(property "Description" ""
-			(at 58.42 167.64 0)
+			(at 59.69 167.64 0)
 			(effects
 				(font

Commit message: Software and hardware
Parts:
- renumbered C520 to C517, C521 to C518, C517 to C519, C518 to C520, C519 to C521, R504 to R503, R505 to R504, R506 to R505, R503 to R506
Other:
- moved on the sheet: C517, C518, C523, L507, U505E

Commit message: Hardware
Connections:
- net -5VA is gone; now on net -5V: RV501.3
Other:
- moved on the sheet: C523, C525, L507, L508

Commit message: Hardware
Parts:
- C523, C525: footprint (none) -> Capacitor_SMD:C_0805_2012Metric_Pad1.18x1.45mm_HandSolder
- RV501: value 10k -> TS53YJ103MR10; footprint (none) -> Potentiometer_SMD:Potentiometer_Vishay_TS53YJ_Vertical
Other:
- moved on the sheet: R523, R524, RV501
Changed lines of the file:
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@@
 	)
 	(junction
-		(at 254 62.23)
+		(at 259.08 62.23)
 		(diameter 0)
 		(color 0 0 0 0)
@@
 	(wire
 		(pts
-			(xy 254 62.23) (xy 255.27 62.23)
+			(xy 259.08 62.23) (xy 260.35 62.23)
 		)
 		(stroke
@@
 	(wire
 		(pts
-			(xy 254 62.23) (xy 254 63.5)
+			(xy 259.08 62.23) (xy 259.08 63.5)
 		)
 		(stroke
@@
 	(wire
 		(pts
-			(xy 213.36 54.61) (xy 264.16 54.61)
+			(xy 213.36 54.61) (xy 269.24 54.61)
 		)
 		(stroke
@@
 	(wire
 		(pts
-			(xy 234.95 62.23) (xy 254 62.23)
+			(xy 234.95 62.23) (xy 259.08 62.23)
 		)
 		(stroke
@@
 	(wire
 		(pts
-			(xy 262.89 62.23) (xy 264.16 62.23)
+			(xy 267.97 62.23) (xy 269.24 62.23)
 		)
 		(stroke
@@
 	(hierarchical_label "DAC0_OUT"
 		(shape input)
-		(at 264.16 62.23 0)
+		(at 269.24 62.23 0)
 		(fields_autoplaced yes)
 		(effects
@@
 	(hierarchical_label "SINE"
 		(shape output)
-		(at 264.16 54.61 0)
+		(at 269.24 54.61 0)
 		(fields_autoplaced yes)
 		(effects
@@
 	(symbol
 		(lib_id "Device:R")
-		(at 254 67.31 0)
+		(at 259.08 67.31 0)
 		(unit 1)
 		(exclude_from_sim no)
@@
 		(fields_autoplaced yes)
 		(property "Reference" "R523"
-			(at 256.54 66.0399 0)
+			(at 261.62 66.0399 0)
 			(effects
 				(font
@@
 		)
 		(property "Value" "100k"
-			(at 256.54 68.5799 0)
+			(at 261.62 68.5799 0)
 			(effects
 				(font
@@
 		)
 		(property "Footprint" "Resistor_SMD:R_0603_1608Metric_Pad0.98x0.95mm_HandSolder"
-			(at 252.222 67.31 90)
+			(at 257.302 67.31 90)
 			(effects
 				(font
@@
 		)
 		(property "Datasheet" "~"
-			(at 254 67.31 0)
+			(at 259.08 67.31 0)
 			(effects
 				(font
@@
 		)
 		(property "Description" "Resistor"
-			(at 254 67.31 0)
+			(at 259.08 67.31 0)
 			(effects
 				(font
@@
 	(symbol
 		(lib_id "Device:R_Potentiometer_Trim")
-		(at 254 74.93 90)
+		(at 259.08 74.93 90)
 		(unit 1)
 		(exclude_from_sim no)
@@
 		(fields_autoplaced yes)
 		(property "Reference" "RV501"
-			(at 254 78.74 90)
+			(at 259.08 78.74 90)
 			(effects
 				(font
@@
 			)
 		)
-		(property "Value" "10k"
-			(at 254 81.28 90)
+		(property "Value" "TS53YJ103MR10"
+			(at 259.08 81.28 90)
 			(effects
 				(font
@@
 			)
 		)
-		(property "Footprint" ""
-			(at 254 74.93 0)
+		(property "Footprint" "Potentiometer_SMD:Potentiometer_Vishay_TS53YJ_Vertical"
+			(at 259.08 74.93 0)
 			(effects
 				(font
@@
 		)
 		(property "Datasheet" "~"
-			(at 254 74.93 0)
+			(at 259.08 74.93 0)
 			(effects
 				(font
@@
 		)
 		(property "Description" "Trim-potentiometer"
-			(at 254 74.93 0)
+			(at 259.08 74.93 0)
 			(effects
 				(font
@@
 			)
 		)
-		(property "Footprint" ""
+		(property "Footprint" "Capacitor_SMD:C_0805_2012Metric_Pad1.18x1.45mm_HandSolder"
 			(at 223.2152 29.21 0)
 			(effects
@@
 	(symbol
 		(lib_id "Device:R")
-		(at 259.08 62.23 90)
+		(at 264.16 62.23 90)
 		(unit 1)
 		(exclude_from_sim no)
@@
 		(dnp no)
 		(property "Reference" "R524"
-			(at 259.08 57.404 90)
+			(at 264.16 57.404 90)
 			(effects
 				(font
@@
 		)
 		(property "Value" "300"
-			(at 259.08 59.944 90)
+			(at 264.16 59.944 90)
 			(effects
 				(font
@@
 		)
 		(property "Footprint" "Resistor_SMD:R_0603_1608Metric_Pad0.98x0.95mm_HandSolder"
-			(at 259.08 64.008 90)
+			(at 264.16 64.008 90)
 			(effects
 				(font
@@
 		)
 		(property "Datasheet" "~"
-			(at 259.08 62.23 0)
+			(at 264.16 62.23 0)
 			(effects
 				(font
@@
 		)
 		(property "Description" "Resistor"
-			(at 259.08 62.23 0)
+			(at 264.16 62.23 0)
 			(effects
 				(font
@@
 	(symbol
 		(lib_id "power:+5V")
-		(at 250.19 74.93 90)
+		(at 255.27 74.93 90)
 		(unit 1)
 		(exclude_from_sim no)
@@
 		(dnp no)
 		(property "Reference" "#PWR0545"
-			(at 254 74.93 0)
+			(at 259.08 74.93 0)
 			(effects
 				(font
@@
 		)
 		(property "Value" "+5V"
-			(at 246.38 74.9301 90)
+			(at 251.46 74.9301 90)
 			(effects
 				(font
@@
 		)
 		(property "Footprint" ""
-			(at 250.19 74.93 0)
+			(at 255.27 74.93 0)
 			(effects
 				(font
@@
 		)
 		(property "Datasheet" ""
-			(at 250.19 74.93 0)
+			(at 255.27 74.93 0)
 			(effects
 				(font
@@
 		)
 		(property "Description" "Power symbol creates a global label with name \"+5V\""
-			(at 250.19 74.93 0)
+			(at 255.27 74.93 0)
 			(effects
 				(font
@@
 			)
 		)
-		(property "Footprint" ""
+		(property "Footprint" "Capacitor_SMD:C_0805_2012Metric_Pad1.18x1.45mm_HandSolder"
 			(at 181.3052 29.21 0)
 			(effects
@@
 	(symbol
 		(lib_id "power:-5V")
-		(at 257.81 74.93 270)
+		(at 262.89 74.93 270)
 		(unit 1)
 		(exclude_from_sim no)
@@
 		(fields_autoplaced yes)
 		(property "Reference" "#PWR0549"
-			(at 254 74.93 0)
+			(at 259.08 74.93 0)
 			(effects
 				(font
@@
 		)
 		(property "Value" "-5V"
-			(at 261.62 74.9299 90)
+			(at 266.7 74.9299 90)
 			(effects
 				(font
@@
 		)
 		(property "Footprint" ""
-			(at 257.81 74.93 0)
+			(at 262.89 74.93 0)
 			(effects
 				(font
@@
 		)
 		(property "Datasheet" ""
-			(at 257.81 74.93 0)
+			(at 262.89 74.93 0)
 			(effects
 				(font
@@
 		)
 		(property "Description" "Power symbol creates a global label with name \"-5V\""
-			(at 257.81 74.93 0)
+			(at 262.89 74.93 0)
 			(effects
 				(font

Commit message: PCB layout
Parts:
- U504: footprint Package_TO_SOT_SMD:SOT-23-5 -> Package_TO_SOT_SMD:SOT-23-5_HandSoldering
- U506: footprint Package_TO_SOT_SMD:SOT-23-6 -> Package_TO_SOT_SMD:SOT-23-6_Handsoldering
Changed lines of the file:
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@@
 			)
 		)
-		(property "Footprint" "Package_TO_SOT_SMD:SOT-23-6"
+		(property "Footprint" "Package_TO_SOT_SMD:SOT-23-6_Handsoldering"
 			(at 190.5 135.255 0)
 			(effects
@@
 			)
 		)
-		(property "Footprint" "Package_TO_SOT_SMD:SOT-23-5"
+		(property "Footprint" "Package_TO_SOT_SMD:SOT-23-5_HandSoldering"
 			(at 109.22 184.15 0)
 			(effects
