File: Hardware/ETH1LCR3/DDS.kicad_sch (KiCad schematic)
At the start: 71 parts, among them U501 SN74LVC1G04DBV, U502 AD9834, U503 AD9834, U504 SN74LV1T34DBV, U505 LMH6644MT, U506 TLV3501AIDBV, U507 74LVC1G74DP, X501 SG-5032CAN

Commit message: PCB layout
Parts:
- renumbered C524 to C523, C523 to C524
Changed lines of the file:
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@@
 		(dnp no)
 		(fields_autoplaced yes)
-		(property "Reference" "#PWR0540"
+		(property "Reference" "#PWR0542"
 			(at 222.25 36.83 0)
 			(effects
@@
 			(project "ETH1LCR3"
 				(path "/6623bacb-57aa-43ce-9e51-b38a560dd9fc/69949141-78d8-43de-bf63-b55bbbab5791"
-					(reference "#PWR0540")
+					(reference "#PWR0542")
 					(unit 1)
 				)
@@
 		(on_board yes)
 		(dnp no)
-		(property "Reference" "#PWR0544"
+		(property "Reference" "#PWR0546"
 			(at 243.84 138.43 0)
 			(effects
@@
 			(project "ETH1LCR3"
 				(path "/6623bacb-57aa-43ce-9e51-b38a560dd9fc/69949141-78d8-43de-bf63-b55bbbab5791"
-					(reference "#PWR0544")
+					(reference "#PWR0546")
 					(unit 1)
 				)
@@
 		(dnp no)
 		(fields_autoplaced yes)
-		(property "Reference" "#PWR0533"
+		(property "Reference" "#PWR0535"
 			(at 180.34 20.32 0)
 			(effects
@@
 			(project ""
 				(path "/6623bacb-57aa-43ce-9e51-b38a560dd9fc/69949141-78d8-43de-bf63-b55bbbab5791"
-					(reference "#PWR0533")
+					(reference "#PWR0535")
 					(unit 1)
 				)
@@
 		(dnp no)
 		(fields_autoplaced yes)
-		(property "Reference" "#PWR0539"
+		(property "Reference" "#PWR0541"
 			(at 222.25 20.32 0)
 			(effects
@@
 			(project ""
 				(path "/6623bacb-57aa-43ce-9e51-b38a560dd9fc/69949141-78d8-43de-bf63-b55bbbab5791"
-					(reference "#PWR0539")
+					(reference "#PWR0541")
 					(unit 1)
 				)
@@
 		(on_board yes)
 		(dnp no)
-		(property "Reference" "#PWR0545"
+		(property "Reference" "#PWR0547"
 			(at 259.08 74.93 0)
 			(effects
@@
 			(project "ETH1LCR3"
 				(path "/6623bacb-57aa-43ce-9e51-b38a560dd9fc/69949141-78d8-43de-bf63-b55bbbab5791"
-					(reference "#PWR0545")
+					(reference "#PWR0547")
 					(unit 1)
 				)
@@
 		(on_board yes)
 		(dnp no)
-		(property "Reference" "#PWR0536"
+		(property "Reference" "#PWR0537"
 			(at 187.96 121.92 0)
 			(effects
@@
 			(project ""
 				(path "/6623bacb-57aa-43ce-9e51-b38a560dd9fc/69949141-78d8-43de-bf63-b55bbbab5791"
-					(reference "#PWR0536")
+					(reference "#PWR0537")
 					(unit 1)
 				)
@@
 		(on_board yes)
 		(dnp no)
-		(property "Reference" "#PWR0543"
+		(property "Reference" "#PWR0545"
 			(at 240.03 107.95 0)
 			(effects
@@
 			(project "ETH1LCR3"
 				(path "/6623bacb-57aa-43ce-9e51-b38a560dd9fc/69949141-78d8-43de-bf63-b55bbbab5791"
-					(reference "#PWR0543")
+					(reference "#PWR0545")
 					(unit 1)
 				)
@@
 		(dnp no)
 		(fields_autoplaced yes)
-		(property "Reference" "#PWR0537"
+		(property "Reference" "#PWR0539"
 			(at 187.96 20.32 0)
 			(effects
@@
 			(project ""
 				(path "/6623bacb-57aa-43ce-9e51-b38a560dd9fc/69949141-78d8-43de-bf63-b55bbbab5791"
-					(reference "#PWR0537")
+					(reference "#PWR0539")
 					(unit 1)
 				)
@@
 		(on_board yes)
 		(dnp no)
-		(property "Reference" "#PWR0547"
+		(property "Reference" "#PWR0548"
 			(at 261.62 22.86 0)
 			(effects
@@
 			(project "ETH1LCR3"
 				(path "/6623bacb-57aa-43ce-9e51-b38a560dd9fc/69949141-78d8-43de-bf63-b55bbbab5791"
-					(reference "#PWR0547")
+					(reference "#PWR0548")
 					(unit 1)
 				)
@@
 		(dnp no)
 		(fields_autoplaced yes)
-		(property "Reference" "#PWR0550"
+		(property "Reference" "#PWR0533"
 			(at 167.64 33.02 0)
 			(effects
@@
 			(project "ETH1LCR3"
 				(path "/6623bacb-57aa-43ce-9e51-b38a560dd9fc/69949141-78d8-43de-bf63-b55bbbab5791"
-					(reference "#PWR0550")
+					(reference "#PWR0533")
 					(unit 1)
 				)
@@
 		(dnp no)
 		(fields_autoplaced yes)
-		(property "Reference" "C523"
+		(property "Reference" "C524"
 			(at 184.15 24.1299 0)
 			(effects
@@
 			(project ""
 				(path "/6623bacb-57aa-43ce-9e51-b38a560dd9fc/69949141-78d8-43de-bf63-b55bbbab5791"
-					(reference "C523")
+					(reference "C524")
 					(unit 1)
 				)
@@
 		(on_board yes)
 		(dnp no)
-		(property "Reference" "#PWR0548"
+		(property "Reference" "#PWR0549"
 			(at 261.62 38.1 0)
 			(effects
@@
 			(project "ETH1LCR3"
 				(path "/6623bacb-57aa-43ce-9e51-b38a560dd9fc/69949141-78d8-43de-bf63-b55bbbab5791"
-					(reference "#PWR0548")
+					(reference "#PWR0549")
 					(unit 1)
 				)
@@
 		(dnp no)
 		(fields_autoplaced yes)
-		(property "Reference" "#PWR0541"
+		(property "Reference" "#PWR0543"
 			(at 229.87 20.32 0)
 			(effects
@@
 			(project "ETH1LCR3"
 				(path "/6623bacb-57aa-43ce-9e51-b38a560dd9fc/69949141-78d8-43de-bf63-b55bbbab5791"
-					(reference "#PWR0541")
+					(reference "#PWR0543")
 					(unit 1)
 				)
@@
 		(on_board yes)
 		(dnp no)
-		(property "Reference" "#PWR0546"
+		(property "Reference" "#PWR0540"
 			(at 209.55 33.02 0)
 			(effects
@@
 			(project "ETH1LCR3"
 				(path "/6623bacb-57aa-43ce-9e51-b38a560dd9fc/69949141-78d8-43de-bf63-b55bbbab5791"
-					(reference "#PWR0546")
+					(reference "#PWR0540")
 					(unit 1)
 				)
@@
 		(dnp no)
 		(fields_autoplaced yes)
-		(property "Reference" "#PWR0549"
+		(property "Reference" "#PWR0550"
 			(at 259.08 74.93 0)
 			(effects
@@
 			(project ""
 				(path "/6623bacb-57aa-43ce-9e51-b38a560dd9fc/69949141-78d8-43de-bf63-b55bbbab5791"
-					(reference "#PWR0549")
+					(reference "#PWR0550")
 					(unit 1)
 				)
@@
 		(on_board yes)
 		(dnp no)
-		(property "Reference" "C524"
+		(property "Reference" "C523"
 			(at 176.53 104.902 90)
 			(effects
@@
 			(project ""
 				(path "/6623bacb-57aa-43ce-9e51-b38a560dd9fc/69949141-78d8-43de-bf63-b55bbbab5791"
-					(reference "C524")
+					(reference "C523")
 					(unit 1)
 				)
@@
 		(dnp no)
 		(fields_autoplaced yes)
-		(property "Reference" "#PWR0535"
+		(property "Reference" "#PWR0536"
 			(at 180.34 36.83 0)
 			(effects
@@
 			(project ""
 				(path "/6623bacb-57aa-43ce-9e51-b38a560dd9fc/69949141-78d8-43de-bf63-b55bbbab5791"
-					(reference "#PWR0535")
+					(reference "#PWR0536")
 					(unit 1)
 				)
@@
 		(on_board yes)
 		(dnp no)
-		(property "Reference" "#PWR0542"
+		(property "Reference" "#PWR0544"
 			(at 246.38 80.01 0)
 			(effects
@@
 			(project "ETH1LCR3"
 				(path "/6623bacb-57aa-43ce-9e51-b38a560dd9fc/69949141-78d8-43de-bf63-b55bbbab5791"
-					(reference "#PWR0542")
+					(reference "#PWR0544")
 					(unit 1)
 				)

Commit message: PCB layout
Parts:
- RV501: value TS53YJ103MR10 -> 3266W-1-103LF; footprint Potentiometer_SMD:Potentiometer_Vishay_TS53YJ_Vertical -> Potentiometer_THT:Potentiometer_Bourns_3266W_Vertical
Changed lines of the file:
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@@
 			)
 		)
-		(property "Value" "TS53YJ103MR10"
+		(property "Value" "3266W-1-103LF"
 			(at 259.08 81.28 90)
 			(effects
@@
 			)
 		)
-		(property "Footprint" "Potentiometer_SMD:Potentiometer_Vishay_TS53YJ_Vertical"
+		(property "Footprint" "Potentiometer_THT:Potentiometer_Bourns_3266W_Vertical"
 			(at 259.08 74.93 0)
 			(effects

Commit message: Updated project to KiCAD 9
Changed lines of the file:
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@@
 (kicad_sch
-	(version 20231120)
+	(version 20250114)
 	(generator "eeschema")
-	(generator_version "8.0")
+	(generator_version "9.0")
 	(paper "A4")
 	(junction
@@
 	(label "27MHz"
 		(at 46.99 63.5 0)
-		(fields_autoplaced yes)
 		(effects
 			(font
@@
 		(shape input)
 		(at 30.48 48.26 180)
-		(fields_autoplaced yes)
 		(effects
 			(font
@@
 		(shape output)
 		(at 261.62 120.65 0)
-		(fields_autoplaced yes)
 		(effects
 			(font
@@
 		(shape output)
 		(at 264.16 46.99 0)
-		(fields_autoplaced yes)
 		(effects
 			(font
@@
 		(shape input)
 		(at 40.64 194.31 180)
-		(fields_autoplaced yes)
 		(effects
 			(font
@@
 		(shape input)
 		(at 30.48 43.18 180)
-		(fields_autoplaced yes)
 		(effects
 			(font
@@
 		(shape input)
 		(at 269.24 62.23 0)
-		(fields_autoplaced yes)
 		(effects
 			(font
@@
 		(shape output)
 		(at 269.24 54.61 0)
-		(fields_autoplaced yes)
 		(effects
 			(font
@@
 		(shape input)
 		(at 30.48 125.73 180)
-		(fields_autoplaced yes)
 		(effects
 			(font
@@
 		(shape input)
 		(at 147.32 90.17 0)
-		(fields_autoplaced yes)
 		(effects
 			(font
@@
 		(shape input)
 		(at 30.48 45.72 180)
-		(fields_autoplaced yes)
 		(effects
 			(font
