File: Hardware/ETH1LCR3/PSD.kicad_sch (KiCad schematic)
At the start: 12 parts, among them U701 SN74LVC1G3157DB, U702 SN74LVC1G3157DB, U703 SN74LV1T34DBV, U704 SN74LV1T34DBV, U705 SN74LV1T34DBV, U706 TLV3501AIDBV

Commit message: Hardware
Parts:
- added C701, C719: 1u, Capacitor_SMD:C_0603_1608Metric_Pad1.08x0.95mm_HandSolder, symbol Device:C
- added C702, C704, C705, C706, C708, C709, C710, C711, C712, C713, C714, C720: 0.1u, Capacitor_SMD:C_0603_1608Metric_Pad1.08x0.95mm_HandSolder, symbol Device:C
- added C703: 22p, Capacitor_SMD:C_0603_1608Metric_Pad1.08x0.95mm_HandSolder, symbol Device:C
- added C707: 100p, Capacitor_SMD:C_0603_1608Metric_Pad1.08x0.95mm_HandSolder, symbol Device:C
- added C715, C716: 15p/C0G, symbol Device:C
- added C717, C718, C721: 4u7, symbol Device:C
- added C722, C723, C724, C725: 100n/C0G, symbol Device:C
- added D701, D702, D703: NSVRB751V40T1G, symbol Device:D
- added L701: MLZ1608DR47DT, Inductor_SMD:L_0603_1608Metric_Pad1.05x0.95mm_HandSolder, symbol Device:L
- added R701: 30/.1%, Resistor_SMD:R_0603_1608Metric_Pad0.98x0.95mm_HandSolder, symbol Device:R
- added R704: 1k5, Resistor_SMD:R_0603_1608Metric_Pad0.98x0.95mm_HandSolder, symbol Device:R
- added R707: 2k, Resistor_SMD:R_0603_1608Metric_Pad0.98x0.95mm_HandSolder, symbol Device:R
- added R708: 10/.1%, Resistor_SMD:R_0603_1608Metric_Pad0.98x0.95mm_HandSolder, symbol Device:R
- added R709: 51/.1%, Resistor_SMD:R_0603_1608Metric_Pad0.98x0.95mm_HandSolder, symbol Device:R
- added R710: 240/.1%, Resistor_SMD:R_0603_1608Metric_Pad0.98x0.95mm_HandSolder, symbol Device:R
- added R711: 1k/.1%, Resistor_SMD:R_0603_1608Metric_Pad0.98x0.95mm_HandSolder, symbol Device:R
- added R712: 5k1/.1%, Resistor_SMD:R_0603_1608Metric_Pad0.98x0.95mm_HandSolder, symbol Device:R
- added R713: 20k/.1%, Resistor_SMD:R_0603_1608Metric_Pad0.98x0.95mm_HandSolder, symbol Device:R
- added R714: 51k/.1%, Resistor_SMD:R_0603_1608Metric_Pad0.98x0.95mm_HandSolder, symbol Device:R
- added R715: 75k/.1%, Resistor_SMD:R_0603_1608Metric_Pad0.98x0.95mm_HandSolder, symbol Device:R
- added R716, R717: 1k6/.1%, Resistor_SMD:R_0603_1608Metric_Pad0.98x0.95mm_HandSolder, symbol Device:R
- added R724, R725: 3k, Resistor_SMD:R_0603_1608Metric_Pad0.98x0.95mm_HandSolder, symbol Device:R
- added R726: 51, Resistor_SMD:R_0603_1608Metric_Pad0.98x0.95mm_HandSolder, symbol Device:R
- added R727, R728: 100k, Resistor_SMD:R_0603_1608Metric_Pad0.98x0.95mm_HandSolder, symbol Device:R
- added RN701: 51, symbol Device:R_Pack06
- added U701: LMH6618MK, Package_TO_SOT_SMD:TSOT-23-6_HandSoldering, symbol ETH1LCR3:LMH6618MK
- added U703: 74HCT4051PW, Package_SO:TSSOP-16_4.4x5mm_P0.65mm, symbol ETH1LCR3:74HCT4051PW
- added U709: ADS1246IPWR, Package_SO:TSSOP-16_4.4x5mm_P0.65mm, symbol ETH1LCR3:ADS1246IPWR
- added U710: REF2025, Package_TO_SOT_SMD:SOT-23-5, symbol Reference_Voltage:REF2025
- R702: value 100n/C0G -> 120k/.1%; footprint (none) -> Resistor_SMD:R_0603_1608Metric_Pad0.98x0.95mm_HandSolder
- R703: value 100n/C0G -> 510; footprint (none) -> Resistor_SMD:R_0603_1608Metric_Pad0.98x0.95mm_HandSolder
- R705: value 100n/C0G -> 3k; footprint (none) -> Resistor_SMD:R_0603_1608Metric_Pad0.98x0.95mm_HandSolder
- R706: value 100n/C0G -> 12k; footprint (none) -> Resistor_SMD:R_0603_1608Metric_Pad0.98x0.95mm_HandSolder
- R718: renamed from R701; value 100 -> 100/.05%; footprint (none) -> Resistor_SMD:R_0603_1608Metric_Pad0.98x0.95mm_HandSolder
- R720: renamed from R704; value 100 -> 100/.05%; footprint (none) -> Resistor_SMD:R_0603_1608Metric_Pad0.98x0.95mm_HandSolder
- U704: renamed from U701; footprint (none) -> Package_TO_SOT_SMD:SOT-23-6_Handsoldering
- U705: renamed from U702; footprint (none) -> Package_TO_SOT_SMD:SOT-23-6_Handsoldering
- renumbered U706 to U702, U705 to U706, U704 to U707, U703 to U708
Connections:
- net +5V: now also U702.4 (V+), C704.1, C705.1, C706.1, C708.1, C709.1, C710.1, C711.1, C712.1, C719.1, C720.1, D702.1 (K), R707.2, R726.1, U701.6 (V+), U703.16 (VCC), U710.3 (EN), U710.4 (IN)
- net GND: now also U702.2 (V-), U702.6 (SHDN), C702.2, C703.2, C704.2, C705.2, C706.2, C707.2, C708.2, C709.2, C710.2, C711.2, C712.2, C713.2, C714.2, C715.1, C716.2, C717.2, C718.1, C719.2, C720.2, C721.2, C722.2, C723.2, C724.2, C725.2, D701.2 (A), R717.1, U703.6 (~{E}), U703.8 (GND), U709.2 (DGND), U709.3 (CLK), U709.6 (REFN), U709.9 (AVSS), U710.2 (GND); no longer R703.2, R705.2
- net at U704.1: now also R724.1
- net at U704.3, U705.1: now also U703.3 (Z)
- net at R702.1, R703.1: now also D702.2 (A), R701.2, U701.3 (+); no longer R718.2
- net at U702.1 (-): now also R705.2, R706.1, C702.1
- net at U702.3 (+): now also D701.1 (K), R704.2
- net at U702.5: now also D703.2 (A)
- net PSD_RC_B: now reaches U707.2 (A)
- net at U707.4 (Y): now also U703.10 (S1)
- net PSD_RC_C: now reaches U708.2 (A)
- net at U708.4 (Y): now also U703.9 (S2)
- net at U705.3: now also R725.1
- net PSD_RC_A: now reaches U706.2 (A)
- net at U706.4 (Y): now also U703.11 (S0)
- new net: R707.1, U701.5 (~{DISABLE})
- new net: C703.1, R708.1, R709.1, R710.1, R711.1, R712.1, R713.1, R714.1, R715.1, U701.1, U701.4 (-)
- new net: R712.2, U703.1 (Y4)
- new net: C701.1, R703.2
- new net: R708.2, U703.13 (Y0)
- new net: C716.1, R725.2, U709.8 (AINN)
- new net: R713.2, U703.5 (Y5)
- new net: C722.1, C723.1, R718.2
- new net: C718.2, L701.1, U709.1 (DVDD)
- new net: R714.2, U703.2 (Y6)
- new net: C724.1, C725.1, R720.2
- new net: C721.1, R726.2, U709.10 (AVDD)
- new net: R710.2, U703.15 (Y2)
- new net: R711.2, U703.12 (Y3)
- new net: C715.2, R724.2, U709.7 (AINP)
- new net: R709.2, U703.14 (Y1)
- new net: R715.2, U703.4 (Y7)
- new net: R727.1, RN701.6 (R6.1), U709.11 (START)
- new net: RN701.5 (R5.1), U709.12 (~{CS})
- new net: RN701.4 (R4.1), U709.13 (~{DRDY})
- new net: RN701.3 (R3.1), U709.14 (DOUT/~{DRDY})
- new net: RN701.2 (R2.1), U709.15 (DIN)
- new net: RN701.1 (R1.1), U709.16 (SCLK)
- new net: R728.1, U709.4 (~{RESET})
- new net: C707.1, D703.1 (K), R716.1
- new net +2V5: C717.1, R701.1, R705.1, U709.5 (REFP), U710.5 (Vref)
- new net +3.3V: L701.2, R727.2, R728.2
- new net -5V: C713.1, C714.1, U701.2 (V-), U703.7 (VEE)
- new net ADS_DIN: RN701.11 (R2.2)
- new net ADS_DOUT: RN701.10 (R3.2)
- new net ADS_SCLK: RN701.12 (R1.2)
- new net ADS_START: RN701.7 (R6.2)
- new net ADS_~{CS}: RN701.8 (R5.2)
- new net ADS_~{DRDY}: RN701.9 (R4.2)
- new net INPUT_CPO: R716.2, R717.2
- new net PGA_OUT: C701.2, R704.1
- no-connect marks 0 -> 1
Other:
- moved on the sheet: R718, R720, U702, U704A, U704B, U705A, U705B, U706, U707, U708

Commit message: Hardware
Parts:
- R701: value 30/.1% -> 30k/.1%
- R716, R717: value 1k6/.1% -> 1k6
- renumbered C722 to C713, C725 to C714, C713 to C715, C723 to C716, C724 to C717, C714 to C718, C715 to C719, C716 to C720, C717 to C721, C718 to C722, C719 to C723, C720 to C724, C721 to C725, R720 to R719, R724 to R720, R725 to R721, R726 to R722, R727 to R723, R728 to R724
Changed lines of the file:
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@@
 	(wire
 		(pts
-			(xy 265.43 40.64) (xy 269.24 40.64)
+			(xy 265.43 40.64) (xy 266.7 40.64)
 		)
 		(stroke
@@
 	(wire
 		(pts
-			(xy 265.43 50.8) (xy 269.24 50.8)
+			(xy 265.43 50.8) (xy 266.7 50.8)
 		)
 		(stroke
@@
 	(wire
 		(pts
-			(xy 265.43 45.72) (xy 269.24 45.72)
+			(xy 265.43 45.72) (xy 266.7 45.72)
 		)
 		(stroke
@@
 	(wire
 		(pts
-			(xy 265.43 48.26) (xy 269.24 48.26)
+			(xy 265.43 48.26) (xy 266.7 48.26)
 		)
 		(stroke
@@
 	(wire
 		(pts
-			(xy 265.43 43.18) (xy 269.24 43.18)
+			(xy 265.43 43.18) (xy 266.7 43.18)
 		)
 		(stroke
@@
 	(wire
 		(pts
-			(xy 265.43 53.34) (xy 269.24 53.34)
+			(xy 265.43 53.34) (xy 266.7 53.34)
 		)
 		(stroke
@@
 	(hierarchical_label "ADS_~{CS}"
 		(shape input)
-		(at 269.24 50.8 0)
+		(at 266.7 50.8 0)
 		(fields_autoplaced yes)
 		(effects
@@
 	(hierarchical_label "ADS_DOUT"
 		(shape input)
-		(at 269.24 45.72 0)
+		(at 266.7 45.72 0)
 		(fields_autoplaced yes)
 		(effects
@@
 	(hierarchical_label "ADS_~{DRDY}"
 		(shape input)
-		(at 269.24 48.26 0)
+		(at 266.7 48.26 0)
 		(fields_autoplaced yes)
 		(effects
@@
 	(hierarchical_label "ADS_START"
 		(shape input)
-		(at 269.24 53.34 0)
+		(at 266.7 53.34 0)
 		(fields_autoplaced yes)
 		(effects
@@
 	(hierarchical_label "ADS_DIN"
 		(shape input)
-		(at 269.24 43.18 0)
+		(at 266.7 43.18 0)
 		(fields_autoplaced yes)
 		(effects
@@
 	(hierarchical_label "ADS_SCLK"
 		(shape input)
-		(at 269.24 40.64 0)
+		(at 266.7 40.64 0)
 		(fields_autoplaced yes)
 		(effects
@@
 			)
 		)
-		(property "Value" "1k6/.1%"
+		(property "Value" "1k6"
 			(at 109.22 149.8599 0)
 			(effects
@@
 		(on_board yes)
 		(dnp no)
-		(property "Reference" "R725"
+		(property "Reference" "R721"
 			(at 186.69 60.96 90)
 			(effects
@@
 			(project "ETH1LCR3"
 				(path "/6623bacb-57aa-43ce-9e51-b38a560dd9fc/effecda5-769f-4dde-a513-c082279edfb3"
-					(reference "R725")
+					(reference "R721")
 					(unit 1)
 				)
@@
 			)
 		)
-		(property "Value" "30/.1%"
+		(property "Value" "30k/.1%"
 			(at 19.05 46.9899 0)
 			(effects
@@
 		(dnp no)
 		(fields_autoplaced yes)
-		(property "Reference" "C716"
+		(property "Reference" "C720"
 			(at 195.58 67.3099 0)
 			(effects
@@
 			(project ""
 				(path "/6623bacb-57aa-43ce-9e51-b38a560dd9fc/effecda5-769f-4dde-a513-c082279edfb3"
-					(reference "C716")
+					(reference "C720")
 					(unit 1)
 				)
@@
 		(dnp no)
 		(fields_autoplaced yes)
-		(property "Reference" "R720"
+		(property "Reference" "R719"
 			(at 149.86 64.7699 0)
 			(effects
@@
 			(project "ETH1LCR3"
 				(path "/6623bacb-57aa-43ce-9e51-b38a560dd9fc/effecda5-769f-4dde-a513-c082279edfb3"
-					(reference "R720")
+					(reference "R719")
 					(unit 1)
 				)
@@
 		(dnp no)
 		(fields_autoplaced yes)
-		(property "Reference" "C718"
+		(property "Reference" "C722"
 			(at 214.63 21.59 90)
 			(effects
@@
 			(project "ETH1LCR3"
 				(path "/6623bacb-57aa-43ce-9e51-b38a560dd9fc/effecda5-769f-4dde-a513-c082279edfb3"
-					(reference "C718")
+					(reference "C722")
 					(unit 1)
 				)
@@
 		(dnp no)
 		(fields_autoplaced yes)
-		(property "Reference" "C721"
+		(property "Reference" "C725"
 			(at 250.19 21.59 90)
 			(effects
@@
 			(project "ETH1LCR3"
 				(path "/6623bacb-57aa-43ce-9e51-b38a560dd9fc/effecda5-769f-4dde-a513-c082279edfb3"
-					(reference "C721")
+					(reference "C725")
 					(unit 1)
 				)
@@
 		(dnp no)
 		(fields_autoplaced yes)
-		(property "Reference" "R726"
+		(property "Reference" "R722"
 			(at 240.03 22.8599 0)
 			(effects
@@
 			(project ""
 				(path "/6623bacb-57aa-43ce-9e51-b38a560dd9fc/effecda5-769f-4dde-a513-c082279edfb3"
-					(reference "R726")
+					(reference "R722")
 					(unit 1)
 				)
@@
 		(dnp no)
 		(fields_autoplaced yes)
-		(property "Reference" "C722"
+		(property "Reference" "C713"
 			(at 151.13 48.2599 0)
 			(effects
@@
 			(project ""
 				(path "/6623bacb-57aa-43ce-9e51-b38a560dd9fc/effecda5-769f-4dde-a513-c082279edfb3"
-					(reference "C722")
+					(reference "C713")
 					(unit 1)
 				)
@@
 		(dnp no)
 		(fields_autoplaced yes)
-		(property "Reference" "C717"
+		(property "Reference" "C721"
 			(at 212.09 43.1799 0)
 			(effects
@@
 			(project ""
 				(path "/6623bacb-57aa-43ce-9e51-b38a560dd9fc/effecda5-769f-4dde-a513-c082279edfb3"
-					(reference "C717")
+					(reference "C721")
 					(unit 1)
 				)
@@
 		(on_board yes)
 		(dnp no)
-		(property "Reference" "C713"
+		(property "Reference" "C715"
 			(at 159.258 184.404 0)
 			(effects
@@
 			(project "ETH1LCR3"
 				(path "/6623bacb-57aa-43ce-9e51-b38a560dd9fc/effecda5-769f-4dde-a513-c082279edfb3"
-					(reference "C713")
+					(reference "C715")
 					(unit 1)
 				)
@@
 		(dnp no)
 		(fields_autoplaced yes)
-		(property "Reference" "C715"
+		(property "Reference" "C719"
 			(at 195.58 49.5299 0)
 			(effects
@@
 			(project "ETH1LCR3"
 				(path "/6623bacb-57aa-43ce-9e51-b38a560dd9fc/effecda5-769f-4dde-a513-c082279edfb3"
-					(reference "C715")
+					(reference "C719")
 					(unit 1)
 				)
@@
 		(on_board yes)
 		(dnp no)
-		(property "Reference" "R727"
+		(property "Reference" "R723"
 			(at 260.35 57.404 90)
 			(effects
@@
 			(project "ETH1LCR3"
 				(path "/6623bacb-57aa-43ce-9e51-b38a560dd9fc/effecda5-769f-4dde-a513-c082279edfb3"
-					(reference "R727")
+					(reference "R723")
 					(unit 1)
 				)
@@
 			)
 		)
-		(property "Value" "1k6/.1%"
+		(property "Value" "1k6"
 			(at 100.33 139.7 90)
 			(effects
@@
 		(on_board yes)
 		(dnp no)
-		(property "Reference" "C719"
+		(property "Reference" "C723"
 			(at 237.998 114.554 0)
 			(effects
@@
 			(project "ETH1LCR3"
 				(path "/6623bacb-57aa-43ce-9e51-b38a560dd9fc/effecda5-769f-4dde-a513-c082279edfb3"
-					(reference "C719")
+					(reference "C723")
 					(unit 1)
 				)
@@
 		(on_board yes)
 		(dnp no)
-		(property "Reference" "R728"
+		(property "Reference" "R724"
 			(at 260.35 66.04 90)
 			(effects
@@
 			(project ""
 				(path "/6623bacb-57aa-43ce-9e51-b38a560dd9fc/effecda5-769f-4dde-a513-c082279edfb3"
-					(reference "R728")
+					(reference "R724")
 					(unit 1)
 				)
@@
 		(dnp no)
 		(fields_autoplaced yes)
-		(property "Reference" "C725"
+		(property "Reference" "C714"
 			(at 151.13 74.9299 0)
 			(effects
@@
 			(project "ETH1LCR3"
 				(path "/6623bacb-57aa-43ce-9e51-b38a560dd9fc/effecda5-769f-4dde-a513-c082279edfb3"
-					(reference "C725")
+					(reference "C714")
 					(unit 1)
 				)
@@
 		(dnp no)
 		(fields_autoplaced yes)
-		(property "Reference" "C720"
+		(property "Reference" "C724"
 			(at 249.301 114.4016 0)
 			(effects
@@
 			(project "ETH1LCR3"
 				(path "/6623bacb-57aa-43ce-9e51-b38a560dd9fc/effecda5-769f-4dde-a513-c082279edfb3"
-					(reference "C720")
+					(reference "C724")
 					(unit 1)
 				)
@@
 		(dnp no)
 		(fields_autoplaced yes)
-		(property "Reference" "C724"
+		(property "Reference" "C717"
 			(at 168.91 74.9299 0)
 			(effects
@@
 			(project "ETH1LCR3"
 				(path "/6623bacb-57aa-43ce-9e51-b38a560dd9fc/effecda5-769f-4dde-a513-c082279edfb3"
-					(reference "C724")
+					(reference "C717")
 					(unit 1)
 				)
@@
 		(on_board yes)
 		(dnp no)
-		(property "Reference" "C714"
+		(property "Reference" "C718"
 			(at 170.688 184.404 0)
 			(effects
@@
 			(project "ETH1LCR3"
 				(path "/6623bacb-57aa-43ce-9e51-b38a560dd9fc/effecda5-769f-4dde-a513-c082279edfb3"
-					(reference "C714")
+					(reference "C718")
 					(unit 1)
 				)
@@
 		(dnp no)
 		(fields_autoplaced yes)
-		(property "Reference" "C723"
+		(property "Reference" "C716"
 			(at 168.91 48.2599 0)
 			(effects
@@
 			(project "ETH1LCR3"
 				(path "/6623bacb-57aa-43ce-9e51-b38a560dd9fc/effecda5-769f-4dde-a513-c082279edfb3"
-					(reference "C723")
+					(reference "C716")
 					(unit 1)
 				)
@@
 		(on_board yes)
 		(dnp no)
-		(property "Reference" "R724"
+		(property "Reference" "R720"
 			(at 186.69 53.34 90)
 			(effects
@@
 			(project ""
 				(path "/6623bacb-57aa-43ce-9e51-b38a560dd9fc/effecda5-769f-4dde-a513-c082279edfb3"
-					(reference "R724")
+					(reference "R720")
 					(unit 1)
 				)

Commit message: Hardware
Parts:
- added C726, C728: 0.1u, Capacitor_SMD:C_0603_1608Metric_Pad1.08x0.95mm_HandSolder, symbol Device:C
- added C727, C729: 1u, Capacitor_SMD:C_0603_1608Metric_Pad1.08x0.95mm_HandSolder, symbol Device:C
Connections:
- net +2V5: now also C726.1, C727.1
- net GND: now also C726.2, C727.2, C728.2, C729.2
- net +1V25: now reaches U710.1 (Vbias)
- net +1V25: now also C728.1, C729.1
- no-connect marks 1 -> 0

Commit message: Hardware
Changed lines of the file:
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@@
 		)
 		(property "Value" "GND"
-			(at 191.77 76.2 0)
+			(at 191.77 76.708 0)
 			(effects
 				(font
@@
 		)
 		(property "Value" "GND"
-			(at 191.77 43.18 0)
+			(at 191.77 42.926 0)
 			(effects
 				(font
@@
 		)
 		(property "Value" "GND"
-			(at 208.28 53.34 0)
+			(at 208.28 53.848 0)
 			(effects
 				(font

Commit message: Software and hardware
Parts:
- renumbered C726 to C701, C727 to C702, C701 to C703, C728 to C704, C702 to C705, C729 to C706, C703 to C707, C704 to C708, C705 to C709, C706 to C710, C707 to C711, C708 to C712, C709 to C713, C710 to C714, C711 to C715, C712 to C716, C713 to C717, C714 to C718, C715 to C719, C716 to C720, C717 to C721, C718 to C722, C719 to C723, C720 to C724, C721 to C725, C722 to C726, C723 to C727, C724 to C728, C725 to C729
Connections:
- net INPUT_CPO renamed INPUT_COMP

Commit message: Hardware
Other:
- moved on the sheet: D703
Changed lines of the file:
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@@
 	(wire
 		(pts
-			(xy 68.58 143.51) (xy 77.47 143.51)
+			(xy 68.58 143.51) (xy 80.01 143.51)
 		)
 		(stroke
@@
 	(wire
 		(pts
-			(xy 85.09 143.51) (xy 93.98 143.51)
+			(xy 87.63 143.51) (xy 93.98 143.51)
 		)
 		(stroke
@@
 	)
 	(symbol
-		(lib_id "power:PWR_FLAG")
-		(at 261.62 90.17 180)
-		(unit 1)
-		(exclude_from_sim no)
-		(in_bom yes)
-		(on_board yes)
-		(dnp no)
-		(fields_autoplaced yes)
-		(property "Reference" "#FLG0701"
-			(at 261.62 92.075 0)
-			(effects
-				(font
-					(size 1.27 1.27)
-				)
-				(hide yes)
-			)
-		)
-		(property "Value" "PWR_FLAG"
-			(at 261.62 95.25 0)
-			(effects
-				(font
-					(size 1.27 1.27)
-				)
-			)
-		)
-		(property "Footprint" ""
-			(at 261.62 90.17 0)
-			(effects
-				(font
-					(size 1.27 1.27)
-				)
-				(hide yes)
-			)
-		)
-		(property "Datasheet" "~"
-			(at 261.62 90.17 0)
-			(effects
-				(font
-					(size 1.27 1.27)
-				)
-				(hide yes)
-			)
-		)
-		(property "Description" "Special symbol for telling ERC where power comes from"
-			(at 261.62 90.17 0)
-			(effects
-				(font
-					(size 1.27 1.27)
-				)
-				(hide yes)
-			)
-		)
-		(pin "1"
-		)
-		(instances
-			(project ""
-				(path "/6623bacb-57aa-43ce-9e51-b38a560dd9fc/effecda5-769f-4dde-a513-c082279edfb3"
-					(reference "#FLG0701")
-					(unit 1)
-				)
-			)
-		)
-	)
-	(symbol
 		(lib_id "power:GND")
 		(at 191.77 72.39 0)
@@
 	)
 	(symbol
+		(lib_id "power:+2V5")
+		(at 261.62 91.44 0)
+		(unit 1)
+		(exclude_from_sim no)
+		(in_bom yes)
+		(on_board yes)
+		(dnp no)
+		(fields_autoplaced yes)
+		(property "Reference" "#PWR0745"
+			(at 261.62 95.25 0)
+			(effects
+				(font
+					(size 1.27 1.27)
+				)
+				(hide yes)
+			)
+		)
+		(property "Value" "+2V5"
+			(at 261.62 86.36 0)
+			(effects
+				(font
+					(size 1.27 1.27)
+				)
+			)
+		)
+		(property "Footprint" ""
+			(at 261.62 91.44 0)
+			(effects
+				(font
+					(size 1.27 1.27)
+				)
+				(hide yes)
+			)
+		)
+		(property "Datasheet" ""
+			(at 261.62 91.44 0)
+			(effects
+				(font
+					(size 1.27 1.27)
+				)
+				(hide yes)
+			)
+		)
+		(property "Description" "Power symbol creates a global label with name \"+2V5\""
+			(at 261.62 91.44 0)
+			(effects
+				(font
+					(size 1.27 1.27)
+				)
+				(hide yes)
+			)
+		)
+		(pin "1"
+		)
+		(instances
+			(project ""
+				(path "/6623bacb-57aa-43ce-9e51-b38a560dd9fc/effecda5-769f-4dde-a513-c082279edfb3"
+					(reference "#PWR0745")
+					(unit 1)
+				)
+			)
+		)
+	)
+	(symbol
 		(lib_id "power:GND")
 		(at 102.87 191.77 0)
@@
 	)
 	(symbol
+		(lib_id "power:PWR_FLAG")
+		(at 261.62 91.44 180)
+		(unit 1)
+		(exclude_from_sim no)
+		(in_bom yes)
+		(on_board yes)
+		(dnp no)
+		(fields_autoplaced yes)
+		(property "Reference" "#FLG0701"
+			(at 261.62 93.345 0)
+			(effects
+				(font
+					(size 1.27 1.27)
+				)
+				(hide yes)
+			)
+		)
+		(property "Value" "PWR_FLAG"
+			(at 261.62 96.52 0)
+			(effects
+				(font
+					(size 1.27 1.27)
+				)
+			)
+		)
+		(property "Footprint" ""
+			(at 261.62 91.44 0)
+			(effects
+				(font
+					(size 1.27 1.27)
+				)
+				(hide yes)
+			)
+		)
+		(property "Datasheet" "~"
+			(at 261.62 91.44 0)
+			(effects
+				(font
+					(size 1.27 1.27)
+				)
+				(hide yes)
+			)
+		)
+		(property "Description" "Special symbol for telling ERC where power comes from"
+			(at 261.62 91.44 0)
+			(effects
+				(font
+					(size 1.27 1.27)
+				)
+				(hide yes)
+			)
+		)
+		(pin "1"
+		)
+		(instances
+			(project ""
+				(path "/6623bacb-57aa-43ce-9e51-b38a560dd9fc/effecda5-769f-4dde-a513-c082279edfb3"
+					(reference "#FLG0701")
+					(unit 1)
+				)
+			)
+		)
+	)
+	(symbol
 		(lib_id "Device:R")
 		(at 71.12 53.34 90)
@@
 	)
 	(symbol
-		(lib_id "power:+1V2")
-		(at 261.62 90.17 0)
-		(unit 1)
-		(exclude_from_sim no)
-		(in_bom yes)
-		(on_board yes)
-		(dnp no)
-		(fields_autoplaced yes)
-		(property "Reference" "#PWR0745"
-			(at 261.62 93.98 0)
-			(effects
-				(font
-					(size 1.27 1.27)
-				)
-				(hide yes)
-			)
-		)
-		(property "Value" "+1V2"
-			(at 261.62 85.09 0)
-			(effects
-				(font
-					(size 1.27 1.27)
-				)
-			)
-		)
-		(property "Footprint" ""
-			(at 261.62 90.17 0)
-			(effects
-				(font
-					(size 1.27 1.27)
-				)
-				(hide yes)
-			)
-		)
-		(property "Datasheet" ""
-			(at 261.62 90.17 0)
-			(effects
-				(font
-					(size 1.27 1.27)
-				)
-				(hide yes)
-			)
-		)
-		(property "Description" "Power symbol creates a global label with name \"+1V2\""
-			(at 261.62 90.17 0)
-			(effects
-				(font
-					(size 1.27 1.27)
-				)
-				(hide yes)
-			)
-		)
-		(pin "1"
-		)
-		(instances
-			(project ""
-				(path "/6623bacb-57aa-43ce-9e51-b38a560dd9fc/effecda5-769f-4dde-a513-c082279edfb3"
-					(reference "#PWR0745")
-					(unit 1)
-				)
-			)
-		)
-	)
-	(symbol
 		(lib_id "Device:R")
 		(at 186.69 55.88 90)
@@
 	(symbol
 		(lib_id "Device:D")
-		(at 81.28 143.51 180)
+		(at 83.82 143.51 180)
 		(unit 1)
 		(exclude_from_sim no)
@@
 		(fields_autoplaced yes)
 		(property "Reference" "D703"
-			(at 81.28 137.16 0)
+			(at 83.82 137.16 0)
 			(effects
 				(font
@@
 		)
 		(property "Value" "NSVRB751V40T1G"
-			(at 81.28 139.7 0)
+			(at 83.82 139.7 0)
 			(effects
 				(font
@@
 		)
 		(property "Footprint" ""
-			(at 81.28 143.51 0)
+			(at 83.82 143.51 0)
 			(effects
 				(font
@@
 		)
 		(property "Datasheet" "~"
-			(at 81.28 143.51 0)
+			(at 83.82 143.51 0)
 			(effects
 				(font
@@
 		)
 		(property "Description" "Diode"
-			(at 81.28 143.51 0)
+			(at 83.82 143.51 0)
 			(effects
 				(font
@@
 		)
 		(property "Sim.Device" "D"
-			(at 81.28 143.51 0)
+			(at 83.82 143.51 0)
 			(effects
 				(font
@@
 		)
 		(property "Sim.Pins" "1=K 2=A"
-			(at 81.28 143.51 0)
+			(at 83.82 143.51 0)
 			(effects
 				(font

Commit message: Hardware
Parts:
- removed RN701: 51, symbol Device:R_Pack06
- added RN701: 51, Resistor_SMD:R_Array_Convex_2x0603, symbol Device:R_Pack02
- added RN702: 51, Resistor_SMD:R_Array_Convex_4x0603, symbol Device:R_Pack04
- C717, C718, C720, C721: footprint (none) -> Capacitor_SMD:C_1206_3216Metric_Pad1.33x1.80mm_HandSolder
- C723, C724: footprint (none) -> Capacitor_SMD:C_0603_1608Metric_Pad1.08x0.95mm_HandSolder
- C725, C726, C729: footprint (none) -> Capacitor_SMD:C_0805_2012Metric_Pad1.18x1.45mm_HandSolder
- D701, D702, D703: footprint (none) -> Diode_SMD:D_SOD-323_HandSoldering
Connections:
- net ADS_DIN: now also RN702.7 (R2.2)
- net ADS_DOUT: now also RN702.6 (R3.2)
- net ADS_SCLK: now also RN702.8 (R1.2)
- net ADS_START: now also RN701.1 (R1.1)
- net ADS_~{CS}: now also RN701.2 (R2.1)
- net ADS_~{DRDY}: now also RN702.5 (R4.2)
- net at R723.1, U709.11 (START): now also RN701.4 (R1.2)
- net at U709.12 (~{CS}): now also RN701.3 (R2.2)
- net at U709.13 (~{DRDY}): now also RN702.4 (R4.1)
- net at U709.14 (DOUT/~{DRDY}): now also RN702.3 (R3.1)
- net at U709.15 (DIN): now also RN702.2 (R2.1)
- net at U709.16 (SCLK): now also RN702.1 (R1.1)
Other:
- moved on the sheet: R723, R724
