File: Hardware/ETH1LCR3/PSD.kicad_sch (KiCad schematic)
At the start: 69 parts, among them U701 LMH6618MK, U702 TLV3501AIDBV, U703 74HCT4051PW, U704 SN74LVC1G3157DB, U705 SN74LVC1G3157DB, U706 SN74LV1T34DBV, U707 SN74LV1T34DBV, U708 SN74LV1T34DBV, U709 ADS1246IPWR, U710 REF2025

Commit message: PCB layout
Parts:
- U701: value LMH6618MK -> LMH6618MKE; footprint Package_TO_SOT_SMD:TSOT-23-6_HandSoldering -> Package_TO_SOT_SMD:SOT-23-6_Handsoldering
- U702: footprint Package_TO_SOT_SMD:SOT-23-6 -> Package_TO_SOT_SMD:SOT-23-6_Handsoldering
- U706, U707, U708: footprint Package_TO_SOT_SMD:SOT-23-5 -> Package_TO_SOT_SMD:SOT-23-5_HandSoldering
Changed lines of the file:
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@@
 			)
 		)
-		(property "Footprint" "Package_TO_SOT_SMD:SOT-23-6"
+		(property "Footprint" "Package_TO_SOT_SMD:SOT-23-6_Handsoldering"
 			(at 60.96 153.035 0)
 			(effects
@@
 			)
 		)
-		(property "Footprint" "Package_TO_SOT_SMD:SOT-23-5"
+		(property "Footprint" "Package_TO_SOT_SMD:SOT-23-5_HandSoldering"
 			(at 147.32 121.92 0)
 			(effects
@@
 			)
 		)
-		(property "Footprint" "Package_TO_SOT_SMD:SOT-23-5"
+		(property "Footprint" "Package_TO_SOT_SMD:SOT-23-5_HandSoldering"
 			(at 168.91 107.95 0)
 			(effects
@@
 			)
 		)
-		(property "Value" "LMH6618MK"
+		(property "Value" "LMH6618MKE"
 			(at 49.53 48.514 0)
 			(effects
@@
 			)
 		)
-		(property "Footprint" "Package_TO_SOT_SMD:TSOT-23-6_HandSoldering"
+		(property "Footprint" "Package_TO_SOT_SMD:SOT-23-6_Handsoldering"
 			(at 46.99 59.69 0)
 			(effects
@@
 			)
 		)
-		(property "Footprint" "Package_TO_SOT_SMD:SOT-23-5"
+		(property "Footprint" "Package_TO_SOT_SMD:SOT-23-5_HandSoldering"
 			(at 124.46 135.89 0)
 			(effects
