File: Hardware/ETH1LCR3/Power.kicad_sch (KiCad schematic)
At the start: 0 parts

Commit message: Hardware
Parts:
- added C407, C426, C428, C432, C433: 4u7, symbol Device:C
- added C409, C411, C423, C427, C435, C437: 2u2, symbol Device:C
- added C424: 100n, symbol Device:C
- added C425: 270p, symbol Device:C
- added C429, C430: 1u, symbol Device:C
- added C431: 1n, symbol Device:C
- added C434: 33u/12V, symbol Device:C_Polarized
- added C436: 10n, symbol Device:C
- added C438: 470u/12V, symbol Device:C_Polarized
- added D402: BZX84C10LT1G, Package_TO_SOT_SMD:SOT-23, symbol Diode:BZX84Cxx
- added D403: 1N4148W, Diode_SMD:D_SOD-123, symbol Diode:1N4148W
- added D404, D405: MBR0520, symbol Device:D_Schottky
- added F401: 1812L075/33DR, Fuse:Fuse_1812_4532Metric_Pad1.30x3.40mm_HandSolder, symbol Device:Fuse
- added J402: 1715721, TerminalBlock_Phoenix:TerminalBlock_Phoenix_MKDS-1,5-2_1x02_P5.00mm_Horizontal, symbol Connector_Generic:Conn_01x02
- added L401, L402, L404, L406: MLZ1608DR47DT, symbol Device:L
- added L403: 1008PS-222KLB, symbol Device:L
- added L405: DRQ73, symbol Device:L_Coupled_Small_1324
- added L407, L408: MLZ2012M100WT, symbol Device:L
- added Q401: SI5618A, Package_TO_SOT_SMD:SOT-23, symbol Device:Q_PMOS_GSD
- added Q402: MMBT3904, Package_TO_SOT_SMD:SOT-23, symbol Transistor_BJT:MMBT3904
- added Q403: BSS123, Package_TO_SOT_SMD:SOT-23, symbol Transistor_FET:BSS123
- added R401, R403: 100k, Resistor_SMD:R_0603_1608Metric_Pad0.98x0.95mm_HandSolder, symbol Device:R
- added R410, R412, R415, R420: 10k, symbol Device:R
- added R411, R418: 51, symbol Device:R
- added R413: 27k, symbol Device:R
- added R414: 2k4, symbol Device:R
- added R416: 12k, symbol Device:R
- added R417: 100k, symbol Device:R
- added R419, R421: 30k, symbol Device:R
- added U401: TEL5-2411, ETH1LCR3:CONV_TEL_5-2411, symbol ETH1LCR3:TEL5-2411
- added U405: LT1946A, Package_SO:MSOP-8-1EP_3x3mm_P0.65mm_EP1.95x2.15mm_ThermalVias, symbol ETH1LCR3:LT1946A
- added U406: TLV70033_SOT23-5, Package_TO_SOT_SMD:SOT-23-5, symbol Regulator_Linear:TLV70033_SOT23-5
- added U407: LT1611, Package_TO_SOT_SMD:SOT-23-5_HandSoldering, symbol ETH1LCR3:LT1611
- added U408: REG103GA-5, Package_TO_SOT_SMD:SOT-223-6, symbol ETH1LCR3:REG103GA-5
Connections:
- new net: Q403.1 (G), R417.1, R418.1
- new net: C427.1, L403.1, L404.2, R410.1, U405.6 (VIN)
- new net: C431.2, C433.1, C434.2, L405.3, L407.1, R421.2
- new net: D403.1 (K), Q402.1 (B), R403.1
- new net: D402.1 (A), Q401.1 (G), Q402.3 (C), R401.1
- new net: C430.1, L405.2, U407.1 (SW1)
- new net: C430.2, D405.2 (A), L405.1
- new net: R414.1, R415.2, R416.1, U405.2 (FB)
- new net: R413.1, U405.1 (VC)
- new net: R410.2, R411.2, R412.1, U405.3 (~{SHDN})
- new net: D404.2 (A), L403.2, U405.5 (SW)
- new net: C424.1, U405.8 (SS)
- new net: C431.1, R420.1, R421.1, U407.3 (NFB)
- new net: C432.1, L405.4, L406.2, R419.1, U407.5 (VIN)
- new net: F401.1, J402.1 (Pin_1)
- new net: C436.1, U408.4 (NR)
- new net: F401.2, Q401.3 (D)
- new net: Q403.3 (D), R416.2
- new net: C429.1, R419.2, U407.4 (~{SHDN})
- new net: C423.1, L402.2, U406.1 (IN), U406.3 (EN)
- new net: C425.1, R413.2
- new net: C435.1, L408.2, U408.1 (VIN), U408.5 (ENA)
- new net: C407.1, L401.1, U401.14 (VOUT+)
- new net +3.3V: C411.1, U406.5 (OUT)
- new net +5V: C437.1, C438.1, U408.2 (VOUT)
- new net +5VP: C409.1, C428.1, L401.2, L402.1, L404.1, L406.1
- new net -5V: L407.2
- new net EN_BOOST: R411.1
- new net GND: C407.2, C409.2, C411.2, C423.2, C424.2, C425.2, C426.2, C427.2, C428.2, C429.2, C432.2, C433.2, C434.1, C435.2, C436.2, C437.2, C438.2, D405.1 (K), Q403.2 (S), R412.2, R414.2, R417.2, R420.2, U401.16 (VOUT-), U405.4 (GND), U405.7 (COMP), U405.9 (GND), U406.2 (GND), U407.2 (GND), U408.3 (GND), U408.6 (GND)
- new net GNDPWR: J402.2 (Pin_2), R401.2, R403.2, U401.2 (VIN-), U401.3 (VIN-)
- new net MAX_BOOST: R418.2
- new net VIN+: D402.3 (K), D403.2 (A), Q401.2 (S), Q402.2 (E), U401.22 (VIN+), U401.23 (VIN+)
- new net V_BOOST: C426.1, D404.1 (K), L408.1, R415.1

Commit message: Hardware
Parts:
- C405: renamed from C425; footprint (none) -> Capacitor_SMD:C_0603_1608Metric_Pad1.08x0.95mm_HandSolder
- C406: renamed from C424; value 100n -> 0.1u; footprint (none) -> Capacitor_SMD:C_0603_1608Metric_Pad1.08x0.95mm_HandSolder
- C408: renamed from C436; footprint (none) -> Capacitor_SMD:C_0603_1608Metric_Pad1.08x0.95mm_HandSolder
- C415: renamed from C429; footprint (none) -> Capacitor_SMD:C_0603_1608Metric_Pad1.08x0.95mm_HandSolder
- C416: renamed from C430; footprint (none) -> Capacitor_SMD:C_0603_1608Metric_Pad1.08x0.95mm_HandSolder
- C417: renamed from C431; footprint (none) -> Capacitor_SMD:C_0603_1608Metric_Pad1.08x0.95mm_HandSolder
- L401: renamed from L404; footprint (none) -> Inductor_SMD:L_0603_1608Metric_Pad1.05x0.95mm_HandSolder
- L402: footprint (none) -> Inductor_SMD:L_0603_1608Metric_Pad1.05x0.95mm_HandSolder
- L404: renamed from L408; footprint (none) -> Inductor_SMD:L_0805_2012Metric_Pad1.05x1.20mm_HandSolder
- L405: renamed from L406; footprint (none) -> Inductor_SMD:L_0603_1608Metric_Pad1.05x0.95mm_HandSolder
- L406: renamed from L401; footprint (none) -> Inductor_SMD:L_0603_1608Metric_Pad1.05x0.95mm_HandSolder
- L408: renamed from L407; footprint (none) -> Inductor_SMD:L_0805_2012Metric_Pad1.05x1.20mm_HandSolder
- R401: renamed from R411; footprint (none) -> Resistor_SMD:R_0603_1608Metric_Pad0.98x0.95mm_HandSolder
- R402: renamed from R412; footprint (none) -> Resistor_SMD:R_0603_1608Metric_Pad0.98x0.95mm_HandSolder
- R403: renamed from R410; footprint (none) -> Resistor_SMD:R_0603_1608Metric_Pad0.98x0.95mm_HandSolder
- R404: renamed from R413; footprint (none) -> Resistor_SMD:R_0603_1608Metric_Pad0.98x0.95mm_HandSolder
- R406: renamed from R415; footprint (none) -> Resistor_SMD:R_0603_1608Metric_Pad0.98x0.95mm_HandSolder
- R407: renamed from R414; footprint (none) -> Resistor_SMD:R_0603_1608Metric_Pad0.98x0.95mm_HandSolder
- R408: renamed from R416; footprint (none) -> Resistor_SMD:R_0603_1608Metric_Pad0.98x0.95mm_HandSolder
- R409: renamed from R417; footprint (none) -> Resistor_SMD:R_0603_1608Metric_Pad0.98x0.95mm_HandSolder
- R411: renamed from R418; footprint (none) -> Resistor_SMD:R_0603_1608Metric_Pad0.98x0.95mm_HandSolder
- R412: renamed from R419; footprint (none) -> Resistor_SMD:R_0603_1608Metric_Pad0.98x0.95mm_HandSolder
- R413: renamed from R420; footprint (none) -> Resistor_SMD:R_0603_1608Metric_Pad0.98x0.95mm_HandSolder
- R414: renamed from R421; footprint (none) -> Resistor_SMD:R_0603_1608Metric_Pad0.98x0.95mm_HandSolder
- renumbered C428 to C401, C427 to C402, C423 to C403, C411 to C404, C435 to C407, C437 to C409, C426 to C410, C438 to C411, C407 to C412, C432 to C413, C409 to C414, C433 to C418, C434 to C419, D404 to D401, D405 to D404, J402 to J401, L405 to L407, Q403 to Q402, Q402 to Q403, R401 to R405, R403 to R410, U406 to U401, U405 to U402, U408 to U403, U401 to U404, U407 to U405

Commit message: Hardware
Parts:
- removed J401: 1715721, TerminalBlock_Phoenix:TerminalBlock_Phoenix_MKDS-1,5-2_1x02_P5.00mm_Horizontal, symbol Connector_Generic:Conn_01x02
- removed U401: TLV70033_SOT23-5, Package_TO_SOT_SMD:SOT-23-5, symbol Regulator_Linear:TLV70033_SOT23-5
- added C420: 2u2, symbol Device:C
- added C421: 33u/12V, symbol Device:C_Polarized
- added R415: 51, Resistor_SMD:R_0603_1608Metric_Pad0.98x0.95mm_HandSolder, symbol Device:R
- added U401: REG103GA-3.3, Package_TO_SOT_SMD:SOT-223-6, symbol ETH1LCR3:REG103GA-5
- C404: value 2u2 -> 10n; footprint (none) -> Capacitor_SMD:C_0603_1608Metric_Pad1.08x0.95mm_HandSolder
- L402: value MLZ1608DR47DT -> MLZ2012M100WT; footprint Inductor_SMD:L_0603_1608Metric_Pad1.05x0.95mm_HandSolder -> Inductor_SMD:L_0805_2012Metric_Pad1.05x1.20mm_HandSolder
Connections:
- net +3.3V: now also C420.1, C421.1, U401.2 (VOUT); no longer C404.1
- net GND: now also C420.2, C421.2, U401.3 (GND), U401.6 (GND)
- net at C402.1, L401.2, L403.1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: now also R415.1
- net at R401.2, R402.1, R403.2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: now also R415.2
- net +24V: now reaches F401.1
- net at C403.1, L402.2: now also U401.1 (VIN), U401.5 (ENA)
- new net: C404.1, U401.4 (NR)
Other:
- moved on the sheet: C405, C406, C407, C408, C409, C410, C411, C413, C415, C416, C417, C418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

Commit message: Software and hardware
Parts:
- renumbered C403 to C402, C402 to C403, C420 to C405, C405 to C406, C421 to C407, C406 to C408, C407 to C409, C408 to C410, C409 to C411, C410 to C412, C411 to C413, C412 to C414, C413 to C415, C414 to C416, C415 to C417, C416 to C418, C417 to C419, C418 to C420, C419 to C421, D402 to D401, D401 to D402, L402 to L401, L401 to L402, L406 to L405, L405 to L406, Q403 to Q402, Q402 to Q403, R415 to R401, R401 to R402, R402 to R403, R403 to R404, R404 to R405, R405 to R406, R406 to R407, R407 to R408, R408 to R409, R409 to R411, R411 to R412, R412 to R413, R413 to R414, R414 to R415
Other:
- moved on the sheet: C402, C404, C405, C407, C409, C410, C411, C413, L401, L404, U401, U403

Commit message: Hardware
Connections:
- net VIN+: no longer names the net of D401.3 (K), D403.2 (A), Q401.2 (S), Q402.2 (E), U404.22 (VIN+), U404.23 (VIN+)
Changed lines of the file:
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@@
 	(paper "A4")
 	(junction
+		(at 134.62 22.86)
+		(diameter 0)
+		(color 0 0 0 0)
+	)
+	(junction
 		(at 88.9 36.83)
 		(diameter 0)
@@
 	(wire
 		(pts
+			(xy 134.62 21.59) (xy 134.62 22.86)
+		)
+		(stroke
+			(width 0)
+			(type default)
+		)
+	)
+	(wire
+		(pts
 			(xy 93.98 22.86) (xy 95.25 22.86)
 		)
@@
 	)
 	(symbol
+		(lib_id "power:GND")
+		(at 250.19 147.32 180)
+		(unit 1)
+		(exclude_from_sim no)
+		(in_bom yes)
+		(on_board yes)
+		(dnp no)
+		(fields_autoplaced yes)
+		(property "Reference" "#PWR0428"
+			(at 250.19 140.97 0)
+			(effects
+				(font
+					(size 1.27 1.27)
+				)
+				(hide yes)
+			)
+		)
+		(property "Value" "GND"
+			(at 250.19 142.24 0)
+			(effects
+				(font
+					(size 1.27 1.27)
+				)
+			)
+		)
+		(property "Footprint" ""
+			(at 250.19 147.32 0)
+			(effects
+				(font
+					(size 1.27 1.27)
+				)
+				(hide yes)
+			)
+		)
+		(property "Datasheet" ""
+			(at 250.19 147.32 0)
+			(effects
+				(font
+					(size 1.27 1.27)
+				)
+				(hide yes)
+			)
+		)
+		(property "Description" "Power symbol creates a global label with name \"GND\" , ground"
+			(at 250.19 147.32 0)
+			(effects
+				(font
+					(size 1.27 1.27)
+				)
+				(hide yes)
+			)
+		)
+		(pin "1"
+		)
+		(instances
+			(project ""
+				(path "/6623bacb-57aa-43ce-9e51-b38a560dd9fc/43994c6d-e030-4cc9-803d-7f33181d98ca"
+					(reference "#PWR0428")
+					(unit 1)
+				)
+			)
+		)
+	)
+	(symbol
 		(lib_id "Transistor_FET:BSS123")
 		(at 121.92 114.3 0)
@@
 	(symbol
 		(lib_id "power:PWR_FLAG")
+		(at 250.19 147.32 180)
+		(unit 1)
+		(exclude_from_sim no)
+		(in_bom yes)
+		(on_board yes)
+		(dnp no)
+		(fields_autoplaced yes)
+		(property "Reference" "#FLG0411"
+			(at 250.19 149.225 0)
+			(effects
+				(font
+					(size 1.27 1.27)
+				)
+				(hide yes)
+			)
+		)
+		(property "Value" "PWR_FLAG"
+			(at 250.19 152.4 0)
+			(effects
+				(font
+					(size 1.27 1.27)
+				)
+			)
+		)
+		(property "Footprint" ""
+			(at 250.19 147.32 0)
+			(effects
+				(font
+					(size 1.27 1.27)
+				)
+				(hide yes)
+			)
+		)
+		(property "Datasheet" "~"
+			(at 250.19 147.32 0)
+			(effects
+				(font
+					(size 1.27 1.27)
+				)
+				(hide yes)
+			)
+		)
+		(property "Description" "Special symbol for telling ERC where power comes from"
+			(at 250.19 147.32 0)
+			(effects
+				(font
+					(size 1.27 1.27)
+				)
+				(hide yes)
+			)
+		)
+		(pin "1"
+		)
+		(instances
+			(project "ETH1LCR3"
+				(path "/6623bacb-57aa-43ce-9e51-b38a560dd9fc/43994c6d-e030-4cc9-803d-7f33181d98ca"
+					(reference "#FLG0411")
+					(unit 1)
+				)
+			)
+		)
+	)
+	(symbol
+		(lib_id "power:PWR_FLAG")
 		(at 62.23 44.45 0)
 		(unit 1)
@@
 					(unit 1)
 				)
+			)
+		)
+	)
+	(symbol
+		(lib_id "power:PWR_FLAG")
+		(at 134.62 21.59 0)
+		(unit 1)
+		(exclude_from_sim no)
+		(in_bom yes)
+		(on_board yes)
+		(dnp no)
+		(fields_autoplaced yes)
+		(property "Reference" "#FLG0410"
+			(at 134.62 19.685 0)
+			(effects
+				(font
+					(size 1.27 1.27)
+				)
+				(hide yes)
+			)
+		)
+		(property "Value" "PWR_FLAG"
+			(at 134.62 16.51 0)
+			(effects
+				(font
+					(size 1.27 1.27)
+				)
+			)
+		)
+		(property "Footprint" ""
+			(at 134.62 21.59 0)
+			(effects
+				(font
+					(size 1.27 1.27)
+				)
+				(hide yes)
+			)
+		)
+		(property "Datasheet" "~"
+			(at 134.62 21.59 0)
+			(effects
+				(font
+					(size 1.27 1.27)
+				)
+				(hide yes)
+			)
+		)
+		(property "Description" "Special symbol for telling ERC where power comes from"
+			(at 134.62 21.59 0)
+			(effects
+				(font
+					(size 1.27 1.27)
+				)
+				(hide yes)
+			)
+		)
+		(pin "1"
+		)
+		(instances
+			(project "ETH1LCR3"
+				(path "/6623bacb-57aa-43ce-9e51-b38a560dd9fc/43994c6d-e030-4cc9-803d-7f33181d98ca"
+					(reference "#FLG0410")
+					(unit 1)
+				)

Commit message: Hardware
Parts:
- added C422: 470u/12V, Capacitor_SMD:CP_Elec_10x10.5, symbol Device:C_Polarized
- C401, C402, C403, C405, C409, C411, C412, C414, C415, C416, C420: footprint (none) -> Capacitor_SMD:C_0805_2012Metric_Pad1.18x1.45mm_HandSolder
- C407, C421: footprint (none) -> Capacitor_Tantalum_SMD:CP_EIA-3528-21_Kemet-B_Pad1.50x2.35mm_HandSolder
- C413: value 470u/12V -> 33u/12V; footprint (none) -> Capacitor_Tantalum_SMD:CP_EIA-3528-21_Kemet-B_Pad1.50x2.35mm_HandSolder
- D402, D404: footprint (none) -> Diode_SMD:D_SOD-123F
- L403: value 1008PS-222KLB -> SRN3010TA-2R2M
- L407: value DRQ73 -> DRQ73-220-R; footprint (none) -> ETH1LCR3:DRQ73
Connections:
- net +5V: now also C422.1
- net GND: now also C422.2
Other:
- moved on the sheet: C401, C402, C403, C404, C405, C406, C407, C408, C409, C410, C411, C412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

Commit message: PCB layout
Parts:
- L403: footprint (none) -> ETH1LCR3:SRN3010TA
Other:
- moved on the sheet: C420, C421, L408
Changed lines of the file:
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@@
 	)
 	(junction
-		(at 265.43 87.63)
-		(diameter 0)
-		(color 0 0 0 0)
-	)
-	(junction
 		(at 62.23 151.13)
 		(diameter 0)
@@
 	)
 	(junction
+		(at 262.89 87.63)
+		(diameter 0)
+		(color 0 0 0 0)
+	)
+	(junction
 		(at 187.96 87.63)
 		(diameter 0)
@@
 	)
 	(junction
-		(at 265.43 115.57)
+		(at 250.19 87.63)
 		(diameter 0)
 		(color 0 0 0 0)
 	)
 	(junction
-		(at 48.26 74.93)
+		(at 262.89 115.57)
 		(diameter 0)
 		(color 0 0 0 0)
 	)
 	(junction
-		(at 68.58 74.93)
+		(at 48.26 74.93)
 		(diameter 0)
 		(color 0 0 0 0)
 	)
 	(junction
-		(at 85.09 134.62)
+		(at 68.58 74.93)
 		(diameter 0)
 		(color 0 0 0 0)
 	)
 	(junction
-		(at 72.39 172.72)
+		(at 85.09 134.62)
 		(diameter 0)
 		(color 0 0 0 0)
 	)
 	(junction
-		(at 252.73 87.63)
+		(at 72.39 172.72)
 		(diameter 0)
 		(color 0 0 0 0)
@@
 	(wire
 		(pts
-			(xy 265.43 115.57) (xy 265.43 116.84)
+			(xy 262.89 115.57) (xy 262.89 116.84)
 		)
 		(stroke
@@
 	(wire
 		(pts
-			(xy 252.73 115.57) (xy 265.43 115.57)
+			(xy 250.19 115.57) (xy 262.89 115.57)
 		)
 		(stroke
@@
 	(wire
 		(pts
+			(xy 264.16 87.63) (xy 262.89 87.63)
+		)
+		(stroke
+			(width 0)
+			(type default)
+		)
+	)
+	(wire
+		(pts
 			(xy 58.42 83.82) (xy 58.42 86.36)
 		)
@@
 	(wire
 		(pts
-			(xy 252.73 87.63) (xy 246.38 87.63)
+			(xy 110.49 86.36) (xy 110.49 88.9)
 		)
 		(stroke
@@
 	(wire
 		(pts
-			(xy 110.49 86.36) (xy 110.49 88.9)
+			(xy 250.19 87.63) (xy 246.38 87.63)
 		)
 		(stroke
@@
 	(wire
 		(pts
-			(xy 252.73 99.06) (xy 252.73 87.63)
+			(xy 250.19 99.06) (xy 250.19 87.63)
 		)
 		(stroke
@@
 	(wire
 		(pts
-			(xy 265.43 115.57) (xy 265.43 106.68)
+			(xy 262.89 115.57) (xy 262.89 106.68)
 		)
 		(stroke
@@
 	(wire
 		(pts
-			(xy 283.21 87.63) (xy 283.21 86.36)
+			(xy 279.4 87.63) (xy 279.4 86.36)
 		)
 		(stroke
@@
 	(wire
 		(pts
-			(xy 252.73 106.68) (xy 252.73 115.57)
+			(xy 250.19 106.68) (xy 250.19 115.57)
 		)
 		(stroke
@@
 	(wire
 		(pts
-			(xy 265.43 99.06) (xy 265.43 87.63)
+			(xy 262.89 99.06) (xy 262.89 87.63)
 		)
 		(stroke
@@
 	(wire
 		(pts
-			(xy 265.43 87.63) (xy 269.24 87.63)
-		)
-		(stroke
-			(width 0)
-			(type default)
-		)
-	)
-	(wire
-		(pts
 			(xy 184.15 99.06) (xy 184.15 87.63)
 		)
@@
 	(wire
 		(pts
+			(xy 250.19 87.63) (xy 262.89 87.63)
+		)
+		(stroke
+			(width 0)
+			(type default)
+		)
+	)
+	(wire
+		(pts
 			(xy 110.49 76.2) (xy 110.49 74.93)
 		)
@@
 	(wire
 		(pts
-			(xy 276.86 87.63) (xy 283.21 87.63)
+			(xy 271.78 87.63) (xy 279.4 87.63)
 		)
 		(stroke
@@
 	(wire
 		(pts
-			(xy 265.43 87.63) (xy 252.73 87.63)
-		)
-		(stroke
-			(width 0)
-			(type default)
-		)
-	)
-	(wire
-		(pts
 			(xy 205.74 76.2) (xy 198.12 76.2)
 		)
@@
 	(symbol
 		(lib_id "Device:C_Polarized")
-		(at 265.43 102.87 180)
+		(at 262.89 102.87 180)
 		(unit 1)
 		(exclude_from_sim no)
@@
 		(fields_autoplaced yes)
 		(property "Reference" "C421"
-			(at 269.24 102.4889 0)
+			(at 266.7 102.4889 0)
 			(effects
 				(font
@@
 		)
 		(property "Value" "33u/12V"
-			(at 269.24 105.0289 0)
+			(at 266.7 105.0289 0)
 			(effects
 				(font
@@
 		)
 		(property "Footprint" "Capacitor_Tantalum_SMD:CP_EIA-3528-21_Kemet-B_Pad1.50x2.35mm_HandSolder"
-			(at 264.4648 99.06 0)
+			(at 261.9248 99.06 0)
 			(effects
 				(font
@@
 		)
 		(property "Datasheet" "~"
-			(at 265.43 102.87 0)
+			(at 262.89 102.87 0)
 			(effects
 				(font
@@
 		)
 		(property "Description" "Polarized capacitor"
-			(at 265.43 102.87 0)
+			(at 262.89 102.87 0)
 			(effects
 				(font
@@
 	(symbol
 		(lib_id "power:-5V")
-		(at 283.21 86.36 0)
+		(at 279.4 86.36 0)
 		(unit 1)
 		(exclude_from_sim no)
@@
 		(fields_autoplaced yes)
 		(property "Reference" "#PWR0427"
-			(at 283.21 90.17 0)
+			(at 279.4 90.17 0)
 			(effects
 				(font
@@
 		)
 		(property "Value" "-5V"
-			(at 283.21 81.28 0)
+			(at 279.4 81.28 0)
 			(effects
 				(font
@@
 		)
 		(property "Footprint" ""
-			(at 283.21 86.36 0)
+			(at 279.4 86.36 0)
 			(effects
 				(font
@@
 		)
 		(property "Datasheet" ""
-			(at 283.21 86.36 0)
+			(at 279.4 86.36 0)
 			(effects
 				(font
@@
 		)
 		(property "Description" "Power symbol creates a global label with name \"-5V\""
-			(at 283.21 86.36 0)
+			(at 279.4 86.36 0)
 			(effects
 				(font
@@
 		(pin "2"
 		)
+		(pin "11"
+		)
 		(instances
 			(project ""
@@
 			)
 		)
-		(property "Footprint" ""
+		(property "Footprint" "ETH1LCR3:SRN3010TA"
 			(at 90.17 74.93 0)
 			(effects
@@
 	(symbol
 		(lib_id "Device:L")
-		(at 273.05 87.63 90)
+		(at 267.97 87.63 90)
 		(unit 1)
 		(exclude_from_sim no)
@@
 		(fields_autoplaced yes)
 		(property "Reference" "L408"
-			(at 273.05 82.55 90)
+			(at 267.97 82.55 90)
 			(effects
 				(font
@@
 		)
 		(property "Value" "MLZ2012M100WT"
-			(at 273.05 85.09 90)
+			(at 267.97 85.09 90)
 			(effects
 				(font
@@
 		)
 		(property "Footprint" "Inductor_SMD:L_0805_2012Metric_Pad1.05x1.20mm_HandSolder"
-			(at 273.05 87.63 0)
+			(at 267.97 87.63 0)
 			(effects
 				(font
@@
 		)
 		(property "Datasheet" "~"
-			(at 273.05 87.63 0)
+			(at 267.97 87.63 0)
 			(effects
 				(font
@@
 		)
 		(property "Description" "Inductor"
-			(at 273.05 87.63 0)
+			(at 267.97 87.63 0)
 			(effects
 				(font
@@
 	(symbol
 		(lib_id "power:GND")
-		(at 265.43 116.84 0)
+		(at 262.89 116.84 0)
 		(unit 1)
 		(exclude_from_sim no)
@@
 		(fields_autoplaced yes)
 		(property "Reference" "#PWR0426"
-			(at 265.43 123.19 0)
+			(at 262.89 123.19 0)
 			(effects
 				(font
@@
 		)
 		(property "Value" "GND"
-			(at 265.43 121.92 0)
+			(at 262.89 121.92 0)
 			(effects
 				(font
@@
 		)
 		(property "Footprint" ""
-			(at 265.43 116.84 0)
+			(at 262.89 116.84 0)
 			(effects
 				(font
@@
 		)
 		(property "Datasheet" ""
-			(at 265.43 116.84 0)
+			(at 262.89 116.84 0)
 			(effects
 				(font
@@
 		)
 		(property "Description" "Power symbol creates a global label with name \"GND\" , ground"
-			(at 265.43 116.84 0)
+			(at 262.89 116.84 0)
 			(effects
 				(font
@@
 	(symbol
 		(lib_id "Device:C")
-		(at 252.73 102.87 0)
+		(at 250.19 102.87 0)
 		(unit 1)
 		(exclude_from_sim no)
@@
 		(dnp no)
 		(property "Reference" "C420"
-			(at 256.54 101.5999 0)
+			(at 254 101.5999 0)
 			(effects
 				(font
@@
 		)
 		(property "Value" "4u7"
-			(at 256.54 104.1399 0)
+			(at 254 104.1399 0)
 			(effects
 				(font
@@
 		)
 		(property "Footprint" "Capacitor_SMD:C_0805_2012Metric_Pad1.18x1.45mm_HandSolder"
-			(at 253.6952 106.68 0)
+			(at 251.1552 106.68 0)
 			(effects
 				(font
@@
 		)
 		(property "Datasheet" "~"
-			(at 252.73 102.87 0)
+			(at 250.19 102.87 0)
 			(effects
 				(font
@@
 		)
 		(property "Description" "Unpolarized capacitor"
-			(at 252.73 102.87 0)
+			(at 250.19 102.87 0)
 			(effects
 				(font

Commit message: PCB layout
Parts:
- renumbered C403 to C402, C409 to C403, C402 to C404, C410 to C405, C404 to C406, C411 to C407, C405 to C408, C406 to C409, C408 to C410, C413 to C411, C407 to C412, C422 to C413, C412 to C414, C414 to C415, C415 to C417, C417 to C418, C418 to C419, C419 to C420, C420 to C421, C421 to C422, L402 to L401, L404 to L402, L401 to L403, L403 to L404, R410 to R409, R409 to R410, U403 to U401, U401 to U402, U402 to U403
