File: Hardware/ETH1LCR3/Power.kicad_sch (KiCad schematic)
At the start: 58 parts, among them Q401 SI5618A, Q402 MMBT3904, Q403 BSS123, U401 REG103GA-5, U402 REG103GA-3.3, U403 LT1946A, U404 TEL5-2411, U405 LT1611

Commit message: PCB layout
Parts:
- C419: footprint Capacitor_SMD:C_0603_1608Metric_Pad1.08x0.95mm_HandSolder -> Capacitor_SMD:C_0805_2012Metric_Pad1.18x1.45mm_HandSolder
Changed lines of the file:
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@@
 			)
 		)
-		(property "Footprint" "Capacitor_SMD:C_0603_1608Metric_Pad1.08x0.95mm_HandSolder"
+		(property "Footprint" "Capacitor_SMD:C_0805_2012Metric_Pad1.18x1.45mm_HandSolder"
 			(at 232.41 86.6648 0)
 			(effects

Commit message: Updated project to KiCAD 9
Changed lines of the file:
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@@
 (kicad_sch
-	(version 20231120)
+	(version 20250114)
 	(generator "eeschema")
-	(generator_version "8.0")
+	(generator_version "9.0")
 	(paper "A4")
 	(junction
@@
 		(shape input)
 		(at 147.32 63.5 0)
-		(fields_autoplaced yes)
 		(effects
 			(font
@@
 		(shape input)
 		(at 139.7 102.87 0)
-		(fields_autoplaced yes)
 		(effects
 			(font
