File: Hardware/ETH1LCR3/ETH1LCR3.kicad_pcb (KiCad board)
At the start: 2 copper layers, 472 parts, among them J301 20021111-00010T4LF, K1401 G5V-2-DC5, K1402 G5V-2-DC5, K801 UMS05-1A80-75D, K802 UMS05-1A80-75D, K803 UMS05-1A80-75D, K804 UMS05-1A80-75D, K805 UMS05-1A80-75D, Q1001 BSS123, Q1101 BSS123, Q1201 BSS123, Q1401 MMBT3904, Q1402 MMBT3904, Q401 SI5618A, Q402 MMBT3904, Q403 BSS123, Q801 MMBT3904, Q802 MMBT3904, Q803 MMBT3904, Q804 MMBT3904, Q805 BFR106, Q806 MMBT3904, Q807 BFR106, Q901 BSS123, U1001 AQY221R2S, U1002 AD8099ARDZ, U1003 AQY221R2S, U1101 AQY221R2S, U1102 AD8099ARDZ, U1103 AQY221R2S, U1201 AQY221R2S, U1202 AD8099ARDZ, U1203 AQY221R2S, U1601 TXB0104PW, U1602 ADuM5402, U1603 74AC125, U201 LAN8742A, U202 SRV05-4, U301 SN74LV1T34DBV, U302 74LVC1G74DP, U303 STM32H743VITx, U304 24LC08B-E/MS, U305 REF2033, U401 REG103GA-3.3, U402 LT1946A, U403 REG103GA-5, U404 TEL5-2411, U405 LT1611, U501 SN74LVC1G04DBV, U502 AD9834, U503 AD9834, U504 SN74LV1T34DBV, U505 LMH6644MT, U506 TLV3501AIDBV, U507 74LVC1G74DP, U601 LMH6618MK, U602 ADG1604BRUZ, U603 LMH6720MA, U604 LMH6720MA, U605 LMH6720MA, U701 LMH6618MK, U702 TLV3501AIDBV, U703 74HCT4051PW, U704 SN74LVC1G3157DB, U705 SN74LVC1G3157DB, U706 SN74LV1T34DBV, U707 SN74LV1T34DBV, U708 SN74LV1T34DBV, U709 ADS1246IPWR, U710 REF2025, U801 74LVC1G3157DB, U802 LMH6644MT, U803 OPA2727AID, U804 AQY221R2S, U805 AQY221R2S, U806 SN74LV1T34DBV, U807 SN74LV1T34DBV, U808 SN74LV1T34DBV, U901 AQY221R2S, U902 AD8099ARDZ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

Commit message: Hardware
Parts:
- removed H101, H102, H103, H104: MountingHole, MountingHole:MountingHole_3.2mm_M3_DIN965_Pad
- added C1501: 1u, Capacitor_SMD:C_0603_1608Metric_Pad1.08x0.95mm_HandSolder, F.Cu at (-274.1, 78.1)
- added C213: 1n/1kV, Capacitor_SMD:C_1206_3216Metric_Pad1.33x1.80mm_HandSolder, F.Cu at (-270.9, 155.6)
- added C401: 4u7, Capacitor_SMD:C_0805_2012Metric_Pad1.18x1.45mm_HandSolder, F.Cu at (-226.9, 134.3)
- added C402: 2u2, Capacitor_SMD:C_0805_2012Metric_Pad1.18x1.45mm_HandSolder, F.Cu at (-226.9, 137.4)
- added C403: 2u2, Capacitor_SMD:C_0805_2012Metric_Pad1.18x1.45mm_HandSolder, F.Cu at (-226.9, 140.4)
- added C407: 33u/12V, Capacitor_Tantalum_SMD:CP_EIA-3528-21_Kemet-B_Pad1.50x2.35mm_HandSolder, F.Cu at (-221.3, 147.1)
- added C409: 2u2, Capacitor_SMD:C_0805_2012Metric_Pad1.18x1.45mm_HandSolder, F.Cu at (-226.9, 143.4)
- added C411: 2u2, Capacitor_SMD:C_0805_2012Metric_Pad1.18x1.45mm_HandSolder, F.Cu at (-226.9, 146.4)
- added C412: 4u7, Capacitor_SMD:C_0805_2012Metric_Pad1.18x1.45mm_HandSolder, F.Cu at (-226.9, 149.4)
- added C413: 33u/12V, Capacitor_Tantalum_SMD:CP_EIA-3528-21_Kemet-B_Pad1.50x2.35mm_HandSolder, F.Cu at (-221.3, 151.4)
- added C414: 4u7, Capacitor_SMD:C_0805_2012Metric_Pad1.18x1.45mm_HandSolder, F.Cu at (-226.9, 152.4)
- added C420: 4u7, Capacitor_SMD:C_0805_2012Metric_Pad1.18x1.45mm_HandSolder, F.Cu at (-226.9, 155.4)
- added C421: 33u/12V, Capacitor_Tantalum_SMD:CP_EIA-3528-21_Kemet-B_Pad1.50x2.35mm_HandSolder, F.Cu at (-221.3, 155.8)
- added C422: 470u/12V, Capacitor_SMD:CP_Elec_10x10.5, F.Cu at (-217.1, 138.9)
- added C523: 4u7, Capacitor_SMD:C_0805_2012Metric_Pad1.18x1.45mm_HandSolder, F.Cu at (-286.6, 150.8)
- added C525: 4u7, Capacitor_SMD:C_0805_2012Metric_Pad1.18x1.45mm_HandSolder, F.Cu at (-286.6, 153.8)
- added C603: JZ200, Capacitor_SMD:C_Trimmer_Voltronics_JZ, F.Cu at (-279.0, 151.6)
- added C607: JZ200, Capacitor_SMD:C_Trimmer_Voltronics_JZ, F.Cu at (-279.0, 156.4)
- added C717: 100n/C0G, Capacitor_SMD:C_1206_3216Metric_Pad1.33x1.80mm_HandSolder, F.Cu at (-203.6, 134.5)
- added C720: 100n/C0G, Capacitor_SMD:C_1206_3216Metric_Pad1.33x1.80mm_HandSolder, F.Cu at (-203.6, 137.9)
- added C721: 100n/C0G, Capacitor_SMD:C_1206_3216Metric_Pad1.33x1.80mm_HandSolder, F.Cu at (-203.6, 141.2)
- added C725: 4u7, Capacitor_SMD:C_0805_2012Metric_Pad1.18x1.45mm_HandSolder, F.Cu at (-204.2, 144.4)
- added C810: 4u7, Capacitor_SMD:C_0805_2012Metric_Pad1.18x1.45mm_HandSolder, F.Cu at (-204.2, 149.9)
- added C811: 4u7, Capacitor_SMD:C_0805_2012Metric_Pad1.18x1.45mm_HandSolder, F.Cu at (-204.2, 153.0)
- added C813: JZ100, Capacitor_SMD:C_Trimmer_Voltronics_JZ, F.Cu at (-198.7, 156.9)
- added C814: 4u7, Capacitor_SMD:C_0805_2012Metric_Pad1.18x1.45mm_HandSolder, F.Cu at (-204.2, 156.0)
- added D404: MBR0520, Diode_SMD:D_SOD-123F, F.Cu at (-215.4, 155.8)
- added D701: NSVRB751V40T1G, Diode_SMD:D_SOD-323_HandSoldering, F.Cu at (-198.1, 134.3)
- added D702: NSVRB751V40T1G, Diode_SMD:D_SOD-323_HandSoldering, F.Cu at (-198.1, 137.3)
- added D703: NSVRB751V40T1G, Diode_SMD:D_SOD-323_HandSoldering, F.Cu at (-198.1, 140.2)
- added HS101: Heatsink, ETH1LCR3:960-19-12-S-AB-0, F.Cu at (167.0, 115.0)
- added J1301: 5227161-1, ETH1LCR3:TE_5227161-1, F.Cu at (-288.4, 139.5)
- added J1302: 5227161-1, ETH1LCR3:TE_5227161-1, F.Cu at (-272.1, 139.5)
- added J1303: 5227161-1, ETH1LCR3:TE_5227161-1, F.Cu at (-255.8, 139.5)
- added J1304: 5227161-1, ETH1LCR3:TE_5227161-1, F.Cu at (77.9, 65.0)
- added J1501: DIN41612_02x32_AC, ETH1LCR3:Socket_DIN41612-CaseC1-AC-Male-64Pin-2rows, F.Cu at (183.6, 78.9)
- added K1501: HE3621A0510, ETH1LCR3:HE360_x-5050462-8, F.Cu at (206.0, 64.0)
- added K1502: HE3621A0510, ETH1LCR3:HE360_x-5050462-8, F.Cu at (-286.4, 79.7)
- added K1503: HE3621A0510, ETH1LCR3:HE360_x-5050462-8, F.Cu at (-286.4, 86.0)
- added K1504: HE3621A0510, ETH1LCR3:HE360_x-5050462-8, F.Cu at (-286.4, 92.3)
- added K1505: HE3621A0510, ETH1LCR3:HE360_x-5050462-8, F.Cu at (-286.4, 98.7)
- added K1506: HE3621A0510, ETH1LCR3:HE360_x-5050462-8, F.Cu at (-286.4, 105.0)
- added L1601: CW252016-R33G, ETH1LCR3:CW252016, F.Cu at (121.9, 69.0)
- added L407: DRQ73-220-R, ETH1LCR3:DRQ73, F.Cu at (-213.4, 149.5)
- added R324: 0, Resistor_SMD:R_0603_1608Metric_Pad0.98x0.95mm_HandSolder, F.Cu at (-262.2, 155.2)
- added RN701: 51, Resistor_SMD:R_Array_Convex_2x0603, F.Cu at (-194.4, 143.3)
- added RN702: 51, Resistor_SMD:R_Array_Convex_4x0603, F.Cu at (-198.6, 144.1)
- added RV501: TS53YJ103MR10, Potentiometer_SMD:Potentiometer_Vishay_TS53YJ_Vertical, F.Cu at (-292.8, 152.5)
- added RV801: 3266W-1-500LF, Potentiometer_THT:Potentiometer_Bourns_3266W_Vertical, F.Cu at (-195.2, 150.3)
- added U1501: ULN2003A, Package_SO:TSSOP-16_4.4x5mm_P0.65mm, F.Cu at (-271.5, 73.5)
- added Y201: NX5032GA-25, ETH1LCR3:NX5032GA, F.Cu at (-270.1, 151.6)
- added Y301: NX5032GA-16, ETH1LCR3:NX5032GA, F.Cu at (-260.7, 151.6)
- C1601, C1603, C1604, C1606, C1608: value 100n -> 0.1u
- C214: value 0.1u -> 1n/1kV; footprint Capacitor_SMD:C_0603_1608Metric_Pad1.08x0.95mm_HandSolder -> Capacitor_SMD:C_1206_3216Metric_Pad1.33x1.80mm_HandSolder
- C405: value 270p -> 2u2; footprint Capacitor_SMD:C_0603_1608Metric_Pad1.08x0.95mm_HandSolder -> Capacitor_SMD:C_0805_2012Metric_Pad1.18x1.45mm_HandSolder
- C415, C729: value 1u -> 4u7; footprint Capacitor_SMD:C_0603_1608Metric_Pad1.08x0.95mm_HandSolder -> Capacitor_SMD:C_0805_2012Metric_Pad1.18x1.45mm_HandSolder
- C416: value 1u -> 2u2; footprint Capacitor_SMD:C_0603_1608Metric_Pad1.08x0.95mm_HandSolder -> Capacitor_SMD:C_0805_2012Metric_Pad1.18x1.45mm_HandSolder
- C718: value 0.1u -> 100n/C0G; footprint Capacitor_SMD:C_0603_1608Metric_Pad1.08x0.95mm_HandSolder -> Capacitor_SMD:C_1206_3216Metric_Pad1.33x1.80mm_HandSolder
- C723: value 1u -> 15p/C0G
- C724: value 0.1u -> 15p/C0G
- C726: value 0.1u -> 4u7; footprint Capacitor_SMD:C_0603_1608Metric_Pad1.08x0.95mm_HandSolder -> Capacitor_SMD:C_0805_2012Metric_Pad1.18x1.45mm_HandSolder
- D402: value BZX84C10LT1G -> MBR0520; footprint Package_TO_SOT_SMD:SOT-23 -> Diode_SMD:D_SOD-123F
- R303: value 1k -> 51
- U803: footprint Package_SO:SOP-4_3.8x4.1mm_P2.54mm -> Package_SO:SOIC-8_3.9x4.9mm_P1.27mm
- U804, U805: footprint Package_TO_SOT_SMD:SOT-23-5 -> Package_SO:SOP-4_3.8x4.1mm_P2.54mm
- U806: footprint Package_SO:SOIC-8_3.9x4.9mm_P1.27mm -> Package_TO_SOT_SMD:SOT-23-5
- U807: footprint Package_SO:SOP-4_3.8x4.1mm_P2.54mm -> Package_TO_SOT_SMD:SOT-23-5
- moved C1001 221.8 mm to (-141.5, 114.9)
- moved C1002 221.8 mm to (-141.5, 117.4)
- moved C1003 221.8 mm to (-141.5, 119.9)
- moved C1004 221.8 mm to (-141.5, 122.4)
- moved C701 221.8 mm to (-76.9, 32.2)
- moved C702 221.8 mm to (-76.9, 34.8)
- moved C703 221.8 mm to (-76.9, 37.3)
- moved C704 221.8 mm to (-76.9, 39.8)
- moved C705 221.8 mm to (-76.9, 42.3)
- moved C706 221.8 mm to (-76.9, 44.8)
- moved C707 221.8 mm to (-76.9, 47.3)
- moved C708 221.8 mm to (-76.9, 49.8)
- moved C709 221.8 mm to (-76.9, 52.3)
- moved C710 221.8 mm to (-76.9, 54.8)
- moved C711 221.8 mm to (-72.6, 32.2)
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Connections:
- net /Ethernet PoE/ETH_RXN renamed /Ethernet/ETH_RXN
- net /Ethernet PoE/ETH_RXP renamed /Ethernet/ETH_RXP
- net /Ethernet PoE/ETH_TXN renamed /Ethernet/ETH_TXN
- net /Ethernet PoE/ETH_TXP renamed /Ethernet/ETH_TXP
- net /Ethernet PoE/LED1 renamed /Ethernet/LED1
- net /Ethernet PoE/LED2 renamed /Ethernet/LED2
- net /Ethernet PoE/MODE0 renamed /Ethernet/MODE0
- net /Ethernet PoE/MODE1 renamed /Ethernet/MODE1
- net /Ethernet PoE/MODE2 renamed /Ethernet/MODE2
- net /Ethernet PoE/REFCLK0 renamed /Ethernet/REFCLK0
- net /Ethernet PoE/REF_CLK renamed /Ethernet/REF_CLK
- net /Ethernet PoE/RMII_CRS_DV renamed /Ethernet/RMII_CRS_DV
- net /Ethernet PoE/RMII_MDC renamed /Ethernet/RMII_MDC
- net /Ethernet PoE/RMII_MDIO renamed /Ethernet/RMII_MDIO
- net /Ethernet PoE/RMII_RXD0 renamed /Ethernet/RMII_RXD0
- net /Ethernet PoE/RMII_RXD1 renamed /Ethernet/RMII_RXD1
- net /Ethernet PoE/RMII_TXD0 renamed /Ethernet/RMII_TXD0
- net /Ethernet PoE/RMII_TXD1 renamed /Ethernet/RMII_TXD1
- net /Ethernet PoE/RMII_TXEN renamed /Ethernet/RMII_TXEN
- C1601 pad 1: +3V3 -> +3.3V
- C1602 pad 1: +3V3 -> +3.3V
- C214 pad 1: VCCQ -> Net-(C214-Pad1)
- C214 pad 2: GND -> Earth
- C405 pad 1: Net-(C405-Pad1) -> +3.3V
- C415 pad 1: Net-(U405-~{SHDN}) -> Net-(U405-VIN)
- C416 pad 1: Net-(U405-SW1) -> +5VP
- C416 pad 2: Net-(D404-A) -> GND
- C718 pad 1: -5V -> Net-(C718-Pad1)
- C723 pad 1: +5V -> GND
- C723 pad 2: GND -> Net-(U709-AINP)
- C724 pad 1: +5V -> Net-(U709-AINN)
- C726 pad 1: +2V5 -> GND
- C726 pad 2: GND -> Net-(U709-DVDD)
- C729 pad 1: +1V25 -> Net-(U709-AVDD)
- D401 pad 3: VIN+ -> Net-(D401-K)
- D402 pad 1: Net-(D402-A) -> V_BOOST
- D402 pad 2: unconnected-(D402-NC-Pad2) -> Net-(D402-A)
- D403 pad 2: VIN+ -> Net-(D401-K)
- Q401 pad 2: VIN+ -> Net-(D401-K)
- Q402 pad 2: VIN+ -> Net-(D401-K)
- R1601 pad 1: +3V3 -> +3.3V
- R303 pad 1: Net-(U303-Q) -> /MCU/SYNCH_CDE
- R303 pad 2: /MCU/SYNCH_OUT -> Net-(U301-A)
- U1601 pad 1: +3V3 -> +3.3V
- U303 pad 87: unconnected-(U303-PD6-Pad87) -> /Connector/CXN_REL1
- U303 pad 88: unconnected-(U303-PD7-Pad88) -> /Connector/CXN_REL2
- U303 pad 89: unconnected-(U303-PB3-Pad89) -> /Connector/CXN_REL3
- U303 pad 90: unconnected-(U303-PB4-Pad90) -> /Connector/CXN_REL4
- U303 pad 95: unconnected-(U303-PB8-Pad95) -> /Connector/CXN_REL5
- U303 pad 96: unconnected-(U303-PB9-Pad96) -> /Connector/CXN_REL6
- U404 pad 11: unconnected-(U404-NC-Pad11) -> (no net)
- U404 pad 22: VIN+ -> Net-(D401-K)
- U404 pad 23: VIN+ -> Net-(D401-K)
Other:
- board outline added: 160 x 100 mm

Commit message: Hardware
Parts:
- added C1502: 0.1u, Capacitor_SMD:C_0603_1608Metric_Pad1.08x0.95mm_HandSolder, F.Cu at (179.6, 81.0)
- added C1503: 0.1u, Capacitor_SMD:C_0603_1608Metric_Pad1.08x0.95mm_HandSolder, F.Cu at (179.6, 83.5)
- added R1501: 1k, Resistor_SMD:R_0603_1608Metric_Pad0.98x0.95mm_HandSolder, F.Cu at (191.6, 70.4)
- added R1502: 51, Resistor_SMD:R_0603_1608Metric_Pad0.98x0.95mm_HandSolder, F.Cu at (188.8, 82.8)
- added R1503: 51, Resistor_SMD:R_0603_1608Metric_Pad0.98x0.95mm_HandSolder, F.Cu at (184.7, 82.4)
- added U1502: LMH6644MT, Package_SO:TSSOP-14_4.4x5mm_P0.65mm, F.Cu at (190.4, 75.4)
- C1609, C213, C214, C414, C416, F401, R207, RN202, RN203: moved to B.Cu
- moved K1506 491.3 mm to (203.7, 70.4)
- moved K1505 491.3 mm to (203.7, 65.2)
- moved K1502 490.5 mm to (203.7, 59.9)
- moved K1504 490.3 mm to (203.7, 80.8)
- moved K1503 490.2 mm to (203.7, 75.6)
- moved C213 478.3 mm to (204.9, 105.7), turned to 180 degrees
- moved Y201 466.3 mm to (193.8, 105.2), turned to 180 degrees
- moved U1501 451.8 mm to (180.0, 89.9)
- moved C414 394.4 mm to (166.9, 131.6), turned to 180 degrees
- moved J1301 366.4 mm to (78.0, 138.1), turned to 90 degrees
- moved R406 355.5 mm to (213.4, 122.2), turned to 90 degrees
- moved C201 354.1 mm to (239.8, 98.8)
- moved C202 354.1 mm to (239.8, 101.3)
- moved C203 354.1 mm to (239.8, 103.8)
- moved C204 354.1 mm to (239.8, 106.4)
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Connections:
- K1502 pad 1: /Connector/HS_REAR -> /Connector/LD_REAR
- K1504 pad 1: /Connector/LD_REAR -> /Connector/HS_REAR
- K1506 pad 1: unconnected-(K1506-Pad1) -> Net-(K1506-Pad1)
Other:
- outline, holes or cut-outs redrawn

Commit message: PCB layout
Parts:
- added L403: SRN3010TA-2R2M, ETH1LCR3:SRN3010TA, F.Cu at (169.4, 144.7)
- added R625: 51, Resistor_SMD:R_0603_1608Metric_Pad0.98x0.95mm_HandSolder, F.Cu at (103.4, 99.5)
- added R626: 51, Resistor_SMD:R_0603_1608Metric_Pad0.98x0.95mm_HandSolder, F.Cu at (103.4, 102.0)
- C1203: value DNP -> 1p
- C201, C203, C204, C404, C419, L405, R208, R209, R404, R408, R412, R415, U304: moved to B.Cu
- U301, U504, U706, U707, U708, U806, U807, U808: footprint Package_TO_SOT_SMD:SOT-23-5 -> Package_TO_SOT_SMD:SOT-23-5_HandSoldering
- U506, U702: footprint Package_TO_SOT_SMD:SOT-23-6 -> Package_TO_SOT_SMD:SOT-23-6_Handsoldering
- U601: value LMH6618MK -> LMH6618MKE; footprint Package_TO_SOT_SMD:TSOT-23-6 -> Package_TO_SOT_SMD:SOT-23-6_Handsoldering
- U603, U604, U605: value LMH6720MA -> LMH6720MF
- U701: value LMH6618MK -> LMH6618MKE; footprint Package_TO_SOT_SMD:TSOT-23-6_HandSoldering -> Package_TO_SOT_SMD:SOT-23-6_Handsoldering
- moved C401 400.6 mm to (173.6, 139.7)
- moved C403 400.5 mm to (173.6, 142.1)
- moved C402 394.7 mm to (167.8, 133.3), turned to 180 degrees
- moved C407 387.2 mm to (165.5, 129.4), turned to -90 degrees
- moved C412 386.7 mm to (159.8, 145.8), turned to 180 degrees
- moved C409 381.9 mm to (154.8, 133.2), turned to 180 degrees
- moved C411 380.0 mm to (152.4, 124.5), turned to 90 degrees
- moved C413 374.4 mm to (152.4, 129.4), turned to -90 degrees
- moved C422 359.1 mm to (141.7, 126.4), turned to 180 degrees
- moved C420 358.9 mm to (131.8, 143.9), turned to -90 degrees
- moved D404 357.8 mm to (141.7, 134.5), turned to 180 degrees
- moved R410 357.5 mm to (215.4, 132.1)
- moved C421 352.0 mm to (130.3, 139.1), turned to -90 degrees
- moved L407 350.9 mm to (137.4, 141.1), turned to -90 degrees
- moved D403 329.8 mm to (210.9, 135.5), turned to -90 degrees
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Connections:
- U404 pad 11: (no net) -> unconnected-(U404-NC-Pad11)
- U602 pad 1: /MCU/PGA_A0 -> Net-(U602-A0)
- U602 pad 14: /MCU/PGA_G1 -> Net-(U602-A1)

Commit message: PCB layout
Parts:
- added C313: 0.1u, Capacitor_SMD:C_0603_1608Metric_Pad1.08x0.95mm_HandSolder, F.Cu at (154.1, 110.7)
- C1501: renamed from C1502; moved to B.Cu
- C1502: renamed from C1503; moved to B.Cu
- C1503: renamed from C1501; moved to B.Cu
- C1601, C1602, C1603, C1604, C1605, C1606, C1607, C1608, C202, C205, C209, C210, C211, C212, C301, C302, C303, C304, C305, C306, C307, C308, C309, C310, D1402, FB301, Q1402, R1402, R1601, R1604, R1606, R202, R203, R204, R205, R206, R301, R304, R305, R306, R309, R310, R316, R318, R401, Y301: moved to B.Cu
- C311: renamed from C312; moved to B.Cu
- C312: renamed from C313; moved to B.Cu
- C314: renamed from C311; moved to B.Cu
- C315: renamed from C314; moved to B.Cu
- C316: renamed from C315; moved to B.Cu
- C317: renamed from C316; moved to B.Cu
- C318: renamed from C317; moved to B.Cu
- C319: renamed from C318; moved to B.Cu
- C320: renamed from C319; moved to B.Cu
- C321: renamed from C320; moved to B.Cu
- C405: renamed from C410; moved to B.Cu
- R312: renamed from R311; moved to B.Cu
- R313: renamed from R312; moved to B.Cu
- R319: renamed from R324; moved to B.Cu
- R320: renamed from R319; moved to B.Cu
- R323: renamed from R322; moved to B.Cu
- R324: renamed from R323; moved to B.Cu
- moved C1503 454.2 mm to (180.0, 91.7), turned to 180 degrees
- moved C524 446.3 mm to (141.3, 24.3)
- moved C525 446.3 mm to (141.3, 27.3)
- moved RV501 446.3 mm to (135.1, 26.0)
- moved Y301 428.4 mm to (165.2, 105.0), turned to 180 degrees
- moved R319 418.9 mm to (154.1, 108.3)
- moved C603 378.9 mm to (99.7, 161.0)
- moved C607 378.9 mm to (99.7, 165.7)
- moved RN701 344.6 mm to (144.7, 113.8)
- moved D301 343.3 mm to (188.2, 119.3), turned to -90 degrees
- moved C301 342.6 mm to (173.0, 116.8)
- moved C311 340.7 mm to (179.1, 110.7)
- moved RN702 340.2 mm to (144.7, 116.7), turned to 180 degrees
- moved C302 337.4 mm to (172.5, 104.1), turned to -90 degrees
- moved R310 336.0 mm to (184.8, 101.7), turned to 90 degrees
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- renumbered C403 to C402, C409 to C403, C402 to C404, C404 to C406, C411 to C407, C405 to C408, C406 to C409, C408 to C410, C413 to C411, C407 to C412, C422 to C413, C412 to C414, C414 to C415, C415 to C417, C417 to C418, C418 to C419, C419 to C420, C420 to C421, C421 to C422, C524 to C523, C523 to C524, L402 to L401, L404 to L402, L401 to L403, L403 to L404, R1502 to R1501, R1503 to R1502, R1501 to R1503, R314 to R311, R313 to R314, R320 to R321, R321 to R322, R410 to R409, R409 to R410, R625 to R602, R626 to R603, R602 to R604, R603 to R605, R604 to R606, R605 to R607, R606 to R608, R607 to R609, R608 to R610, R609 to R611, R610 to R612, R611 to R613, R612 to R614, R613 to R615, R614 to R616, R615 to R617, R616 to R618, R617 to R619, R618 to R620, R619 to R621, R620 to R622, R621 to R623, R622 to R624, R623 to R625, R624 to R626, R824 to R823, R825 to R824, R823 to R825, RN702 to RN701, RN701 to RN702, U1502 to U1501, U1501 to U1502, U403 to U401, U401 to U402, U402 to U403

Commit message: PCB layout
Parts:
- added C806: 0.1u, Capacitor_SMD:C_0603_1608Metric_Pad1.08x0.95mm_HandSolder, B.Cu at (111.4, 87.4)
- added C809: 0.1u, Capacitor_SMD:C_0603_1608Metric_Pad1.08x0.95mm_HandSolder, B.Cu at (90.6, 60.2)
- added R823: 100k, Resistor_SMD:R_0603_1608Metric_Pad0.98x0.95mm_HandSolder, F.Cu at (109.9, 145.9)
- added U804: OPA727AIDG, Package_SO:MSOP-8_3x3mm_P0.65mm, F.Cu at (105.8, 142.9)
- C1001, C1002, C1003, C1006, C1101, C1102, C1103, C1106, C1201, C1202, C1203, C1206, C502, C503, C504, C505, C506, C507, C508, C510, C511, C517, C518, C601, C604, C605, C606, C608, C609, C610, C611, C612, C613, C615, C617, C618, C708, C709, C710, C711, C712, C713, C714, C715, C716, C719, C722, C801, C802, C803, C804, C805, C901, C902, C903, C906, D1401, D801, D803, Q1401, Q806, R1401, R621, R724, R809, R815: moved to B.Cu
- C807: renamed from C806; moved to B.Cu
- C808: renamed from C807; moved to B.Cu
- C810: renamed from C808; moved to B.Cu
- Q805, Q807: footprint Package_TO_SOT_SMD:SOT-23_Handsoldering -> Package_TO_SOT_SMD:SOT-23
- U803: value OPA2727AID -> OPA727AIDG; footprint Package_SO:SOIC-8_3.9x4.9mm_P1.27mm -> Package_SO:MSOP-8_3x3mm_P0.65mm
- moved K804 327.2 mm to (176.8, 57.0)
- moved R807 320.0 mm to (182.6, 61.5), turned to 90 degrees
- moved K803 315.7 mm to (165.2, 57.0)
- moved C815 313.2 mm to (113.5, 131.4), turned to 90 degrees
- moved R808 312.7 mm to (175.4, 61.5), turned to -90 degrees
- moved C813 312.1 mm to (92.7, 56.9), turned to 180 degrees
- moved C816 310.2 mm to (105.8, 145.9), turned to 180 degrees
- moved R805 308.5 mm to (170.9, 61.5), turned to 90 degrees
- moved C812 305.7 mm to (90.6, 69.0), turned to -90 degrees
- moved K802 305.0 mm to (154.2, 57.0)
- moved RV801 304.3 mm to (108.4, 130.1)
- moved R806 301.2 mm to (163.7, 61.5), turned to -90 degrees
- moved R803 298.0 mm to (160.2, 61.5), turned to 90 degrees
- moved Q804 294.7 mm to (179.1, 61.5)
- moved R804 290.6 mm to (152.9, 61.5), turned to -90 degrees
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- renumbered C809 to C811, C810 to C812, C811 to C813, C812 to C814, C813 to C815, C814 to C816, C815 to C817, C816 to C818, C817 to C819, R822 to R821, R821 to R822, R823 to R824, R824 to R825, R825 to R826, R826 to R827, R827 to R828, R828 to R829, R829 to R830, R830 to R831, R831 to R832, R832 to R833, R833 to R834, R834 to R835, R835 to R836, R836 to R837, U804 to U805, U805 to U806, U806 to U807, U807 to U808, U808 to U809
Connections:
- C813 pad 1: Net-(C811-Pad1) -> Net-(C813-Pad1)
- C816 pad 1: Net-(U802C-+) -> Net-(C816-Pad1)
- C816 pad 2: Net-(U803B--) -> Net-(U804--)
- R811 pad 2: Net-(C811-Pad1) -> Net-(C813-Pad1)
- R827 pad 1: Net-(U803B--) -> Net-(U804--)
- U803 pad 1: Net-(C811-Pad1) -> unconnected-(U803-NC-Pad1)
- U803 pad 5: GND -> unconnected-(U803-NC-Pad5)
- U803 pad 6: Net-(U803B--) -> Net-(C813-Pad1)
- U803 pad 7: Net-(U802C-+) -> +5V
- U803 pad 8: +5V -> unconnected-(U803-NC-Pad8)
