File: Hardware/ETH1LCR3/ETH1LCR3.kicad_pcb (KiCad board)
At the start: 2 copper layers, 160 x 100 mm, 534 parts, among them J1301 5227161-1, J1302 5227161-1, J1303 5227161-1, J1304 5227161-1, J1501 DIN41612_02x32_AC, J301 20021111-00010T4LF, K1401 G5V-2-DC5, K1402 G5V-2-DC5, K1501 HE3621A0510, K1502 HE3621A0510, K1503 HE3621A0510, K1504 HE3621A0510, K1505 HE3621A0510, K1506 HE3621A0510, K801 UMS05-1A80-75D, K802 UMS05-1A80-75D, K803 UMS05-1A80-75D, K804 UMS05-1A80-75D, K805 UMS05-1A80-75D, Q1001 BSS123, Q1101 BSS123, Q1201 BSS123, Q1401 MMBT3904, Q1402 MMBT3904, Q401 SI5618A, Q402 MMBT3904, Q403 BSS123, Q801 MMBT3904, Q802 MMBT3904, Q803 MMBT3904, Q804 MMBT3904, Q805 BFR106, Q806 MMBT3904, Q807 BFR106, Q901 BSS123, U1001 AQY221R2S, U1002 AD8099ARDZ, U1003 AQY221R2S, U1101 AQY221R2S, U1102 AD8099ARDZ, U1103 AQY221R2S, U1201 AQY221R2S, U1202 AD8099ARDZ, U1203 AQY221R2S, U1501 LMH6644MT, U1502 ULN2003A, U1601 TXB0104PW, U1602 ADuM5402, U1603 74AC125, U201 LAN8742A, U202 SRV05-4, U301 SN74LV1T34DBV, U302 74LVC1G74DP, U303 STM32H743VITx, U304 24LC08B-E/MS, U305 REF2033, U401 REG103GA-5, U402 REG103GA-3.3, U403 LT1946A, U404 TEL5-2411, U405 LT1611, U501 SN74LVC1G04DBV, U502 AD9834, U503 AD9834, U504 SN74LV1T34DBV, U505 LMH6644MT, U506 TLV3501AIDBV, U507 74LVC1G74DP, U601 LMH6618MKE, U602 ADG1604BRUZ, U603 LMH6720MF, U604 LMH6720MF, U605 LMH6720MF, U701 LMH6618MKE, U702 TLV3501AIDBV, U703 74HCT4051PW, U704 SN74LVC1G3157DB, U705 SN74LVC1G3157DB, U706 SN74LV1T34DBV, U707 SN74LV1T34DBV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

Commit message: PCB layout
Parts:
- C418: moved to B.Cu
- C419: footprint Capacitor_SMD:C_0603_1608Metric_Pad1.08x0.95mm_HandSolder -> Capacitor_SMD:C_0805_2012Metric_Pad1.18x1.45mm_HandSolder
- C420, R415: moved to F.Cu
- RV501: value TS53YJ103MR10 -> 3266W-1-103LF; footprint Potentiometer_SMD:Potentiometer_Vishay_TS53YJ_Vertical -> Potentiometer_THT:Potentiometer_Bourns_3266W_Vertical
- moved L406 16.1 mm to (133.3, 143.1), turned to 90 degrees
- moved C419 12.4 mm to (148.6, 139.8), turned to -90 degrees
- moved D404 11.9 mm to (148.6, 144.3), turned to 90 degrees
- moved C417 11.7 mm to (136.1, 143.1), turned to -90 degrees
- moved R413 9.56 mm to (143.4, 134.6), turned to 90 degrees
- moved C420 8.41 mm to (141.0, 134.6), turned to -90 degrees
- moved R414 7.64 mm to (136.1, 134.6), turned to -90 degrees
- moved C421 7.06 mm to (136.1, 138.3), turned to 90 degrees
- moved C418 6.61 mm to (143.4, 134.6), turned to -90 degrees
- moved R415 5.33 mm to (138.6, 134.6), turned to -90 degrees
- moved U405 4.87 mm to (147.3, 134.6), turned to 180 degrees
- moved L407 4.83 mm to (142.2, 141.0), turned to 180 degrees
- moved RV501 3.51 mm to (163.9, 75.7)
- moved D301 2.84 mm to (190.4, 121.2)
- moved Q804 2.54 mm to (181.6, 61.5)
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Other:
- copper layers 2 -> 4
