File: Hardware/ETH1LCR3/ETH1LCR3.kicad_sch (KiCad schematic)
At the start: 0 parts

Commit message: Hardware
Other:
- sheet Ethernet renamed Ethernet PoE
- added sheet PSD (PSD.kicad_sch)
- sheet DDS ports: added DAC0_OUT, DAC1_OUT, DC_BIAS_VOLTAGE, DDS_SCLK, DDS_SDATA, DDS_~{FSYNC1}, DDS_~{FSYNC2}, PHI_OUT, RESET_DDS, SINE; removed none
- sheet Ethernet PoE ports: added NRST, REF_CLK, RMII_CRS_DV, RMII_MDC, RMII_MDIO, RMII_RXD0, RMII_RXD1, RMII_TXD0, RMII_TXD1, RMII_TXEN; removed none
- sheet MCU ports: added NRST, REF_CLK, RMII_CRS_DV, RMII_MDC, RMII_MDIO, RMII_RXD0, RMII_RXD1, RMII_TXD0, RMII_TXD1, RMII_TXEN; removed none
- sheet PGA ports: added PGA_A0, PGA_A1, PGA_G1, PGA_G10, PGA_G3, PGA_IN, PGA_OUT; removed none

Commit message: Hardware
Parts:
- added H101, H102, H103, H104: MountingHole, symbol Mechanical:MountingHole
- added HS101: Heatsink, symbol Mechanical:Heatsink
Other:
- added sheet Frontend (Frontend.kicad_sch)
- sheet PSD ports: added ADS_DIN, ADS_DOUT, ADS_SCLK, ADS_START, ADS_~{CS}, ADS_~{DRDY}, INPUT_CPO, PGA_OUT, PHI_OUT, PSD_RC_A, PSD_RC_B, PSD_RC_C; removed none
- sheet Power ports: added EN_BOOST, MAX_BOOST; removed none

Commit message: Hardware
Parts:
- H101, H102, H103, H104: footprint (none) -> MountingHole:MountingHole_3.2mm_M3_DIN965_Pad
Other:
- added sheet Connector (Connector.kicad_sch)
- added sheet Front (Front.kicad_sch)
- added sheet Select front-rear (Select.kicad_sch)
- added sheet Trigger (Trigger.kicad_sch)
- sheet DDS ports: added DDS_RESET; removed RESET_DDS
- sheet Ethernet PoE ports: added RX+, RX-, TX+, TX-; removed none
- sheet Frontend ports: added CALIB_100, CALIB_100K, CALIB_10K, CALIB_1K, PGA_IN, SINE; removed CALC_100, CALC_100K, CALC_10K, CALC_1K, SINUS
- sheet MCU ports: added ADS_DIN, ADS_DOUT, ADS_SCLK, ADS_START, ADS_~{CS}, ADS_~{DRDY}, CALIB_100, CALIB_100K, CALIB_10K, CALIB_1K, DAC0_OUT, DAC1_OUT, DC_BIAS_U-I, DDS_RESET, DDS_SCLK, DDS_SDATA, DDS_~{FSYNC1}, DDS_~{FSYNC2}, EN_BOOST, FE_SW1, FE_SW2, FE_SW3, FE_SW4, FE_SW5, FE_SW6, FE_V_SHORT, INPUT_CPO, I_VOLTAGE, MAX_BOOST, PGA_A0, PGA_A1, PGA_G1, PGA_G10, PGA_G3, PHI_OUT, PSD_RC_A, PSD_RC_B, PSD_RC_C, SELECT_RELAY, TRIG_EN, TRIG_IN, TRIG_OUT; removed none
- moved on the sheet: H101, H102, H103, H104, HS101

Commit message: Software and hardware
Other:
- sheet Connector ports: added EXT_TRIG, HD_REAR, HS_REAR, LD_REAR, LS_REAR; removed none
- sheet MCU ports: added INPUT_COMP; removed INPUT_CPO
- sheet PSD ports: added INPUT_COMP; removed INPUT_CPO
Changed lines of the file:
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@@
+	(wire
+		(pts
+			(xy 173.99 17.78) (xy 214.63 17.78)
+		)
+		(stroke
+			(width 0)
+			(type default)
+		)
+	)
 	(wire
 		(pts
@@
 	(wire
 		(pts
+			(xy 173.99 25.4) (xy 214.63 25.4)
+		)
+		(stroke
+			(width 0)
+			(type default)
+		)
+	)
+	(wire
+		(pts
 			(xy 64.77 73.66) (xy 58.42 73.66)
 		)
@@
 	(wire
 		(pts
+			(xy 173.99 22.86) (xy 214.63 22.86)
+		)
+		(stroke
+			(width 0)
+			(type default)
+		)
+	)
+	(wire
+		(pts
 			(xy 129.54 44.45) (xy 135.89 44.45)
 		)
@@
 	(wire
 		(pts
+			(xy 173.99 20.32) (xy 214.63 20.32)
+		)
+		(stroke
+			(width 0)
+			(type default)
+		)
+	)
+	(wire
+		(pts
 			(xy 173.99 72.39) (xy 181.61 72.39)
 		)
@@
 		(pts
 			(xy 129.54 20.32) (xy 135.89 20.32)
+		)
+		(stroke
+			(width 0)
+			(type default)
+		)
+	)
+	(wire
+		(pts
+			(xy 205.74 129.54) (xy 214.63 129.54)
 		)
 		(stroke
@@
 			)
 		)
+		(pin "HS_REAR" bidirectional
+			(at 214.63 20.32 180)
+			(effects
+				(font
+					(size 1.27 1.27)
+				)
+				(justify left)
+			)
+		)
+		(pin "HD_REAR" bidirectional
+			(at 214.63 17.78 180)
+			(effects
+				(font
+					(size 1.27 1.27)
+				)
+				(justify left)
+			)
+		)
+		(pin "LS_REAR" bidirectional
+			(at 214.63 22.86 180)
+			(effects
+				(font
+					(size 1.27 1.27)
+				)
+				(justify left)
+			)
+		)
+		(pin "LD_REAR" bidirectional
+			(at 214.63 25.4 180)
+			(effects
+				(font
+					(size 1.27 1.27)
+				)
+				(justify left)
+			)
+		)
+		(pin "EXT_TRIG" bidirectional
+			(at 214.63 129.54 180)
+			(effects
+				(font
+					(size 1.27 1.27)
+				)
+				(justify left)
+			)
+		)
 		(instances
 			(project "ETH1LCR3"
@@
 	)
 	(sheet
-		(at 135.89 58.42)
-		(size 38.1 110.49)
+		(at 135.89 57.15)
+		(size 38.1 111.76)
 		(fields_autoplaced yes)
 		(stroke
@@
 		)
 		(property "Sheetname" "MCU"
-			(at 135.89 57.7084 0)
+			(at 135.89 56.4384 0)
 			(effects
 				(font
@@
 			)
 		)
-		(pin "ADS_~{DRDY}" output
+		(pin "ADS_~{DRDY}" input
 			(at 135.89 140.97 180)
 			(effects
@@
 			)
 		)
-		(pin "ADS_DOUT" output
+		(pin "ADS_DOUT" input
 			(at 135.89 143.51 180)
 			(effects
@@
 			)
 		)
-		(pin "INPUT_CPO" input
+		(pin "INPUT_COMP" input
 			(at 135.89 153.67 180)
 			(effects
@@
 			)
 		)
-		(pin "ADS_DOUT" input
+		(pin "ADS_DOUT" output
 			(at 58.42 64.77 0)
 			(effects
@@
 			)
 		)
-		(pin "ADS_~{DRDY}" input
+		(pin "ADS_~{DRDY}" output
 			(at 58.42 62.23 0)
 			(effects
@@
 			)
 		)
-		(pin "INPUT_CPO" output
+		(pin "INPUT_COMP" output
 			(at 58.42 77.47 0)
 			(effects

Commit message: Hardware
Parts:
- HS101: footprint (none) -> ETH1LCR3:960-19-12-S-AB-0
Other:
- sheet Ethernet PoE renamed Ethernet
- sheet Connector ports: added CXN_REL1, CXN_REL2, CXN_REL3, CXN_REL4, CXN_REL5, CXN_REL6; removed none
- sheet MCU ports: added CXN_REL1, CXN_REL2, CXN_REL3, CXN_REL4, CXN_REL5, CXN_REL6; removed none

Commit message: Hardware
Parts:
- removed H101, H102, H103, H104: MountingHole, MountingHole:MountingHole_3.2mm_M3_DIN965_Pad, symbol Mechanical:MountingHole

Commit message: PCB layout
Other:
- sheet Connector ports: added DC_BIAS_VOLTAGE, SINE; removed none
Changed lines of the file:
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@@
+			)
+		)
+		(pin "SINE" input
+			(at 214.63 30.48 180)
+			(effects
+				(font
+					(size 1.27 1.27)
+				)
+				(justify left)
+			)
+		)
+		(pin "DC_BIAS_VOLTAGE" input
+			(at 214.63 33.02 180)
+			(effects
+				(font
+					(size 1.27 1.27)
+				)
+				(justify left)
 			)
 		)
