File: Hardware/ETH1LCR3/Frontend.kicad_sch (KiCad schematic)
At the start: 78 parts, among them K801 UMS05-1A80-75D, K802 UMS05-1A80-75D, K803 UMS05-1A80-75D, K804 UMS05-1A80-75D, K805 UMS05-1A80-75D, Q801 MMBT3904, Q802 MMBT3904, Q803 MMBT3904, Q804 MMBT3904, Q805 BFR106, Q806 BFR106, U801 74LVC1G3157DB, U802 LMH6644MT, U803 OPA2727AID, U804 AQY221R2S, U805 AQY221R2S, U806 SN74LV1T34DBV, U807 SN74LV1T34DBV, U808 SN74LV1T34DBV

Commit message: Hardware
Parts:
- removed R822: 240, Resistor_SMD:R_0603_1608Metric_Pad0.98x0.95mm_HandSolder, symbol Device:R
- added R826: 240, Resistor_SMD:R_0603_1608Metric_Pad0.98x0.95mm_HandSolder, symbol Device:R
- C809: footprint (none) -> Capacitor_SMD:C_0805_2012Metric_Pad1.18x1.45mm_HandSolder
- C816: footprint Capacitor_SMD:C_0603_1608Metric_Pad1.08x0.95mm_HandSolder -> (none)
- renumbered R823 to R822, R824 to R823, R825 to R824, R826 to R825
Connections:
- net GND: now also R826.2
- net at C816.1: now also C815.2, R822.2, R823.2, R825.2, U802.8, U804.3
- net PGA_IN: now reaches U804.4, U805.4
- new net: C816.2, R826.1
Other:
- moved on the sheet: C814, R825, R831, R832, U803B, U806, U807

Commit message: Hardware
Parts:
- added Q807: MMBT3904, Package_TO_SOT_SMD:SOT-23, symbol Transistor_BJT:MMBT3904
- added R836: 10k, Resistor_SMD:R_0603_1608Metric_Pad0.98x0.95mm_HandSolder, symbol Device:R
- C816: footprint (none) -> Capacitor_SMD:C_0603_1608Metric_Pad1.08x0.95mm_HandSolder
Connections:
- net FE_V_SHORT: now also R836.1; no longer K805.2
- net GND: now also Q807.2 (E)
- net CALC_100 renamed CALIB_100
- net CALC_100K renamed CALIB_100K
- net CALC_10K renamed CALIB_10K
- net CALC_1K renamed CALIB_1K
- net SINUS renamed SINE
- new net: Q807.1 (B), R836.2
- new net: K805.2, Q807.3 (C)
Other:
- moved on the sheet: K801, K802, K803, K804, Q801, Q802, Q803, Q804, R801, R802, R803, R804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

Commit message: Software and hardware
Parts:
- renumbered Q807 to Q806, Q806 to Q807, R836 to R809, R809 to R810, R810 to R811, R811 to R812, R812 to R813, R813 to R814, R814 to R815, R815 to R816, R816 to R817, R817 to R818, R818 to R819, R819 to R820, R820 to R821, R821 to R822, R822 to R823, R823 to R824, R824 to R825, R825 to R826, R826 to R827, R827 to R828, R828 to R829, R829 to R830, R830 to R831, R831 to R832, R832 to R833, R833 to R834, R834 to R835, R835 to R836

Commit message: Hardware
Other:
- moved on the sheet: C809, D801, L801, R812

Commit message: Hardware
Parts:
- C810, C811, C814: footprint (none) -> Capacitor_SMD:C_0805_2012Metric_Pad1.18x1.45mm_HandSolder
- C813: value 3-10p -> JZ100; footprint (none) -> Capacitor_SMD:C_Trimmer_Voltronics_JZ
- RV801: value 50 -> 3266W-1-500LF; footprint (none) -> Potentiometer_THT:Potentiometer_Bourns_3266W_Vertical
- U803: footprint Package_SO:SOP-4_3.8x4.1mm_P2.54mm -> Package_SO:SOIC-8_3.9x4.9mm_P1.27mm
- U804, U805: footprint Package_TO_SOT_SMD:SOT-23-5 -> Package_SO:SOP-4_3.8x4.1mm_P2.54mm
- U806: footprint Package_SO:SOIC-8_3.9x4.9mm_P1.27mm -> Package_TO_SOT_SMD:SOT-23-5
- U807: footprint Package_SO:SOP-4_3.8x4.1mm_P2.54mm -> Package_TO_SOT_SMD:SOT-23-5
Other:
- moved on the sheet: R823
Changed lines of the file:
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@@
 	(wire
 		(pts
-			(xy 311.15 34.29) (xy 304.8 34.29)
+			(xy 311.15 34.29) (xy 308.61 34.29)
 		)
 		(stroke
@@
 	(wire
 		(pts
-			(xy 292.1 34.29) (xy 297.18 34.29)
+			(xy 292.1 34.29) (xy 300.99 34.29)
 		)
 		(stroke
@@
 			)
 		)
-		(property "Footprint" "Package_TO_SOT_SMD:SOT-23-5"
+		(property "Footprint" "Package_SO:SOP-4_3.8x4.1mm_P2.54mm"
 			(at 334.01 118.11 0)
 			(effects
@@
 			)
 		)
-		(property "Value" "3-10p"
+		(property "Value" "JZ100"
 			(at 278.13 45.72 90)
 			(effects
@@
 			)
 		)
-		(property "Footprint" ""
+		(property "Footprint" "Capacitor_SMD:C_Trimmer_Voltronics_JZ"
 			(at 278.13 41.91 0)
 			(effects
@@
 			)
 		)
-		(property "Footprint" ""
+		(property "Footprint" "Capacitor_SMD:C_0805_2012Metric_Pad1.18x1.45mm_HandSolder"
 			(at 294.64 84.1248 0)
 			(effects
@@
 			)
 		)
-		(property "Footprint" "Package_TO_SOT_SMD:SOT-23-5"
+		(property "Footprint" "Package_SO:SOP-4_3.8x4.1mm_P2.54mm"
 			(at 334.01 156.21 0)
 			(effects
@@
 			)
 		)
-		(property "Footprint" "Package_SO:SOP-4_3.8x4.1mm_P2.54mm"
+		(property "Footprint" "Package_TO_SOT_SMD:SOT-23-5"
 			(at 336.55 149.86 0)
 			(effects
@@
 		(dnp no)
 		(property "Reference" "RV801"
-			(at 288.29 29.464 90)
+			(at 288.29 28.956 90)
 			(effects
 				(font
@@
 			)
 		)
-		(property "Value" "50"
-			(at 288.29 32.004 90)
+		(property "Value" "3266W-1-500LF"
+			(at 290.83 30.988 90)
 			(effects
 				(font
@@
 			)
 		)
-		(property "Footprint" ""
+		(property "Footprint" "Potentiometer_THT:Potentiometer_Bourns_3266W_Vertical"
 			(at 288.29 34.29 0)
 			(effects
@@
 			)
 		)
-		(property "Footprint" "Package_SO:SOIC-8_3.9x4.9mm_P1.27mm"
+		(property "Footprint" "Package_TO_SOT_SMD:SOT-23-5"
 			(at 336.55 111.76 0)
 			(effects
@@
 			)
 		)
-		(property "Footprint" "Package_SO:SOP-4_3.8x4.1mm_P2.54mm"
+		(property "Footprint" "Package_SO:SOIC-8_3.9x4.9mm_P1.27mm"
 			(at 60.96 266.7 0)
 			(effects
@@
 			)
 		)
-		(property "Footprint" "Package_SO:SOP-4_3.8x4.1mm_P2.54mm"
+		(property "Footprint" "Package_SO:SOIC-8_3.9x4.9mm_P1.27mm"
 			(at 293.37 74.93 0)
 			(effects
@@
 	(symbol
 		(lib_id "Device:R")
-		(at 300.99 34.29 90)
+		(at 304.8 34.29 90)
 		(unit 1)
 		(exclude_from_sim no)
@@
 		(dnp no)
 		(property "Reference" "R823"
-			(at 300.99 29.464 90)
+			(at 304.8 29.464 90)
 			(effects
 				(font
@@
 		)
 		(property "Value" "2k/.1%"
-			(at 300.99 31.75 90)
+			(at 304.8 31.75 90)
 			(effects
 				(font
@@
 		)
 		(property "Footprint" "Resistor_SMD:R_0603_1608Metric_Pad0.98x0.95mm_HandSolder"
-			(at 300.99 36.068 90)
+			(at 304.8 36.068 90)
 			(effects
 				(font
@@
 		)
 		(property "Datasheet" "~"
-			(at 300.99 34.29 0)
+			(at 304.8 34.29 0)
 			(effects
 				(font
@@
 		)
 		(property "Description" "Resistor"
-			(at 300.99 34.29 0)
+			(at 304.8 34.29 0)
 			(effects
 				(font
@@
 			)
 		)
-		(property "Footprint" ""
+		(property "Footprint" "Capacitor_SMD:C_0805_2012Metric_Pad1.18x1.45mm_HandSolder"
 			(at 214.3252 220.98 0)
 			(effects
@@
 			)
 		)
-		(property "Footprint" ""
+		(property "Footprint" "Capacitor_SMD:C_0805_2012Metric_Pad1.18x1.45mm_HandSolder"
 			(at 228.6 233.9848 0)
 			(effects
@@
 			)
 		)
-		(property "Footprint" "Package_SO:SOP-4_3.8x4.1mm_P2.54mm"
+		(property "Footprint" "Package_SO:SOIC-8_3.9x4.9mm_P1.27mm"
 			(at 226.06 246.38 0)
 			(effects

Commit message: PCB layout
Parts:
- JP801, JP802: now left out of the parts list
- U806, U807, U808: footprint Package_TO_SOT_SMD:SOT-23-5 -> Package_TO_SOT_SMD:SOT-23-5_HandSoldering
Changed lines of the file:
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@@
 			)
 		)
-		(property "Footprint" "Package_TO_SOT_SMD:SOT-23-5"
+		(property "Footprint" "Package_TO_SOT_SMD:SOT-23-5_HandSoldering"
 			(at 350.52 83.82 0)
 			(effects
@@
 			)
 		)
-		(property "Footprint" "Package_TO_SOT_SMD:SOT-23-5"
+		(property "Footprint" "Package_TO_SOT_SMD:SOT-23-5_HandSoldering"
 			(at 336.55 149.86 0)
 			(effects
@@
 		(unit 1)
 		(exclude_from_sim no)
-		(in_bom yes)
+		(in_bom no)
 		(on_board yes)
 		(dnp no)
@@
 			)
 		)
-		(property "Footprint" "Package_TO_SOT_SMD:SOT-23-5"
+		(property "Footprint" "Package_TO_SOT_SMD:SOT-23-5_HandSoldering"
 			(at 336.55 111.76 0)
 			(effects
@@
 		(unit 1)
 		(exclude_from_sim no)
-		(in_bom yes)
+		(in_bom no)
 		(on_board yes)
 		(dnp no)

Commit message: PCB layout
Parts:
- renumbered R824 to R823, R825 to R824, R823 to R825
Changed lines of the file:
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@@
 		(on_board yes)
 		(dnp no)
-		(property "Reference" "R825"
+		(property "Reference" "R824"
 			(at 300.99 58.674 90)
 			(effects
@@
 			(project "ETH1LCR3"
 				(path "/6623bacb-57aa-43ce-9e51-b38a560dd9fc/37965f22-1055-43ab-ab57-7d9b27fac2d0"
-					(reference "R825")
+					(reference "R824")
 					(unit 1)
 				)
@@
 		(on_board yes)
 		(dnp no)
-		(property "Reference" "R824"
+		(property "Reference" "R823"
 			(at 300.99 43.434 90)
 			(effects
@@
 			(project ""
 				(path "/6623bacb-57aa-43ce-9e51-b38a560dd9fc/37965f22-1055-43ab-ab57-7d9b27fac2d0"
-					(reference "R824")
+					(reference "R823")
 					(unit 1)
 				)
@@
 		(on_board yes)
 		(dnp no)
-		(property "Reference" "R823"
+		(property "Reference" "R825"
 			(at 304.8 29.464 90)
 			(effects
@@
 			(project "ETH1LCR3"
 				(path "/6623bacb-57aa-43ce-9e51-b38a560dd9fc/37965f22-1055-43ab-ab57-7d9b27fac2d0"
-					(reference "R823")
-					(unit 1)
-				)
+					(reference "R825")
+					(unit 1)
+				)

Commit message: PCB layout
Parts:
- removed U803: OPA2727AID, Package_SO:SOIC-8_3.9x4.9mm_P1.27mm, symbol ETH1LCR3:OPA2727AID
- added C806, C809: 0.1u, Capacitor_SMD:C_0603_1608Metric_Pad1.08x0.95mm_HandSolder, symbol Device:C
- added R823: 100k, Resistor_SMD:R_0603_1608Metric_Pad0.98x0.95mm_HandSolder, symbol Device:R
- added U803, U804: OPA727AIDG, Package_SO:MSOP-8_3x3mm_P0.65mm, symbol ETH1LCR3:OPA727AIDG
- Q805, Q807: footprint Package_TO_SOT_SMD:SOT-23_Handsoldering -> Package_TO_SOT_SMD:SOT-23
- renumbered C806 to C807, C807 to C808, C808 to C810, C809 to C811, C810 to C812, C811 to C813, C812 to C814, C813 to C815, C814 to C816, C815 to C817, C816 to C818, C817 to C819, R822 to R821, R821 to R822, R823 to R824, R824 to R825, R825 to R826, R826 to R827, R827 to R828, R828 to R829, R829 to R830, R830 to R831, R831 to R832, R832 to R833, R833 to R834, R834 to R835, R835 to R836, R836 to R837, U804 to U805, U805 to U806, U806 to U807, U807 to U808, U808 to U809
Connections:
- net +5V: now also C806.1, U803.7 (V+), U804.7 (V+)
- net -5V: now also C809.1, U803.4 (V-), U804.4 (V-)
- net GND: now also C806.2, C809.2, U803.3 (+), U804.3 (+)
- net at R821.2, R825.1, U802.10 (+): now also R823.1; no longer C816.1
- net at C816.2, R827.1: now also U804.2 (-)
- net at C813.1, R811.2: now also U803.6
- net at C813.2, R818.1: now also U803.2 (-)
- new net: C816.1, R823.2, U804.6
Other:
- moved on the sheet: C801, C802, C803, C804, C805, C807, C808, C810, C813, C816, R821, R827
