File: Hardware/ETH1LCR3/Ethernet.kicad_sch (KiCad schematic)
At the start: 25 parts, among them J201 RJ45_Wuerth_7499010121A, U201 LAN8742A, Y201 NX5032GA-25

Commit message: Schematic
Parts:
- Y201: footprint ETH1HMSR-SMS:NX5032GA -> (none)
Changed lines of the file:
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@@
 			)
 		)
-		(property "Footprint" "ETH1HMSR-SMS:NX5032GA"
+		(property "Footprint" ""
 			(at 80.01 125.73 0)
 			(effects

Commit message: Hardware
Parts:
- removed J201: RJ45_Wuerth_7499010121A, Connector_RJ:RJ45_Wuerth_7499010121A_Horizontal, symbol Connector:RJ45_Wuerth_7499010121A
- added C213: 10u, symbol Device:C_Polarized
- added C214: 100u, symbol Device:C_Polarized
- added D201: VS-30BQ040-M3/9ATD, symbol Device:D
- added J201: RJ45_Abracon_ARJP11A-MASA-B-A-EMU2, Connector_RJ:RJ45_Abracon_ARJP11A-MA_Horizontal, symbol Connector:RJ45_Abracon_ARJP11A-MASA-B-A-EMU2
- added R207: DNP, symbol Device:R
- added R208: 0, symbol Device:R
- added U202: Ag9905LP, Converter_DCDC:Converter_DCDC_Silvertel_Ag99xxLP_THT, symbol Converter_DCDC:Ag9905LP
Connections:
- net ETH_RXN: now also J201.6 (RD-)
- net ETH_RXP: now also J201.3 (RD+)
- net ETH_TXN: now also J201.2 (TD-)
- net ETH_TXP: now also J201.1 (TD+)
- net Earth: now also J201.7, J201.SH
- net GND: now also C213.2, C214.2, R208.2, U202.3 (-VDC)
- net LED1: now also J201.13
- net LED2: now also J201.11
- net VCCQ: now also J201.4 (TCT), J201.5 (RCT)
- net at R205.1: now also J201.14
- net at R206.1: now also J201.12
- new net: C213.1, C214.1, D201.2 (A), R207.1, U202.1 (+VDC), U202.2 (+VDC)
- new net: J201.10 (V-), U202.7 (VIN-), U202.8 (VIN-)
- new net: J201.9 (V+), U202.5 (VIN+), U202.6 (VIN+)
- new net: R207.2, R208.1, U202.4 (ADJ)
- new net +5VP: D201.1 (K)
Other:
- moved on the sheet: C201, C202, C203, C204, C205, C206, C207, C208, C209, C210, C211, C212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

Commit message: Hardware
Parts:
- added C211: 10u/25V, symbol Device:C_Polarized
- added L201: 1u8, symbol Device:L
- C212: renamed from C213; value 10u -> 10u/25V
- C213: renamed from C214; value 100u -> 100u/25V; footprint (none) -> Capacitor_SMD:C_0603_1608Metric_Pad1.08x0.95mm_HandSolder
- R205: renamed from R207; value DNP -> 0; footprint (none) -> Resistor_SMD:R_0603_1608Metric_Pad0.98x0.95mm_HandSolder
- R206: renamed from R208; footprint (none) -> Resistor_SMD:R_0603_1608Metric_Pad0.98x0.95mm_HandSolder
- renumbered C211 to C214, C212 to C215, R205 to R207, R206 to R208
Connections:
- net GND: now also C211.2
- net at C212.1, C213.1, R205.1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: now also L201.2; no longer D201.2 (A)
- new net: C211.1, D201.2 (A), L201.1
Other:
- moved on the sheet: C212, C213, D201, J201, R205, R206, R207, R208, U202

Commit message: Hardware
Parts:
- C213: footprint Capacitor_SMD:C_0603_1608Metric_Pad1.08x0.95mm_HandSolder -> (none)
- L201: value 1u8 -> 74438356018HT1u8
Other:
- moved on the sheet: L201
Changed lines of the file:
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@@
 	(wire
 		(pts
-			(xy 148.59 124.46) (xy 149.86 124.46)
+			(xy 144.78 124.46) (xy 149.86 124.46)
 		)
 		(stroke
@@
 	(wire
 		(pts
-			(xy 129.54 124.46) (xy 140.97 124.46)
+			(xy 129.54 124.46) (xy 137.16 124.46)
 		)
 		(stroke
@@
 	(symbol
 		(lib_id "Device:L")
-		(at 144.78 124.46 90)
+		(at 140.97 124.46 90)
 		(unit 1)
 		(exclude_from_sim no)
@@
 		(fields_autoplaced yes)
 		(property "Reference" "L201"
-			(at 144.78 119.38 90)
+			(at 140.97 119.38 90)
 			(effects
 				(font
@@
 			)
 		)
-		(property "Value" "1u8"
-			(at 144.78 121.92 90)
+		(property "Value" "74438356018HT1u8"
+			(at 140.97 121.92 90)
 			(effects
 				(font
@@
 		)
 		(property "Footprint" ""
-			(at 144.78 124.46 0)
+			(at 140.97 124.46 0)
 			(effects
 				(font
@@
 		)
 		(property "Datasheet" "~"
-			(at 144.78 124.46 0)
+			(at 140.97 124.46 0)
 			(effects
 				(font
@@
 		)
 		(property "Description" "Inductor"
-			(at 144.78 124.46 0)
+			(at 140.97 124.46 0)
 			(effects
 				(font
@@
 			)
 		)
-		(property "Footprint" "Capacitor_SMD:C_0603_1608Metric_Pad1.08x0.95mm_HandSolder"
+		(property "Footprint" ""
 			(at 167.3352 138.43 0)
 			(effects

Commit message: Hardware
Parts:
- removed C211, C212: 10u/25V, symbol Device:C_Polarized
- removed C213: 100u/25V, symbol Device:C_Polarized
- removed D201: VS-30BQ040-M3/9ATD, symbol Device:D
- removed J201: RJ45_Abracon_ARJP11A-MASA-B-A-EMU2, Connector_RJ:RJ45_Abracon_ARJP11A-MA_Horizontal, symbol Connector:RJ45_Abracon_ARJP11A-MASA-B-A-EMU2
- removed L201: 74438356018HT1u8, symbol Device:L
- removed U202: Ag9905LP, Converter_DCDC:Converter_DCDC_Silvertel_Ag99xxLP_THT, symbol Converter_DCDC:Ag9905LP
- added C211, C212: 1n/1kV, symbol Device:C
- added D201: YELLOW, LED_SMD:LED_0603_1608Metric_Pad1.05x0.95mm_HandSolder, symbol Device:LED
- added D202: GREEN, LED_SMD:LED_0603_1608Metric_Pad1.05x0.95mm_HandSolder, symbol Device:LED
- added R209: 1M/1kV, Resistor_SMD:R_1206_3216Metric_Pad1.30x1.75mm_HandSolder, symbol Device:R
- added TR201: Wuerth_749013011A, Transformer_SMD:Transformer_Ethernet_Wuerth_749013011A, symbol Transformer:Wuerth_749013011A
- added U202: SRV05-4, Converter_DCDC:Converter_DCDC_Silvertel_Ag99xxLP_THT, symbol Power_Protection:SRV05-4
- R205: value 0 -> 560; now fitted; now in the parts list
- R206: value 0 -> 560
- R207, R208: value 560 -> 75/1%
Connections:
- net ETH_RXN: now also TR201.8 (RD-)
- net ETH_RXP: now also TR201.6 (RD+)
- net ETH_TXN: now also TR201.3 (TD-)
- net ETH_TXP: now also TR201.1 (TD+)
- net Earth: now also C211.1, C212.2, R209.1
- net GND: now also R205.2, C211.2, R209.2; no longer R207.2, R208.2
- net LED1: now also D202.2 (A)
- net LED2: now also D201.2 (A)
- net VCCQ: now also TR201.2 (C_TD), TR201.7 (C_RD)
- net at R205.1: now also D201.1 (K)
- net at R207.1: now also TR201.10 (C_RX)
- net at R208.1: now also TR201.15 (C_TX)
- net at R206.1: now also D202.1 (K); no longer R205.2
- new net: C212.1, R207.2, R208.2
- new net RX+: TR201.11 (RX+), U202.3 (IO2)
- new net RX-: TR201.9 (RX-), U202.4 (IO3)
- new net TX+: TR201.16 (TX+), U202.6 (IO4)
- new net TX-: TR201.14 (TX-), U202.1 (IO1)
- no-connect marks 0 -> 2
Other:
- moved on the sheet: C201, C202, C203, C204, C205, C206, C207, C208, C209, C210, C214, C215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

Commit message: Software and hardware
Parts:
- U202: footprint Converter_DCDC:Converter_DCDC_Silvertel_Ag99xxLP_THT -> Package_TO_SOT_SMD:SOT-23-6
- renumbered C214 to C211, C215 to C212, C211 to C213, C212 to C214, R204 to R203, R203 to R204, R209 to R207, R207 to R208, R208 to R209

Commit message: Hardware
Parts:
- C213, C214: footprint (none) -> Capacitor_SMD:C_1206_3216Metric_Pad1.33x1.80mm_HandSolder
- Y201: footprint (none) -> ETH1LCR3:NX5032GA
Changed lines of the file:
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@@
 			)
 		)
-		(property "Footprint" ""
+		(property "Footprint" "Capacitor_SMD:C_1206_3216Metric_Pad1.33x1.80mm_HandSolder"
 			(at 193.04 117.8052 0)
 			(effects
@@
 			)
 		)
-		(property "Footprint" ""
+		(property "Footprint" "Capacitor_SMD:C_1206_3216Metric_Pad1.33x1.80mm_HandSolder"
 			(at 215.5952 110.49 0)
 			(effects
@@
 			)
 		)
-		(property "Footprint" ""
+		(property "Footprint" "ETH1LCR3:NX5032GA"
 			(at 46.99 118.11 0)
 			(effects

Commit message: PCB layout
Parts:
- removed RN203: EXB-38V510JV, Resistor_SMD:R_Array_Concave_4x0603, symbol Device:R_Pack04
- added R210, R211, R212, R213: 51, Resistor_SMD:R_0603_1608Metric_Pad0.98x0.95mm_HandSolder, symbol Device:R
Connections:
- net ETH_RXN: now also R213.2
- net ETH_RXP: now also R212.2
- net ETH_TXN: now also R211.2
- net ETH_TXP: now also R210.2
- net VCCQ: now also R210.1, R211.1, R212.1, R213.1
Other:
- moved on the sheet: C211
