File: Hardware/ETH1LCR3/Connector.kicad_sch (KiCad schematic)
At the start: 1 part, among them J1501 DIN41612_02x32_AC

Commit message: Software and hardware
Connections:
- no-connect marks 8 -> 36
Changed lines of the file:
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@@
+	)
+	(no_connect
+		(at 109.22 93.98)
+	)
+	(no_connect
+		(at 109.22 76.2)
+	)
+	(no_connect
+		(at 109.22 55.88)
+	)
+	(no_connect
+		(at 121.92 66.04)
+	)
+	(no_connect
+		(at 121.92 68.58)
+	)
+	(no_connect
+		(at 109.22 66.04)
+	)
+	(no_connect
+		(at 121.92 55.88)
 	)
 	(no_connect
@@
 	)
 	(no_connect
+		(at 121.92 71.12)
+	)
+	(no_connect
+		(at 109.22 60.96)
+	)
+	(no_connect
+		(at 109.22 68.58)
+	)
+	(no_connect
 		(at 121.92 109.22)
 	)
 	(no_connect
+		(at 121.92 99.06)
+	)
+	(no_connect
+		(at 109.22 99.06)
+	)
+	(no_connect
+		(at 109.22 96.52)
+	)
+	(no_connect
+		(at 109.22 71.12)
+	)
+	(no_connect
+		(at 121.92 101.6)
+	)
+	(no_connect
+		(at 121.92 63.5)
+	)
+	(no_connect
 		(at 121.92 111.76)
 	)
 	(no_connect
+		(at 121.92 96.52)
+	)
+	(no_connect
 		(at 109.22 109.22)
 	)
 	(no_connect
+		(at 121.92 78.74)
+	)
+	(no_connect
+		(at 121.92 60.96)
+	)
+	(no_connect
 		(at 109.22 83.82)
 	)
 	(no_connect
+		(at 109.22 101.6)
+	)
+	(no_connect
+		(at 109.22 78.74)
+	)
+	(no_connect
+		(at 121.92 93.98)
+	)
+	(no_connect
+		(at 109.22 73.66)
+	)
+	(no_connect
+		(at 109.22 63.5)
+	)
+	(no_connect
 		(at 109.22 111.76)
 	)
 	(no_connect
+		(at 121.92 73.66)
+	)
+	(no_connect
+		(at 109.22 58.42)
+	)
+	(no_connect
 		(at 121.92 38.1)
+	)
+	(no_connect
+		(at 121.92 76.2)
+	)
+	(no_connect
+		(at 121.92 58.42)
 	)
 	(wire
@@
 			)
 			(justify left)
+		)
+	)
+	(hierarchical_label "EXT_TRIG"
+		(shape bidirectional)
+		(at 41.91 69.85 180)
+		(fields_autoplaced yes)
+		(effects
+			(font
+				(size 1.27 1.27)
+			)
+			(justify right)
 		)
 	)
@@
 		(on_board yes)
 		(dnp no)
-		(property "Reference" "#PWR01504"
+		(property "Reference" "#PWR01505"
 			(at 129.54 81.28 0)
 			(effects
@@
 			)
 		)
-		(property "Description" ""
+		(property "Description" "Power symbol creates a global label with name \"Earth\""
 			(at 123.19 81.28 0)
 			(effects
@@
 			(project "ETH1LCR3"
 				(path "/6623bacb-57aa-43ce-9e51-b38a560dd9fc/4b99b960-154b-4647-bcd6-01f80df128c7"
-					(reference "#PWR01504")
+					(reference "#PWR01505")
 					(unit 1)
 				)
@@
 		(on_board yes)
 		(dnp no)
-		(property "Reference" "#PWR01505"
+		(property "Reference" "#PWR01502"
 			(at 110.49 114.3 0)
 			(effects
@@
 			)
 		)
-		(property "Description" ""
+		(property "Description" "Power symbol creates a global label with name \"+24V\""
 			(at 106.68 114.3 0)
 			(effects
@@
 			(project "ETH1LCR3"
 				(path "/6623bacb-57aa-43ce-9e51-b38a560dd9fc/4b99b960-154b-4647-bcd6-01f80df128c7"
-					(reference "#PWR01505")
+					(reference "#PWR01502")
 					(unit 1)
 				)
@@
 		(on_board yes)
 		(dnp no)
-		(property "Reference" "#PWR01501"
+		(property "Reference" "#PWR01504"
 			(at 101.6 91.44 0)
 			(effects
@@
 			)
 		)
-		(property "Description" ""
+		(property "Description" "Power symbol creates a global label with name \"Earth\""
 			(at 107.95 91.44 0)
 			(effects
@@
 			(project "ETH1LCR3"
 				(path "/6623bacb-57aa-43ce-9e51-b38a560dd9fc/4b99b960-154b-4647-bcd6-01f80df128c7"
-					(reference "#PWR01501")
+					(reference "#PWR01504")
 					(unit 1)
 				)
@@
 		(on_board yes)
 		(dnp no)
-		(property "Reference" "#PWR01502"
+		(property "Reference" "#PWR01506"
 			(at 129.54 91.44 0)
 			(effects
@@
 			)
 		)
-		(property "Description" ""
+		(property "Description" "Power symbol creates a global label with name \"Earth\""
 			(at 123.19 91.44 0)
 			(effects
@@
 			(project "ETH1LCR3"
 				(path "/6623bacb-57aa-43ce-9e51-b38a560dd9fc/4b99b960-154b-4647-bcd6-01f80df128c7"
-					(reference "#PWR01502")
+					(reference "#PWR01506")
 					(unit 1)
 				)
@@
 			)
 		)
-		(property "Description" ""
+		(property "Description" "Power symbol creates a global label with name \"Earth\""
 			(at 107.95 81.28 0)
 			(effects
@@
 		(on_board yes)
 		(dnp no)
-		(property "Reference" "#PWR01506"
+		(property "Reference" "#PWR01508"
 			(at 120.65 114.3 0)
 			(effects
@@
 			)
 		)
-		(property "Description" ""
+		(property "Description" "Power symbol creates a global label with name \"+24V\""
 			(at 124.46 114.3 0)
 			(effects
@@
 			(project "ETH1LCR3"
 				(path "/6623bacb-57aa-43ce-9e51-b38a560dd9fc/4b99b960-154b-4647-bcd6-01f80df128c7"
-					(reference "#PWR01506")
+					(reference "#PWR01508")
 					(unit 1)
 				)
@@
 		(on_board yes)
 		(dnp no)
-		(property "Reference" "#PWR01507"
+		(property "Reference" "#PWR01501"
 			(at 101.6 104.14 0)
 			(effects
@@
 			)
 		)
-		(property "Description" ""
+		(property "Description" "Power symbol creates a global label with name \"GNDPWR\" , global ground"
 			(at 106.68 104.14 0)
 			(effects
@@
 			(project "ETH1LCR3"
 				(path "/6623bacb-57aa-43ce-9e51-b38a560dd9fc/4b99b960-154b-4647-bcd6-01f80df128c7"
-					(reference "#PWR01507")
+					(reference "#PWR01501")
 					(unit 1)
 				)
@@
 		(on_board yes)
 		(dnp no)
-		(property "Reference" "#PWR01508"
+		(property "Reference" "#PWR01507"
 			(at 129.54 104.14 0)
 			(effects
@@
 			)
 		)
-		(property "Description" ""
+		(property "Description" "Power symbol creates a global label with name \"GNDPWR\" , global ground"
 			(at 124.46 104.14 0)
 			(effects
@@
 			(project "ETH1LCR3"
 				(path "/6623bacb-57aa-43ce-9e51-b38a560dd9fc/4b99b960-154b-4647-bcd6-01f80df128c7"
-					(reference "#PWR01508")
+					(reference "#PWR01507")
 					(unit 1)
 				)

Commit message: Hardware
Parts:
- added C1501: 1u, Capacitor_SMD:C_0603_1608Metric_Pad1.08x0.95mm_HandSolder, symbol Device:C
- added K1501, K1502, K1503, K1504, K1505, K1506: HE3621A0510, ETH1LCR3:HE360_x-5050462-8, symbol ETH1LCR3:HE3621A0510
- added U1501: ULN2003A, Package_SO:TSSOP-16_4.4x5mm_P0.65mm, symbol Transistor_Array:ULN2003A
Connections:
- net EXT_TRIG: now also J1501.a16 (Pin_a16)
- net HD_REAR: now also K1501.1
- net HS_REAR: now also K1502.1
- net LD_REAR: now also K1504.1
- net LS_REAR: now also K1503.1
- net A: now reaches J1501.a2 (Pin_a2)
- net A: now also J1501.c2 (Pin_c2), K1501.4
- net B: now reaches J1501.a3 (Pin_a3)
- net B: now also J1501.c3 (Pin_c3), K1502.4
- net C: now reaches J1501.a4 (Pin_a4)
- net C: now also J1501.c4 (Pin_c4), K1505.4
- net D: now reaches J1501.a5 (Pin_a5)
- net D: now also J1501.c5 (Pin_c5), K1506.4
- net E: now reaches J1501.a6 (Pin_a6)
- net E: now also J1501.c6 (Pin_c6), K1503.4
- net F: now reaches J1501.a7 (Pin_a7)
- net F: now also J1501.c7 (Pin_c7), K1504.4
- net GNDS: now reaches J1501.c16 (Pin_c16)
- new net: K1501.3, U1501.16 (O1)
- new net: K1506.3, U1501.11 (O6)
- new net: K1505.3, U1501.12 (O5)
- new net: K1504.3, U1501.13 (O4)
- new net: K1503.3, U1501.14 (O3)
- new net: K1502.3, U1501.15 (O2)
- new net +5VP: C1501.1, K1501.2, K1502.2, K1503.2, K1504.2, K1505.2, K1506.2, U1501.9 (COM)
- new net CXN_REL1: U1501.1 (I1)
- new net CXN_REL2: U1501.2 (I2)
- new net CXN_REL3: U1501.3 (I3)
- new net CXN_REL4: U1501.4 (I4)
- new net CXN_REL5: U1501.5 (I5)
- new net CXN_REL6: U1501.6 (I6)
- new net GND: C1501.2, K1505.1, U1501.8 (GND)
Other:
- moved on the sheet: J1501

Commit message: Hardware
Parts:
- J1501: footprint (none) -> ETH1LCR3:Socket_DIN41612-CaseC1-AC-Male-64Pin-2rows
Changed lines of the file:
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@@
 			)
 		)
-		(property "Footprint" ""
+		(property "Footprint" "ETH1LCR3:Socket_DIN41612-CaseC1-AC-Male-64Pin-2rows"
 			(at 111.76 123.19 0)
 			(effects

Commit message: Hardware
Parts:
- added C1502, C1503: 0.1u, Capacitor_SMD:C_0603_1608Metric_Pad1.08x0.95mm_HandSolder, symbol Device:C
- added R1501: 1k, Resistor_SMD:R_0603_1608Metric_Pad0.98x0.95mm_HandSolder, symbol Device:R
- added R1502, R1503: 51, Resistor_SMD:R_0603_1608Metric_Pad0.98x0.95mm_HandSolder, symbol Device:R
- added U1502: LMH6644MT, Package_SO:TSSOP-14_4.4x5mm_P0.65mm, symbol ETH1LCR3:LMH6644MT
Connections:
- net GND: now also C1502.2, C1503.2, U1502.10 (+), U1502.12 (+), U1502.5 (+)
- net HS_REAR: now also K1504.1; no longer K1502.1
- net LD_REAR: now also K1502.1; no longer K1504.1
- net at K1506.1: now also R1501.2
- new net: U1502.6 (-), U1502.7
- new net: R1502.2, R1503.2, U1502.3 (+)
- new net: U1502.8, U1502.9 (-)
- new net: R1501.1, U1502.1, U1502.2 (-)
- new net: U1502.13 (-), U1502.14
- new net -5V: C1503.1, U1502.11 (V-)
- new net DC_BIAS_VOLTAGE: R1502.1
- new net SINE: R1503.1
- new net V_BOOST: C1502.1, U1502.4 (V+)
Other:
- moved on the sheet: C1501, J1501, K1501A, K1501B, K1502A, K1502B, K1503A, K1503B, K1504A, K1504B, K1505A, K1505B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

Commit message: PCB layout
Parts:
- renumbered C1502 to C1501, C1503 to C1502, C1501 to C1503, R1502 to R1501, R1503 to R1502, R1501 to R1503, U1502 to U1501, U1501 to U1502

Commit message: PCB layout
Connections:
- net at U1502.11 (O6): now also K1504.3; no longer K1506.3
- net at U1502.12 (O5): now also K1503.3; no longer K1505.3
- net at U1502.13 (O4): now also K1506.3; no longer K1504.3
- net at U1502.14 (O3): now also K1505.3; no longer K1503.3
Other:
- moved on the sheet: K1503B, K1504B, K1505B, K1506B
