File: Hardware/ETH1LCR3/IV_10k.kicad_sch (KiCad schematic)
At the start: 16 parts, among them Q901 BSS123, U1103 AQY221R2S, U901 AD8099ARDZ, U902 AQY221R2S

Commit message: PCB layout
Parts:
- added Q1102: MMBT3904, Package_TO_SOT_SMD:SOT-23, symbol Transistor_BJT:MMBT3904
- added R1107: 10k, Resistor_SMD:R_0603_1608Metric_Pad0.98x0.95mm_HandSolder, symbol Device:R
Connections:
- net GND: now also Q1102.2 (E)
- net SW3: now also R1107.2; no longer R903.1, U1103.2
- new net: Q1102.1 (B), R1107.1
- new net _SW3: Q1102.3 (C), R903.1, U1103.2
Changed lines of the file:
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@@
 		)
 	)
-	(label "SW3"
+	(label "_SW3"
 		(at 208.28 85.09 0)
 		(fields_autoplaced yes)
@@
 		)
 	)
-	(label "SW3"
+	(label "_SW3"
 		(at 111.76 111.76 0)
 		(fields_autoplaced yes)
@@
 	(hierarchical_label "SW3"
 		(shape input)
-		(at 215.9 85.09 0)
+		(at 220.98 69.85 90)
 		(fields_autoplaced yes)
 		(effects
@@
 	)
 	(symbol
+		(lib_id "power:GND")
+		(at 226.06 85.09 90)
+		(unit 1)
+		(exclude_from_sim no)
+		(in_bom yes)
+		(on_board yes)
+		(dnp no)
+		(fields_autoplaced yes)
+		(property "Reference" "#PWR01114"
+			(at 232.41 85.09 0)
+			(effects
+				(font
+					(size 1.27 1.27)
+				)
+				(hide yes)
+			)
+		)
+		(property "Value" "GND"
+			(at 229.87 85.0899 90)
+			(effects
+				(font
+					(size 1.27 1.27)
+				)
+				(justify right)
+			)
+		)
+		(property "Footprint" ""
+			(at 226.06 85.09 0)
+			(effects
+				(font
+					(size 1.27 1.27)
+				)
+				(hide yes)
+			)
+		)
+		(property "Datasheet" ""
+			(at 226.06 85.09 0)
+			(effects
+				(font
+					(size 1.27 1.27)
+				)
+				(hide yes)
+			)
+		)
+		(property "Description" "Power symbol creates a global label with name \"GND\" , ground"
+			(at 226.06 85.09 0)
+			(effects
+				(font
+					(size 1.27 1.27)
+				)
+				(hide yes)
+			)
+		)
+		(pin "1"
+		)
+		(instances
+			(project "ETH1LCR3"
+				(path "/6623bacb-57aa-43ce-9e51-b38a560dd9fc/37965f22-1055-43ab-ab57-7d9b27fac2d0/f95ea0bc-75a5-443b-a2b0-d8f3dd8654a5"
+					(reference "#PWR01114")
+					(unit 1)
+				)
+			)
+		)
+	)
+	(symbol
 		(lib_id "Device:R")
 		(at 120.65 111.76 90)
@@
 	)
 	(symbol
+		(lib_id "Device:R")
+		(at 220.98 73.66 180)
+		(unit 1)
+		(exclude_from_sim no)
+		(in_bom yes)
+		(on_board yes)
+		(dnp no)
+		(property "Reference" "R1107"
+			(at 215.9 73.66 90)
+			(effects
+				(font
+					(size 1.27 1.27)
+				)
+			)
+		)
+		(property "Value" "10k"
+			(at 218.44 73.66 90)
+			(effects
+				(font
+					(size 1.27 1.27)
+				)
+			)
+		)
+		(property "Footprint" "Resistor_SMD:R_0603_1608Metric_Pad0.98x0.95mm_HandSolder"
+			(at 222.758 73.66 90)
+			(effects
+				(font
+					(size 1.27 1.27)
+				)
+				(hide yes)
+			)
+		)
+		(property "Datasheet" "~"
+			(at 220.98 73.66 0)
+			(effects
+				(font
+					(size 1.27 1.27)
+				)
+				(hide yes)
+			)
+		)
+		(property "Description" "Resistor"
+			(at 220.98 73.66 0)
+			(effects
+				(font
+					(size 1.27 1.27)
+				)
+				(hide yes)
+			)
+		)
+		(pin "1"
+		)
+		(pin "2"
+		)
+		(instances
+			(project "ETH1LCR3"
+				(path "/6623bacb-57aa-43ce-9e51-b38a560dd9fc/37965f22-1055-43ab-ab57-7d9b27fac2d0/f95ea0bc-75a5-443b-a2b0-d8f3dd8654a5"
+					(reference "R1107")
+					(unit 1)
+				)
+			)
+		)
+	)
+	(symbol
 		(lib_id "power:+5V")
 		(at 86.36 85.09 90)
@@
 					(unit 1)
 				)
+			)
+		)
+	)
+	(symbol
+		(lib_id "Transistor_BJT:MMBT3904")
+		(at 220.98 82.55 90)
+		(mirror x)
+		(unit 1)
+		(exclude_from_sim no)
+		(in_bom yes)
+		(on_board yes)
+		(dnp no)
+		(property "Reference" "Q1102"
+			(at 227.584 77.216 90)
+			(effects
+				(font
+					(size 1.27 1.27)
+				)
+			)
+		)
+		(property "Value" "MMBT3904"
+			(at 227.584 79.756 90)
+			(effects
+				(font
+					(size 1.27 1.27)
+				)
+			)
+		)
+		(property "Footprint" "Package_TO_SOT_SMD:SOT-23"
+			(at 222.885 87.63 0)
+			(effects
+				(font
+					(size 1.27 1.27)
+					(italic yes)
+				)
+				(justify left)
+				(hide yes)
+			)
+		)
+		(property "Datasheet" "https://www.onsemi.com/pdf/datasheet/pzt3904-d.pdf"
+			(at 220.98 82.55 0)
+			(effects
+				(font
+					(size 1.27 1.27)
+				)
+				(justify left)
+				(hide yes)
+			)
+		)
+		(property "Description" "0.2A Ic, 40V Vce, Small Signal NPN Transistor, SOT-23"
+			(at 220.98 82.55 0)
+			(effects
+				(font
+					(size 1.27 1.27)
+				)
+				(hide yes)
+			)
+		)
+		(pin "3"
+		)
+		(pin "2"
+		)
+		(pin "1"
+		)
+		(instances
+			(project "ETH1LCR3"
+				(path "/6623bacb-57aa-43ce-9e51-b38a560dd9fc/37965f22-1055-43ab-ab57-7d9b27fac2d0/f95ea0bc-75a5-443b-a2b0-d8f3dd8654a5"
+					(reference "Q1102")
+					(unit 1)
+				)

Commit message: Updated project to KiCAD 9
Parts:
- renumbered C905 to C1102, C903 to C1103, C901 to C1104, C904 to C1105, Q901 to Q1101, R906 to R1101, R903 to R1102, R902 to R1103, R904 to R1104, R901 to R1105, U902 to U1101, U901 to U1102
Changed lines of the file:
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@@
 (kicad_sch
-	(version 20231120)
+	(version 20250114)
 	(generator "eeschema")
-	(generator_version "8.0")
+	(generator_version "9.0")
 	(paper "A4")
 	(junction
@@
 	(label "_SW3"
 		(at 208.28 85.09 0)
-		(fields_autoplaced yes)
 		(effects
 			(font
@@
 	(label "_SW3"
 		(at 111.76 111.76 0)
-		(fields_autoplaced yes)
 		(effects
 			(font
@@
 		(shape bidirectional)
 		(at 68.58 90.17 180)
-		(fields_autoplaced yes)
 		(effects
 			(font
@@
 		(shape input)
 		(at 220.98 69.85 90)
-		(fields_autoplaced yes)
 		(effects
 			(font
@@
 		(shape bidirectional)
 		(at 227.33 90.17 0)
-		(fields_autoplaced yes)
 		(effects
 			(font
@@
 		(on_board yes)
 		(dnp no)
-		(property "Reference" "#PWR0905"
+		(property "Reference" "#PWR01109"
 			(at 146.05 90.17 0)
 			(effects
@@
 		(on_board yes)
 		(dnp no)
-		(property "Reference" "U901"
+		(property "Reference" "U1102"
 			(at 158.496 87.63 0)
 			(effects
@@
 		(dnp no)
 		(fields_autoplaced yes)
-		(property "Reference" "C904"
+		(property "Reference" "C1105"
 			(at 156.21 60.96 90)
 			(effects
@@
 		(on_board yes)
 		(dnp no)
-		(property "Reference" "C901"
+		(property "Reference" "C1104"
 			(at 158.75 113.0299 0)
 			(effects
@@
 		(dnp no)
 		(fields_autoplaced yes)
-		(property "Reference" "C905"
+		(property "Reference" "C1102"
 			(at 146.05 179.0699 0)
 			(effects
@@
 		(on_board yes)
 		(dnp no)
-		(property "Reference" "R906"
+		(property "Reference" "R1101"
 			(at 91.44 80.264 90)
 			(effects
@@
 		(dnp no)
 		(fields_autoplaced yes)
-		(property "Reference" "#PWR0904"
+		(property "Reference" "#PWR01102"
 			(at 127 93.98 0)
 			(effects
@@
 		(on_board yes)
 		(dnp no)
-		(property "Reference" "R902"
+		(property "Reference" "R1103"
 			(at 127 91.44 90)
 			(effects
@@
 		(dnp no)
 		(fields_autoplaced yes)
-		(property "Reference" "#PWR0907"
+		(property "Reference" "#PWR01113"
 			(at 176.53 68.58 0)
 			(effects
@@
 		(dnp no)
 		(fields_autoplaced yes)
-		(property "Reference" "Q901"
+		(property "Reference" "Q1101"
 			(at 135.89 110.4899 0)
 			(effects
@@
 		(on_board yes)
 		(dnp no)
-		(property "Reference" "R903"
+		(property "Reference" "R1102"
 			(at 120.65 106.68 90)
 			(effects
@@
 		(dnp no)
 		(fields_autoplaced yes)
-		(property "Reference" "R901"
+		(property "Reference" "R1105"
 			(at 157.48 102.8699 0)
 			(effects
@@
 		(dnp no)
 		(fields_autoplaced yes)
-		(property "Reference" "U902"
+		(property "Reference" "U1101"
 			(at 105.41 77.47 0)
 			(effects
@@
 		(dnp no)
 		(fields_autoplaced yes)
-		(property "Reference" "R904"
+		(property "Reference" "R1104"
 			(at 143.51 72.39 90)
 			(effects
@@
 		(dnp no)
 		(fields_autoplaced yes)
-		(property "Reference" "#PWR0908"
+		(property "Reference" "#PWR01101"
 			(at 90.17 85.09 0)
 			(effects
@@
 		(dnp yes)
 		(fields_autoplaced yes)
-		(property "Reference" "C903"
+		(property "Reference" "C1103"
 			(at 143.51 60.96 90)
 			(effects
@@
 		(on_board yes)
 		(dnp no)
-		(property "Reference" "#PWR0906"
+		(property "Reference" "#PWR01110"
 			(at 146.05 97.79 0)
 			(effects
@@
 		(dnp no)
 		(fields_autoplaced yes)
-		(property "Reference" "#PWR0902"
+		(property "Reference" "#PWR01106"
 			(at 134.62 97.79 0)
 			(effects
@@
 		(dnp no)
 		(fields_autoplaced yes)
-		(property "Reference" "#PWR0901"
+		(property "Reference" "#PWR01112"
 			(at 154.94 114.3 0)
 			(effects
