File: Hardware/ETH1LCR3/IV_1k.kicad_sch (KiCad schematic)
At the start: 16 parts, among them Q901 BSS123, U1003 AQY221R2S, U901 AD8099ARDZ, U902 AQY221R2S

Commit message: Hardware
Parts:
- renumbered C905 to C1002, C903 to C1003, C901 to C1004, C904 to C1005, Q901 to Q1001, R906 to R1001, R903 to R1002, R902 to R1003, R904 to R1004, R901 to R1005, U902 to U1001, U901 to U1002
Changed lines of the file:
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@@
 		(on_board yes)
 		(dnp no)
-		(property "Reference" "#PWR0905"
+		(property "Reference" "#PWR01009"
 			(at 146.05 90.17 0)
 			(effects
@@
 		(dnp no)
 		(fields_autoplaced yes)
-		(property "Reference" "Q901"
+		(property "Reference" "Q1001"
 			(at 135.89 110.4899 0)
 			(effects
@@
 		(on_board yes)
 		(dnp no)
-		(property "Reference" "C901"
+		(property "Reference" "C1004"
 			(at 158.75 113.0299 0)
 			(effects
@@
 		(dnp no)
 		(fields_autoplaced yes)
-		(property "Reference" "U902"
+		(property "Reference" "U1001"
 			(at 105.41 77.47 0)
 			(effects
@@
 		(on_board yes)
 		(dnp no)
-		(property "Reference" "R902"
+		(property "Reference" "R1003"
 			(at 127 91.44 90)
 			(effects
@@
 		(dnp no)
 		(fields_autoplaced yes)
-		(property "Reference" "C905"
+		(property "Reference" "C1002"
 			(at 146.05 179.0699 0)
 			(effects
@@
 		(dnp no)
 		(fields_autoplaced yes)
-		(property "Reference" "R904"
+		(property "Reference" "R1004"
 			(at 143.51 72.39 90)
 			(effects
@@
 		(dnp no)
 		(fields_autoplaced yes)
-		(property "Reference" "R901"
+		(property "Reference" "R1005"
 			(at 157.48 102.8699 0)
 			(effects
@@
 		(dnp no)
 		(fields_autoplaced yes)
-		(property "Reference" "#PWR0907"
+		(property "Reference" "#PWR01013"
 			(at 176.53 68.58 0)
 			(effects
@@
 		(on_board yes)
 		(dnp no)
-		(property "Reference" "R906"
+		(property "Reference" "R1001"
 			(at 91.44 80.264 90)
 			(effects
@@
 		(on_board yes)
 		(dnp no)
-		(property "Reference" "#PWR0906"
+		(property "Reference" "#PWR01010"
 			(at 146.05 97.79 0)
 			(effects
@@
 		(dnp no)
 		(fields_autoplaced yes)
-		(property "Reference" "#PWR0901"
+		(property "Reference" "#PWR01012"
 			(at 154.94 114.3 0)
 			(effects
@@
 		(on_board yes)
 		(dnp no)
-		(property "Reference" "R903"
+		(property "Reference" "R1002"
 			(at 120.65 106.68 90)
 			(effects
@@
 		(dnp no)
 		(fields_autoplaced yes)
-		(property "Reference" "#PWR0902"
+		(property "Reference" "#PWR01006"
 			(at 134.62 97.79 0)
 			(effects
@@
 		(dnp no)
 		(fields_autoplaced yes)
-		(property "Reference" "#PWR0904"
+		(property "Reference" "#PWR01002"
 			(at 127 93.98 0)
 			(effects
@@
 		(on_board yes)
 		(dnp no)
-		(property "Reference" "U901"
+		(property "Reference" "U1002"
 			(at 158.496 87.63 0)
 			(effects
@@
 		(dnp no)
 		(fields_autoplaced yes)
-		(property "Reference" "C904"
+		(property "Reference" "C1005"
 			(at 156.21 60.96 90)
 			(effects
@@
 		(dnp no)
 		(fields_autoplaced yes)
-		(property "Reference" "#PWR0908"
+		(property "Reference" "#PWR01001"
 			(at 90.17 85.09 0)
 			(effects
@@
 		(dnp yes)
 		(fields_autoplaced yes)
-		(property "Reference" "C903"
+		(property "Reference" "C1003"
 			(at 143.51 60.96 90)
 			(effects

Commit message: PCB layout
Parts:
- added Q1002: MMBT3904, Package_TO_SOT_SMD:SOT-23, symbol Transistor_BJT:MMBT3904
- added R1007: 10k, Resistor_SMD:R_0603_1608Metric_Pad0.98x0.95mm_HandSolder, symbol Device:R
Connections:
- net GND: now also Q1002.2 (E)
- net SW2: now also R1007.2; no longer R1002.1, U1003.2
- new net: Q1002.1 (B), R1007.1
- new net _SW2: Q1002.3 (C), R1002.1, U1003.2
Changed lines of the file:
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@@
 		)
 	)
-	(label "SW2"
+	(label "_SW2"
 		(at 208.28 85.09 0)
 		(fields_autoplaced yes)
@@
 		)
 	)
-	(label "SW2"
+	(label "_SW2"
 		(at 111.76 111.76 0)
 		(fields_autoplaced yes)
@@
 	(hierarchical_label "SW2"
 		(shape input)
-		(at 215.9 85.09 0)
+		(at 220.98 69.85 90)
 		(fields_autoplaced yes)
 		(effects
@@
 	)
 	(symbol
+		(lib_id "Transistor_BJT:MMBT3904")
+		(at 220.98 82.55 90)
+		(mirror x)
+		(unit 1)
+		(exclude_from_sim no)
+		(in_bom yes)
+		(on_board yes)
+		(dnp no)
+		(property "Reference" "Q1002"
+			(at 227.584 77.216 90)
+			(effects
+				(font
+					(size 1.27 1.27)
+				)
+			)
+		)
+		(property "Value" "MMBT3904"
+			(at 227.584 79.756 90)
+			(effects
+				(font
+					(size 1.27 1.27)
+				)
+			)
+		)
+		(property "Footprint" "Package_TO_SOT_SMD:SOT-23"
+			(at 222.885 87.63 0)
+			(effects
+				(font
+					(size 1.27 1.27)
+					(italic yes)
+				)
+				(justify left)
+				(hide yes)
+			)
+		)
+		(property "Datasheet" "https://www.onsemi.com/pdf/datasheet/pzt3904-d.pdf"
+			(at 220.98 82.55 0)
+			(effects
+				(font
+					(size 1.27 1.27)
+				)
+				(justify left)
+				(hide yes)
+			)
+		)
+		(property "Description" "0.2A Ic, 40V Vce, Small Signal NPN Transistor, SOT-23"
+			(at 220.98 82.55 0)
+			(effects
+				(font
+					(size 1.27 1.27)
+				)
+				(hide yes)
+			)
+		)
+		(pin "3"
+		)
+		(pin "2"
+		)
+		(pin "1"
+		)
+		(instances
+			(project "ETH1LCR3"
+				(path "/6623bacb-57aa-43ce-9e51-b38a560dd9fc/37965f22-1055-43ab-ab57-7d9b27fac2d0/24021e57-4b56-4fc1-baed-9b3f1e825e72"
+					(reference "Q1002")
+					(unit 1)
+				)
+			)
+		)
+	)
+	(symbol
 		(lib_id "Device:R")
 		(at 154.94 104.14 0)
@@
 	)
 	(symbol
+		(lib_id "Device:R")
+		(at 220.98 73.66 180)
+		(unit 1)
+		(exclude_from_sim no)
+		(in_bom yes)
+		(on_board yes)
+		(dnp no)
+		(property "Reference" "R1007"
+			(at 215.9 73.66 90)
+			(effects
+				(font
+					(size 1.27 1.27)
+				)
+			)
+		)
+		(property "Value" "10k"
+			(at 218.44 73.66 90)
+			(effects
+				(font
+					(size 1.27 1.27)
+				)
+			)
+		)
+		(property "Footprint" "Resistor_SMD:R_0603_1608Metric_Pad0.98x0.95mm_HandSolder"
+			(at 222.758 73.66 90)
+			(effects
+				(font
+					(size 1.27 1.27)
+				)
+				(hide yes)
+			)
+		)
+		(property "Datasheet" "~"
+			(at 220.98 73.66 0)
+			(effects
+				(font
+					(size 1.27 1.27)
+				)
+				(hide yes)
+			)
+		)
+		(property "Description" "Resistor"
+			(at 220.98 73.66 0)
+			(effects
+				(font
+					(size 1.27 1.27)
+				)
+				(hide yes)
+			)
+		)
+		(pin "1"
+		)
+		(pin "2"
+		)
+		(instances
+			(project "ETH1LCR3"
+				(path "/6623bacb-57aa-43ce-9e51-b38a560dd9fc/37965f22-1055-43ab-ab57-7d9b27fac2d0/24021e57-4b56-4fc1-baed-9b3f1e825e72"
+					(reference "R1007")
+					(unit 1)
+				)
+			)
+		)
+	)
+	(symbol
 		(lib_id "power:+5V")
 		(at 142.24 176.53 0)
@@
 					(unit 1)
 				)
+			)
+		)
+	)
+	(symbol
+		(lib_id "power:GND")
+		(at 226.06 85.09 90)
+		(unit 1)
+		(exclude_from_sim no)
+		(in_bom yes)
+		(on_board yes)
+		(dnp no)
+		(fields_autoplaced yes)
+		(property "Reference" "#PWR01014"
+			(at 232.41 85.09 0)
+			(effects
+				(font
+					(size 1.27 1.27)
+				)
+				(hide yes)
+			)
+		)
+		(property "Value" "GND"
+			(at 229.87 85.0899 90)
+			(effects
+				(font
+					(size 1.27 1.27)
+				)
+				(justify right)
+			)
+		)
+		(property "Footprint" ""
+			(at 226.06 85.09 0)
+			(effects
+				(font
+					(size 1.27 1.27)
+				)
+				(hide yes)
+			)
+		)
+		(property "Datasheet" ""
+			(at 226.06 85.09 0)
+			(effects
+				(font
+					(size 1.27 1.27)
+				)
+				(hide yes)
+			)
+		)
+		(property "Description" "Power symbol creates a global label with name \"GND\" , ground"
+			(at 226.06 85.09 0)
+			(effects
+				(font
+					(size 1.27 1.27)
+				)
+				(hide yes)
+			)
+		)
+		(pin "1"
+		)
+		(instances
+			(project "ETH1LCR3"
+				(path "/6623bacb-57aa-43ce-9e51-b38a560dd9fc/37965f22-1055-43ab-ab57-7d9b27fac2d0/24021e57-4b56-4fc1-baed-9b3f1e825e72"
+					(reference "#PWR01014")
+					(unit 1)
+				)
