File: Hardware/ETH1LCR3/PGA.kicad_sch (KiCad schematic)
At the start: 32 parts, among them U601 LMH6720MA, U602 LMH6720MA, U603 LMH6720MA, U604 LMH6618MK

Commit message: Schematic
Parts:
- added C609, C610, C611, C612, C613, C614, C615, C616, C617, C618: 0.1u, Capacitor_SMD:C_0603_1608Metric_Pad1.08x0.95mm_HandSolder, symbol Device:C
- added R621: 150/0.1%, Resistor_SMD:R_0603_1608Metric_Pad0.98x0.95mm_HandSolder, symbol Device:R
- added R622: 91/0.1%, Resistor_SMD:R_0603_1608Metric_Pad0.98x0.95mm_HandSolder, symbol Device:R
- added R623, R624: 30/0.1%, Resistor_SMD:R_0603_1608Metric_Pad0.98x0.95mm_HandSolder, symbol Device:R
- added U605: ADG1604BRUZ, Package_SO:TSSOP-14_4.4x5mm_P0.65mm, symbol ETH1LCR3:ADG1604BRUZ
- C601, C602, C604, C606, C607, C608: footprint (none) -> Capacitor_SMD:C_0603_1608Metric_Pad1.08x0.95mm_HandSolder
- R601, R602, R603, R604, R605, R606, R607, R608, R609, R610, R611, R612, R613, R614, R615, R616, R617, R618, R619, R620: footprint (none) -> Resistor_SMD:R_0603_1608Metric_Pad0.98x0.95mm_HandSolder
Connections:
- net GND: now also C609.2, C610.2, C611.2, C612.2, C613.2, C614.2, C615.2, C616.2, C617.2, C618.2, R624.2, U605.13 (GND)
- net at R620.2: now also U605.6 (D)
- net at U601.3 (+), U602.3 (+), U603.3 (+): now also C607.2, U604.1, R621.1, U605.4 (S1)
- net +5VA renamed +5V
- net +5V: now also C609.1, C610.1, C611.1, C612.1, C613.1, U605.12 (VDD), U605.2 (EN)
- net -5VA renamed -5V
- net -5V: now also C614.1, C615.1, C616.1, C617.1, C618.1, U605.3 (VSS)
- new net: R622.2, R623.1, U605.11 (S3)
- new net: R623.2, R624.1, U605.10 (S4)
- new net: R621.2, R622.1, U605.5 (S2)
- new net PGA_A0: U605.1 (A0)
- new net PGA_A1: U605.14 (A1)
Other:
- moved on the sheet: C601, C602, C603, C604, C605, C606, C607, C608, R601, R602, R603, R604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

Commit message: Hardware
Parts:
- renumbered C608 to C601, C607 to C602, C605 to C603, C606 to C604, C614 to C605, C615 to C606, C603 to C607, C616 to C608, C602 to C609, C617 to C610, C618 to C611, C609 to C612, C610 to C613, C601 to C614, C611 to C615, C604 to C616, C612 to C617, C613 to C618, R616 to R601, R615 to R602, R620 to R603, R614 to R604, R617 to R605, R618 to R606, R619 to R607, R621 to R608, R622 to R609, R623 to R610, R624 to R611, R608 to R612, R609 to R613, R610 to R614, R612 to R615, R611 to R616, R613 to R617, R604 to R618, R603 to R619, R602 to R620, R601 to R621, R605 to R622, R606 to R623, R607 to R624, U604 to U601, U605 to U602, U602 to U604, U601 to U605

Commit message: Hardware
Parts:
- C603, C607: value C_Trim -> JZ200; footprint (none) -> Capacitor_SMD:C_Trimmer_Voltronics_JZ
Changed lines of the file:
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@@
 			)
 		)
-		(property "Value" "C_Trim"
+		(property "Value" "JZ200"
 			(at 102.87 69.5959 0)
 			(effects
@@
 			)
 		)
-		(property "Footprint" ""
+		(property "Footprint" "Capacitor_SMD:C_Trimmer_Voltronics_JZ"
 			(at 99.06 68.58 0)
 			(effects
@@
 			)
 		)
-		(property "Value" "C_Trim"
+		(property "Value" "JZ200"
 			(at 175.26 69.5959 0)
 			(effects
@@
 			)
 		)
-		(property "Footprint" ""
+		(property "Footprint" "Capacitor_SMD:C_Trimmer_Voltronics_JZ"
 			(at 171.45 68.58 0)
 			(effects

Commit message: PCB layout
Parts:
- added R625, R626: 51, Resistor_SMD:R_0603_1608Metric_Pad0.98x0.95mm_HandSolder, symbol Device:R
- C602, R619: now not fitted; now left out of the parts list
- U601: value LMH6618MK -> LMH6618MKE; footprint Package_TO_SOT_SMD:TSOT-23-6 -> Package_TO_SOT_SMD:SOT-23-6_Handsoldering
- U603, U604, U605: value LMH6720MA -> LMH6720MF; symbol ETH1LCR3:LMH6702MA -> ETH1LCR3:LMH6720MF
Connections:
- net PGA_A0: now also R626.1; no longer U602.1 (A0)
- net PGA_A1: now also R625.1; no longer U602.14 (A1)
- new net: R626.2, U602.1 (A0)
- new net: R625.2, U602.14 (A1)
Changed lines of the file:
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@@
 	(wire
 		(pts
-			(xy 44.45 160.02) (xy 53.34 160.02)
+			(xy 33.02 160.02) (xy 36.83 160.02)
 		)
 		(stroke
@@
 	(wire
 		(pts
+			(xy 44.45 157.48) (xy 53.34 157.48)
+		)
+		(stroke
+			(width 0)
+			(type default)
+		)
+	)
+	(wire
+		(pts
 			(xy 246.38 154.94) (xy 246.38 156.21)
 		)
@@
 	(wire
 		(pts
+			(xy 44.45 160.02) (xy 53.34 160.02)
+		)
+		(stroke
+			(width 0)
+			(type default)
+		)
+	)
+	(wire
+		(pts
 			(xy 83.82 149.86) (xy 83.82 144.78)
 		)
@@
 	(wire
 		(pts
-			(xy 44.45 157.48) (xy 53.34 157.48)
+			(xy 33.02 157.48) (xy 36.83 157.48)
 		)
 		(stroke
@@
 	(hierarchical_label "PGA_A0"
 		(shape input)
-		(at 44.45 160.02 180)
+		(at 33.02 160.02 180)
 		(fields_autoplaced yes)
 		(effects
@@
 	(hierarchical_label "PGA_A1"
 		(shape input)
-		(at 44.45 157.48 180)
+		(at 33.02 157.48 180)
 		(fields_autoplaced yes)
 		(effects
@@
 	)
 	(symbol
+		(lib_id "Device:R")
+		(at 40.64 160.02 90)
+		(mirror x)
+		(unit 1)
+		(exclude_from_sim no)
+		(in_bom yes)
+		(on_board yes)
+		(dnp no)
+		(property "Reference" "R626"
+			(at 40.64 164.846 90)
+			(effects
+				(font
+					(size 1.27 1.27)
+				)
+			)
+		)
+		(property "Value" "51"
+			(at 40.64 162.306 90)
+			(effects
+				(font
+					(size 1.27 1.27)
+				)
+			)
+		)
+		(property "Footprint" "Resistor_SMD:R_0603_1608Metric_Pad0.98x0.95mm_HandSolder"
+			(at 40.64 158.242 90)
+			(effects
+				(font
+					(size 1.27 1.27)
+				)
+				(hide yes)
+			)
+		)
+		(property "Datasheet" "~"
+			(at 40.64 160.02 0)
+			(effects
+				(font
+					(size 1.27 1.27)
+				)
+				(hide yes)
+			)
+		)
+		(property "Description" "Resistor"
+			(at 40.64 160.02 0)
+			(effects
+				(font
+					(size 1.27 1.27)
+				)
+				(hide yes)
+			)
+		)
+		(pin "1"
+		)
+		(pin "2"
+		)
+		(instances
+			(project "ETH1LCR3"
+				(path "/6623bacb-57aa-43ce-9e51-b38a560dd9fc/a955767b-836b-415d-9ade-bdfb6e1524e6"
+					(reference "R626")
+					(unit 1)
+				)
+			)
+		)
+	)
+	(symbol
 		(lib_id "power:-5V")
 		(at 62.23 168.91 180)
@@
 		(unit 1)
 		(exclude_from_sim no)
-		(in_bom yes)
+		(in_bom no)
 		(on_board yes)
-		(dnp no)
+		(dnp yes)
 		(fields_autoplaced yes)
 		(property "Reference" "R619"
@@
 	)
 	(symbol
-		(lib_id "ETH1LCR3:LMH6702MA")
+		(lib_id "ETH1LCR3:LMH6720MF")
 		(at 215.9 38.1 0)
 		(unit 1)
@@
 			)
 		)
-		(property "Value" "LMH6720MA"
+		(property "Value" "LMH6720MF"
 			(at 220.218 33.02 0)
 			(effects
@@
 		(unit 1)
 		(exclude_from_sim no)
-		(in_bom yes)
+		(in_bom no)
 		(on_board yes)
-		(dnp no)
+		(dnp yes)
 		(fields_autoplaced yes)
 		(property "Reference" "C602"
@@
 	)
 	(symbol
-		(lib_id "ETH1LCR3:LMH6702MA")
+		(lib_id "ETH1LCR3:LMH6720MF")
 		(at 143.51 38.1 0)
 		(unit 1)
@@
 			)
 		)
-		(property "Value" "LMH6720MA"
+		(property "Value" "LMH6720MF"
 			(at 147.828 33.02 0)
 			(effects
@@
 			)
 		)
-		(property "Value" "LMH6618MK"
+		(property "Value" "LMH6618MKE"
 			(at 65.786 111.252 0)
 			(effects
@@
 			)
 		)
-		(property "Footprint" "Package_TO_SOT_SMD:TSOT-23-6"
+		(property "Footprint" "Package_TO_SOT_SMD:SOT-23-6_Handsoldering"
 			(at 63.5 121.92 0)
 			(effects
@@
 	)
 	(symbol
-		(lib_id "ETH1LCR3:LMH6702MA")
+		(lib_id "ETH1LCR3:LMH6720MF")
 		(at 69.85 38.1 0)
 		(unit 1)
@@
 			)
 		)
-		(property "Value" "LMH6720MA"
+		(property "Value" "LMH6720MF"
 			(at 74.168 33.02 0)
 			(effects
@@
 					(unit 1)
 				)
+			)
+		)
+	)
+	(symbol
+		(lib_id "Device:R")
+		(at 40.64 157.48 90)
+		(unit 1)
+		(exclude_from_sim no)
+		(in_bom yes)
+		(on_board yes)
+		(dnp no)
+		(property "Reference" "R625"
+			(at 40.64 152.654 90)
+			(effects
+				(font
+					(size 1.27 1.27)
+				)
+			)
+		)
+		(property "Value" "51"
+			(at 40.64 155.194 90)
+			(effects
+				(font
+					(size 1.27 1.27)
+				)
+			)
+		)
+		(property "Footprint" "Resistor_SMD:R_0603_1608Metric_Pad0.98x0.95mm_HandSolder"
+			(at 40.64 159.258 90)
+			(effects
+				(font
+					(size 1.27 1.27)
+				)
+				(hide yes)
+			)
+		)
+		(property "Datasheet" "~"
+			(at 40.64 157.48 0)
+			(effects
+				(font
+					(size 1.27 1.27)
+				)
+				(hide yes)
+			)
+		)
+		(property "Description" "Resistor"
+			(at 40.64 157.48 0)
+			(effects
+				(font
+					(size 1.27 1.27)
+				)
+				(hide yes)
+			)
+		)
+		(pin "1"
+		)
+		(pin "2"
+		)
+		(instances
+			(project "ETH1LCR3"
+				(path "/6623bacb-57aa-43ce-9e51-b38a560dd9fc/a955767b-836b-415d-9ade-bdfb6e1524e6"
+					(reference "R625")
+					(unit 1)
+				)

Commit message: PCB layout
Parts:
- renumbered R625 to R602, R626 to R603, R602 to R604, R603 to R605, R604 to R606, R605 to R607, R606 to R608, R607 to R609, R608 to R610, R609 to R611, R610 to R612, R611 to R613, R612 to R614, R613 to R615, R614 to R616, R615 to R617, R616 to R618, R617 to R619, R618 to R620, R619 to R621, R620 to R622, R621 to R623, R622 to R624, R623 to R625, R624 to R626
Changed lines of the file:
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@@
 		(dnp no)
 		(fields_autoplaced yes)
-		(property "Reference" "R623"
+		(property "Reference" "R625"
 			(at 233.68 64.7699 0)
 			(effects
@@
 			(project ""
 				(path "/6623bacb-57aa-43ce-9e51-b38a560dd9fc/a955767b-836b-415d-9ade-bdfb6e1524e6"
-					(reference "R623")
+					(reference "R625")
 					(unit 1)
 				)
@@
 		(dnp no)
 		(fields_autoplaced yes)
-		(property "Reference" "R620"
+		(property "Reference" "R622"
 			(at 209.55 60.9599 0)
 			(effects
@@
 			(project ""
 				(path "/6623bacb-57aa-43ce-9e51-b38a560dd9fc/a955767b-836b-415d-9ade-bdfb6e1524e6"
-					(reference "R620")
+					(reference "R622")
 					(unit 1)
 				)
@@
 		(dnp no)
 		(fields_autoplaced yes)
-		(property "Reference" "R621"
+		(property "Reference" "R623"
 			(at 228.6 44.4499 0)
 			(effects
@@
 			(project ""
 				(path "/6623bacb-57aa-43ce-9e51-b38a560dd9fc/a955767b-836b-415d-9ade-bdfb6e1524e6"
-					(reference "R621")
+					(reference "R623")
 					(unit 1)
 				)
@@
 		(dnp no)
 		(fields_autoplaced yes)
-		(property "Reference" "R610"
+		(property "Reference" "R612"
 			(at 90.17 158.7499 0)
 			(effects
@@
 			(project "ETH1LCR3"
 				(path "/6623bacb-57aa-43ce-9e51-b38a560dd9fc/a955767b-836b-415d-9ade-bdfb6e1524e6"
-					(reference "R610")
+					(reference "R612")
 					(unit 1)
 				)
@@
 		(dnp no)
 		(fields_autoplaced yes)
-		(property "Reference" "R608"
+		(property "Reference" "R610"
 			(at 90.17 138.4299 0)
 			(effects
@@
 			(project ""
 				(path "/6623bacb-57aa-43ce-9e51-b38a560dd9fc/a955767b-836b-415d-9ade-bdfb6e1524e6"
-					(reference "R608")
+					(reference "R610")
 					(unit 1)
 				)
@@
 		(on_board yes)
 		(dnp no)
-		(property "Reference" "R626"
+		(property "Reference" "R603"
 			(at 40.64 164.846 90)
 			(effects
@@
 			(project "ETH1LCR3"
 				(path "/6623bacb-57aa-43ce-9e51-b38a560dd9fc/a955767b-836b-415d-9ade-bdfb6e1524e6"
-					(reference "R626")
+					(reference "R603")
 					(unit 1)
 				)
@@
 		(dnp no)
 		(fields_autoplaced yes)
-		(property "Reference" "R617"
+		(property "Reference" "R619"
 			(at 161.29 64.7699 0)
 			(effects
@@
 			(project "ETH1LCR3"
 				(path "/6623bacb-57aa-43ce-9e51-b38a560dd9fc/a955767b-836b-415d-9ade-bdfb6e1524e6"
-					(reference "R617")
+					(reference "R619")
 					(unit 1)
 				)
@@
 		(dnp no)
 		(fields_autoplaced yes)
-		(property "Reference" "R612"
+		(property "Reference" "R614"
 			(at 116.84 57.1499 0)
 			(effects
@@
 			(project "ETH1LCR3"
 				(path "/6623bacb-57aa-43ce-9e51-b38a560dd9fc/a955767b-836b-415d-9ade-bdfb6e1524e6"
-					(reference "R612")
+					(reference "R614")
 					(unit 1)
 				)
@@
 		(on_board yes)
 		(dnp no)
-		(property "Reference" "R605"
+		(property "Reference" "R607"
 			(at 80.01 56.134 90)
 			(effects
@@
 			(project "ETH1LCR3"
 				(path "/6623bacb-57aa-43ce-9e51-b38a560dd9fc/a955767b-836b-415d-9ade-bdfb6e1524e6"
-					(reference "R605")
+					(reference "R607")
 					(unit 1)
 				)
@@
 		(dnp no)
 		(fields_autoplaced yes)
-		(property "Reference" "R616"
+		(property "Reference" "R618"
 			(at 161.29 44.4499 0)
 			(effects
@@
 			(project "ETH1LCR3"
 				(path "/6623bacb-57aa-43ce-9e51-b38a560dd9fc/a955767b-836b-415d-9ade-bdfb6e1524e6"
-					(reference "R616")
+					(reference "R618")
 					(unit 1)
 				)
@@
 		(dnp no)
 		(fields_autoplaced yes)
-		(property "Reference" "R603"
+		(property "Reference" "R605"
 			(at 53.34 132.0799 0)
 			(effects
@@
 			(project ""
 				(path "/6623bacb-57aa-43ce-9e51-b38a560dd9fc/a955767b-836b-415d-9ade-bdfb6e1524e6"
-					(reference "R603")
+					(reference "R605")
 					(unit 1)
 				)
@@
 		(on_board yes)
 		(dnp no)
-		(property "Reference" "R615"
+		(property "Reference" "R617"
 			(at 153.67 56.134 90)
 			(effects
@@
 			(project "ETH1LCR3"
 				(path "/6623bacb-57aa-43ce-9e51-b38a560dd9fc/a955767b-836b-415d-9ade-bdfb6e1524e6"
-					(reference "R615")
+					(reference "R617")
 					(unit 1)
 				)
@@
 		(dnp no)
 		(fields_autoplaced yes)
-		(property "Reference" "R606"
+		(property "Reference" "R608"
 			(at 87.63 44.4499 0)
 			(effects
@@
 			(project "ETH1LCR3"
 				(path "/6623bacb-57aa-43ce-9e51-b38a560dd9fc/a955767b-836b-415d-9ade-bdfb6e1524e6"
-					(reference "R606")
+					(reference "R608")
 					(unit 1)
 				)
@@
 		(dnp no)
 		(fields_autoplaced yes)
-		(property "Reference" "R624"
+		(property "Reference" "R626"
 			(at 257.81 53.3399 0)
 			(effects
@@
 			(project ""
 				(path "/6623bacb-57aa-43ce-9e51-b38a560dd9fc/a955767b-836b-415d-9ade-bdfb6e1524e6"
-					(reference "R624")
+					(reference "R626")
 					(unit 1)
 				)
@@
 		(dnp yes)
 		(fields_autoplaced yes)
-		(property "Reference" "R619"
+		(property "Reference" "R621"
 			(at 199.39 60.9599 0)
 			(effects
@@
 			(project "ETH1LCR3"
 				(path "/6623bacb-57aa-43ce-9e51-b38a560dd9fc/a955767b-836b-415d-9ade-bdfb6e1524e6"
-					(reference "R619")
+					(reference "R621")
 					(unit 1)
 				)
@@
 		(on_board yes)
 		(dnp no)
-		(property "Reference" "R604"
+		(property "Reference" "R606"
 			(at 66.04 119.634 90)
 			(effects
@@
 			(project ""
 				(path "/6623bacb-57aa-43ce-9e51-b38a560dd9fc/a955767b-836b-415d-9ade-bdfb6e1524e6"
-					(reference "R604")
+					(reference "R606")
 					(unit 1)
 				)
@@
 		(dnp no)
 		(fields_autoplaced yes)
-		(property "Reference" "R607"
+		(property "Reference" "R609"
 			(at 87.63 64.7699 0)
 			(effects
@@
 			(project "ETH1LCR3"
 				(path "/6623bacb-57aa-43ce-9e51-b38a560dd9fc/a955767b-836b-415d-9ade-bdfb6e1524e6"
-					(reference "R607")
+					(reference "R609")
 					(unit 1)
 				)
@@
 		(dnp no)
 		(fields_autoplaced yes)
-		(property "Reference" "R618"
+		(property "Reference" "R620"
 			(at 189.23 57.1499 0)
 			(effects
@@
 			(project ""
 				(path "/6623bacb-57aa-43ce-9e51-b38a560dd9fc/a955767b-836b-415d-9ade-bdfb6e1524e6"
-					(reference "R618")
+					(reference "R620")
 					(unit 1)
 				)
@@
 		(dnp no)
 		(fields_autoplaced yes)
-		(property "Reference" "R613"
+		(property "Reference" "R615"
 			(at 127 60.9599 0)
 			(effects
@@
 			(project "ETH1LCR3"
 				(path "/6623bacb-57aa-43ce-9e51-b38a560dd9fc/a955767b-836b-415d-9ade-bdfb6e1524e6"
-					(reference "R613")
+					(reference "R615")
 					(unit 1)
 				)
@@
 		(dnp no)
 		(fields_autoplaced yes)
-		(property "Reference" "R609"
+		(property "Reference" "R611"
 			(at 90.17 148.5899 0)
 			(effects
@@
 			(project "ETH1LCR3"
 				(path "/6623bacb-57aa-43ce-9e51-b38a560dd9fc/a955767b-836b-415d-9ade-bdfb6e1524e6"
-					(reference "R609")
+					(reference "R611")
 					(unit 1)
 				)
@@
 		(dnp no)
 		(fields_autoplaced yes)
-		(property "Reference" "R611"
+		(property "Reference" "R613"
 			(at 90.17 168.9099 0)
 			(effects
@@
 			(project "ETH1LCR3"
 				(path "/6623bacb-57aa-43ce-9e51-b38a560dd9fc/a955767b-836b-415d-9ade-bdfb6e1524e6"
-					(reference "R611")
+					(reference "R613")
 					(unit 1)
 				)
@@
 		(on_board yes)
 		(dnp no)
-		(property "Reference" "R622"
+		(property "Reference" "R624"
 			(at 226.06 56.134 90)
 			(effects
@@
 			(project ""
 				(path "/6623bacb-57aa-43ce-9e51-b38a560dd9fc/a955767b-836b-415d-9ade-bdfb6e1524e6"
-					(reference "R622")
+					(reference "R624")
 					(unit 1)
 				)
@@
 		(on_board yes)
 		(dnp no)
-		(property "Reference" "R602"
+		(property "Reference" "R604"
 			(at 45.72 108.204 90)
 			(effects
@@
 			(project ""
 				(path "/6623bacb-57aa-43ce-9e51-b38a560dd9fc/a955767b-836b-415d-9ade-bdfb6e1524e6"
-					(reference "R602")
+					(reference "R604")
 					(unit 1)
 				)
@@
 		(on_board yes)
 		(dnp no)
-		(property "Reference" "R625"
+		(property "Reference" "R602"
 			(at 40.64 152.654 90)
 			(effects
@@
 			(project "ETH1LCR3"
 				(path "/6623bacb-57aa-43ce-9e51-b38a560dd9fc/a955767b-836b-415d-9ade-bdfb6e1524e6"
-					(reference "R625")
+					(reference "R602")
 					(unit 1)
 				)
@@
 		(dnp no)
 		(fields_autoplaced yes)
-		(property "Reference" "R614"
+		(property "Reference" "R616"
 			(at 137.16 60.9599 0)
 			(effects
@@
 			(project "ETH1LCR3"
 				(path "/6623bacb-57aa-43ce-9e51-b38a560dd9fc/a955767b-836b-415d-9ade-bdfb6e1524e6"
-					(reference "R614")
+					(reference "R616")
 					(unit 1)
 				)
