File: Hardware/ETH1LCR3/Select.kicad_sch (KiCad schematic)
At the start: 8 parts, among them K1401 G5V-2-DC5, K1402 G5V-2-DC5, Q1401 MMBT3904, Q1403 MMBT3904

Commit message: Software and hardware
Parts:
- renumbered K1402 to K1401, K1401 to K1402, Q1403 to Q1402
Changed lines of the file:
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@@
 		(dnp no)
 		(fields_autoplaced yes)
-		(property "Reference" "Q1403"
+		(property "Reference" "Q1402"
 			(at 110.49 115.5699 0)
 			(effects
@@
 			(project ""
 				(path "/6623bacb-57aa-43ce-9e51-b38a560dd9fc/bf005894-f421-4bee-8b90-2513b9271d50"
-					(reference "Q1403")
+					(reference "Q1402")
 					(unit 1)
 				)
@@
 		(dnp no)
 		(fields_autoplaced yes)
-		(property "Reference" "K1402"
+		(property "Reference" "K1401"
 			(at 138.43 44.45 90)
 			(effects
@@
 			(project ""
 				(path "/6623bacb-57aa-43ce-9e51-b38a560dd9fc/bf005894-f421-4bee-8b90-2513b9271d50"
-					(reference "K1402")
+					(reference "K1401")
 					(unit 1)
 				)
@@
 		(dnp no)
 		(fields_autoplaced yes)
-		(property "Reference" "K1401"
+		(property "Reference" "K1402"
 			(at 138.43 100.33 90)
 			(effects
@@
 			(project "ETH1LCR3"
 				(path "/6623bacb-57aa-43ce-9e51-b38a560dd9fc/bf005894-f421-4bee-8b90-2513b9271d50"
-					(reference "K1401")
+					(reference "K1402")
 					(unit 1)
 				)
@@
 		(dnp no)
 		(fields_autoplaced yes)
-		(property "Reference" "#PWR01402"
+		(property "Reference" "#PWR01403"
 			(at 144.78 54.61 0)
 			(effects
@@
 			(project "ETH1LCR3"
 				(path "/6623bacb-57aa-43ce-9e51-b38a560dd9fc/bf005894-f421-4bee-8b90-2513b9271d50"
-					(reference "#PWR01402")
+					(reference "#PWR01403")
 					(unit 1)
 				)
@@
 		(dnp no)
 		(fields_autoplaced yes)
-		(property "Reference" "#PWR01403"
+		(property "Reference" "#PWR01402"
 			(at 107.95 129.54 0)
 			(effects
@@
 			(project "ETH1LCR3"
 				(path "/6623bacb-57aa-43ce-9e51-b38a560dd9fc/bf005894-f421-4bee-8b90-2513b9271d50"
-					(reference "#PWR01403")
-					(unit 1)
-				)
+					(reference "#PWR01402")
+					(unit 1)
+				)
