File: Hardware/ETH1LCR3/Trigger.kicad_sch (KiCad schematic)
At the start: 22 parts, among them U1601 TXB0104PW, U1602 ADuM5402, U1603 74AC125

Commit message: Software and hardware
Connections:
- net +5V_TRIG is gone; now on net +5VL: U1602.10 (VSEL)
- net GND_TRIG is gone; now on net GNDS: D1602.2 (A)
Other:
- moved on the sheet: C1601, C1602, C1603, C1604, C1605

Commit message: Hardware
Parts:
- C1601, C1603, C1604, C1606, C1608: value 100n -> 0.1u
- U1603: symbol ETH1CLCR2:74AC125 -> ETH1LCR3:74AC125
Connections:
- net +3V3 renamed +3.3V

Commit message: Hardware
Parts:
- L1601: footprint (none) -> ETH1LCR3:CW252016
Changed lines of the file:
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@@
 			)
 		)
-		(property "Footprint" ""
+		(property "Footprint" "ETH1LCR3:CW252016"
 			(at 222.25 137.16 0)
 			(effects

Commit message: Updated project to KiCAD 9
Changed lines of the file:
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@@
 (kicad_sch
-	(version 20231120)
+	(version 20250114)
 	(generator "eeschema")
-	(generator_version "8.0")
+	(generator_version "9.0")
 	(paper "A4")
 	(junction
@@
 	(label "TRIG_OUT_SIGN"
 		(at 232.41 40.64 180)
-		(fields_autoplaced yes)
 		(effects
 			(font
@@
 	(label "TRIG_OUT_EN"
 		(at 146.05 76.2 180)
-		(fields_autoplaced yes)
 		(effects
 			(font
@@
 	(label "EXT_TRIG_SIGN"
 		(at 146.05 81.28 180)
-		(fields_autoplaced yes)
 		(effects
 			(font
@@
 	(label "EXT_TRIG_SIGN"
 		(at 123.19 137.16 0)
-		(fields_autoplaced yes)
 		(effects
 			(font
@@
 	(label "TRIG_OUT_SIGN"
 		(at 146.05 78.74 180)
-		(fields_autoplaced yes)
 		(effects
 			(font
@@
 	(label "TRIG_OUT_EN"
 		(at 232.41 35.56 180)
-		(fields_autoplaced yes)
 		(effects
 			(font
@@
 		(shape input)
 		(at 66.04 81.28 180)
-		(fields_autoplaced yes)
 		(effects
 			(font
@@
 		(shape output)
 		(at 66.04 86.36 180)
-		(fields_autoplaced yes)
 		(effects
 			(font
@@
 		(shape bidirectional)
 		(at 254 137.16 0)
-		(fields_autoplaced yes)
 		(effects
 			(font
@@
 		(shape input)
 		(at 66.04 76.2 180)
-		(fields_autoplaced yes)
 		(effects
 			(font
